File: _PCB/_NANO prototype board/board.brd (EAGLE design)
At the start: 85.1 x 100 mm, 36 parts, among them T1_5MM 5mm, T2_5MM 5mm, T3_5MM 5mm

Commit message: optimized routes
Parts:
- moved BREAD_450 5.47 mm to (57.8, 64.6)
- moved 3.3V_C 3.92 mm to (30.1, 82.0)
- moved D_B 3.86 mm to (28.7, 72.1)
- moved R_SHIELD 3.68 mm to (22.0, 66.4), turned to 0 degrees
- moved 5V_C 0.72 mm to (20.2, 78.1)
Routing:
- net D+_B: track 14.5 -> 17.7 mm
- net D-_B: track 11.5 -> 14.7 mm
- net 5V: track 152.1 -> 153.9 mm
- net MOSI_NRF: track 42.1 -> 43.6 mm
- net 3.3V: track 171.1 -> 169.8 mm
- net SHIELD_IN: track 62.8 -> 63.7 mm
- net VIN: track 99.5 -> 100.2 mm
- net N$33: track 8.09 -> 8.69 mm
- net N$23: track 8.09 -> 8.69 mm
- net N$32: track 8.09 -> 8.67 mm
- net N$26: track 8.09 -> 8.67 mm
