File: _PCB/_NANO prototype board/board.brd (EAGLE design)
At the start: 85.1 x 100 mm, 36 parts, among them T1_5MM 5mm, T2_5MM 5mm, T3_5MM 5mm

Commit message: prototype board optimization
Parts:
- removed BREAD_450: BREADBOARDMINI, SparkFun-Boards:BREADBOARD-MINI
- added PIEZO: (no value), buzzer:F/CM12P
- added P_HIGH: (no value), pinhead_v2:1X01/OCT
- D_5PIN, D_B: device pinhead:1X02 -> SparkFun-Connectors:1X02_LOCK
- moved H2 76.7 mm to (4.19, 4.19)
- moved 3.3V 39.6 mm to (63.0, 62.2)
- moved 5V 39.6 mm to (63.0, 55.9)
- moved GND 39.6 mm to (63.0, 49.5)
- moved VIN 39.6 mm to (63.0, 68.6)
- moved GY_4-8 10.2 mm to (20.2, 43.3)
- moved GY-521 10.2 mm to (14.1, 34.4)
- moved ES32-433T20D 6.65 mm to (10.5, 9.53)
- moved 3.3/5 6.65 mm to (15.5, 20.8)
- moved J1 6.65 mm to (15.5, 1.78)
- moved TX0-D12_1 5.75 mm to (30.5, 22.0)
- moved TX0-D12_2 5.75 mm to (33.8, 22.0)
- moved NANO 2.50 mm to (45.7, 30.9)
- moved D_B 1.40 mm to (28.8, 73.5), turned to 270 degrees
- moved 5V_C 1.09 mm to (21.1, 77.5)
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Connections:
- removed net D+_B: D_B.1, USB_B.D+
- removed net D-_B: D_B.2, USB_B.D-
- new net N$34: PIEZO.+, P_HIGH.1
- new net N$35: D_B.1, USB_B.D-
- new net N$36: D_B.2, USB_B.D+
- net D+_5PIN: now also D_5PIN.2; no longer D_5PIN.1
- net D-_5PIN: now also D_5PIN.1; no longer D_5PIN.2
- net GND: now also PIEZO.-
Routing:
- net 5V: track 153.9 -> 326.9 mm
- net 3.3V: track 169.8 -> 311.1 mm
- net VIN: track 100.2 -> 147.6 mm
- net MOSI_NRF: track 43.6 -> 66.0 mm
- net D+_B: track 17.7 -> 0.00 mm
- net D-_B: track 14.7 -> 0.00 mm
- net SDA_GY521: track 70.8 -> 83.6 mm
- net N$11: track 6.35 -> 17.2 mm
- net A5: track 65.3 -> 57.5 mm
- net N$5: track 13.3 -> 20.5 mm
- net A7: track 13.3 -> 20.5 mm
- net SCK_NRF: track 83.8 -> 90.6 mm
- net CSN_NRF: track 52.0 -> 58.8 mm
- net N$24: track 13.5 -> 20.2 mm
- net N$18: track 13.5 -> 20.2 mm
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Other:
- board text added: "A4"
- board text added: "A5"
- board text added: "D0"
- board text added: "D1"
- board text added: "D10"
- board text added: "D11"
- board text added: "D12"
- board text added: "D13"
- board text added: "D2"
- board text added: "D3"
- board text added: "INT0"
- board text added: "RX"
- board text added: "SCK_LED"
- board text added: "TX"
- board text added: "~"
- board text added: "~INT1"
- board text added: "~MOSI"
- board text added: "~SS'"
- board text removed: "D0_RX"
- board text removed: "D10_SS"
- board text removed: "D11_MOSI"
- board text removed: "D12_MISO"
- board text removed: "D1_TX"
- board text removed: "D2_INT0"
- board text removed: "D3_INT1"
- board text removed: "I2C"
- board text removed: "PWM"
- board text removed: "PWM_SPI"
- board text removed: "SCK_D13"
- board text removed: "SCL_A5"
- board text removed: "SDA_A4"
- board text removed: "SPI"
- board text removed: "SPI_LED"

Commit message: dir
Parts:
- moved H1 26.3 mm to (62.9, 76.6)
Other:
- board size 85.1 x 100 mm -> 76.3 x 100 mm
Changed lines of the file:
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@@
 <fusionsync huburn="a.cGVyc29uYWw6dWUyYTRmMGNk" projecturn="a.cGVyc29uYWw6dWUyYTRmMGNkIzIwMTgwMTAyMTEwNTQ5ODMx" f3durn="urn:adsk.wipprod:dm.lineage:Bxu1HE7lTUeaXPtey1c6dw" pcbguid="eda9b9f7-04f8-461a-b123-4fdb15b2374b" lastpulledtime="" lastsyncedchangeguid="1f1fda12-eeed-9165-c6f5-a847dca60c4a"/>
 <plain>
-<wire x1="0" y1="0" x2="85.07" y2="0" width="0" layer="20"/>
-<wire x1="85.07" y1="0" x2="85.07" y2="100" width="0" layer="20"/>
-<wire x1="85.07" y1="100" x2="0" y2="100" width="0" layer="20"/>
+<wire x1="0" y1="0" x2="76.307" y2="0" width="0" layer="20"/>
+<wire x1="76.307" y1="0" x2="76.307" y2="100" width="0" layer="20"/>
+<wire x1="76.307" y1="100" x2="0" y2="100" width="0" layer="20"/>
 <wire x1="0" y1="100" x2="0" y2="0" width="0" layer="20"/>
 <text x="2.286" y="87.63" size="1.778" layer="136">TOP</text>
@@
 <text x="15.748" y="25.146" size="1.1176" layer="21" font="vector">VCC</text>
 <text x="1.016" y="92.583" size="1.1176" layer="21" font="vector">M3_3MM</text>
-<text x="77.978" y="92.329" size="1.1176" layer="21" font="vector">M3_3MM</text>
+<text x="59.944" y="73.152" size="1.1176" layer="21" font="vector">M3_3MM</text>
 <polygon width="0.1524" layer="41">
 <vertex x="0.508" y="61.6712"/>
@@
 <attribute name="VALUE" x="20.193" y="47.879" size="0.0254" layer="27" rot="R180"/>
 </element>
-<element name="H1" library="holes" library_urn="urn:adsk.eagle:library:237" package="3,0" package3d_urn="urn:adsk.eagle:package:14277/1" value="MOUNT-HOLE3.0" x="80.899" y="95.758"/>
+<element name="H1" library="holes" library_urn="urn:adsk.eagle:library:237" package="3,0" package3d_urn="urn:adsk.eagle:package:14277/1" value="MOUNT-HOLE3.0" x="62.865" y="76.581"/>
 <element name="H3" library="holes" library_urn="urn:adsk.eagle:library:237" package="3,0" package3d_urn="urn:adsk.eagle:package:14277/1" value="MOUNT-HOLE3.0" x="4.0386" y="95.9612"/>
 <element name="GY_4-8" library="SparkFun-Connectors" library_urn="urn:adsk.eagle:library:513" package="1X04" package3d_urn="urn:adsk.eagle:package:38085/1" value="" x="20.193" y="43.307" smashed="yes" rot="R270">

Commit message: prototype board update
Parts:
- removed H2, H3: MOUNT-HOLE3.0, holes:3,0
- removed IRQ: LSP10, solpad:LSP10
- removed P_HIGH: (no value), pinhead_v2:1X01/OCT
- removed RAW-D13_1, RAW-D13_2, TX0-D12_1, TX0-D12_2: (no value), pinhead:1X15
- removed RAW_C: (no value), resistor:E3,5-8
- added B1: BREADBOARDMINI, SparkFun-Boards:BREADBOARD-MINI
- added J2: (no value), SparkFun-Connectors:1X02_LOCK
- added PH1, PH2: (no value), pinhead:2X15
- added U$1: LORA-RA-02-433MHZ, LikeCircuit:LORA-RA2-SMD
- ES32-433T20D: device con-lsta:FE07 -> SparkFun-Connectors:1X07_LOCK
- GY-521: device Seeed-Connector:H8-2.54 -> SparkFun-Connectors:1X08_LOCK
- GY_4-8: device SparkFun-Connectors:1X04 -> SparkFun-Connectors:1X04_LOCK
- J1: device SparkFun-Connectors:1X05 -> SparkFun-Connectors:1X05_LOCK
- R_SHIELD: device resistor:0204/5 -> rcl:0207/7
- moved T3_5MM 69.2 mm to (72.0, 26.0), turned to 0 degrees
- moved PIN3 63.3 mm to (64.4, 24.8), turned to 90 degrees
- moved H1 61.9 mm to (4.06, 95.9)
- moved T2_5MM 60.5 mm to (72.0, 36.8), turned to 0 degrees
- moved PIN2 52.5 mm to (64.4, 35.6), turned to 90 degrees
- moved VIN 51.8 mm to (70.1, 17.3)
- moved 3.3V 50.3 mm to (70.1, 12.4)
- moved 5V 48.8 mm to (70.1, 7.62)
- moved GND 47.3 mm to (70.1, 2.79)
- moved T1_5MM 44.0 mm to (48.5, 51.7)
- moved PIN1 44.0 mm to (49.8, 44.1)
- moved PIEZO 32.7 mm to (61.7, 49.1), turned to 180 degrees
- moved GY-521 13.0 mm to (8.13, 22.9), turned to 90 degrees
- moved 3.3V_C 11.4 mm to (18.8, 80.4), turned to 270 degrees
- moved D_B 11.1 mm to (17.8, 74.5)
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Connections:
- new net GND.3: U$1.9
- new net GND.4: U$1.16
- net 3.3V: now also PH1.3, PH1.4, U$1.3; no longer RAW-D13_1.2, RAW-D13_2.2
- net 5V: now also PH1.23, PH1.24; no longer RAW-D13_1.12, RAW-D13_2.12
- net A5: now also PH1.17, PH1.18; no longer RAW-D13_1.9, RAW-D13_2.9
- net A6: now also PH1.19, PH1.20; no longer RAW-D13_1.10, RAW-D13_2.10
- net A7: now also PH1.21, PH1.22; no longer RAW-D13_1.11, RAW-D13_2.11
- net CE_NRF: now also PH2.13, PH2.14; no longer TX0-D12_1.7, TX0-D12_2.7
- net CSN_NRF: now also PH2.15, PH2.16; no longer TX0-D12_1.8, TX0-D12_2.8
- net GND: now also PH1.27, PH1.28, RAW.GND@1; no longer RAW-D13_1.14, RAW-D13_2.14, RAW.GND@2, RAW_C.-
- net MISO_NRF: now also PH2.23, PH2.24; no longer TX0-D12_1.12, TX0-D12_2.12
- net MOSI_NRF: now also PH2.21, PH2.22; no longer TX0-D12_1.11, TX0-D12_2.11
- net N$1: now also U$1.1, U$1.2; no longer IRQ.MP, NRF24L01.8
- net N$16: now also PH2.1, PH2.2; no longer TX0-D12_1.1, TX0-D12_2.1
- net N$17: now also PH2.3, PH2.4; no longer TX0-D12_1.2, TX0-D12_2.2
- net N$18: now also PH2.5, PH2.6; no longer TX0-D12_1.3, TX0-D12_2.3
- net N$19: now also PH2.7, PH2.8; no longer TX0-D12_1.4, TX0-D12_2.4
- net N$20: now also PH2.10, PH2.9; no longer TX0-D12_1.5, TX0-D12_2.5
- net N$21: now also PH2.11, PH2.12; no longer TX0-D12_1.6, TX0-D12_2.6
- net N$24: now also PH2.17, PH2.18; no longer TX0-D12_1.9, TX0-D12_2.9
- net N$25: now also PH2.19, PH2.20; no longer TX0-D12_1.10, TX0-D12_2.10
- net N$28: now also PH2.25, PH2.26; no longer TX0-D12_1.13, TX0-D12_2.13
- net N$29: now also PH2.27, PH2.28; no longer TX0-D12_1.14, TX0-D12_2.14
- net N$3: now also PH1.5, PH1.6; no longer RAW-D13_1.3, RAW-D13_2.3
- net N$30: now also PH2.29, PH2.30; no longer TX0-D12_1.15, TX0-D12_2.15
- net N$34: now also J2.1, J2.2; no longer P_HIGH.1
- net N$4: now also PH1.7, PH1.8; no longer RAW-D13_1.4, RAW-D13_2.4
- net N$5: now also PH1.10, PH1.9; no longer RAW-D13_1.5, RAW-D13_2.5
- net N$6: now also PH1.11, PH1.12; no longer RAW-D13_1.6, RAW-D13_2.6
- net N$7: now also PH1.13, PH1.14; no longer RAW-D13_1.7, RAW-D13_2.7
- net RST: now also PH1.25, PH1.26; no longer RAW-D13_1.13, RAW-D13_2.13
- net SCK_NRF: now also PH1.1, PH1.2; no longer RAW-D13_1.1, RAW-D13_2.1
- net SDA_GY521: now also PH1.15, PH1.16; no longer RAW-D13_1.8, RAW-D13_2.8
- net VIN: now also PH1.29, PH1.30; no longer RAW-D13_1.15, RAW-D13_2.15, RAW_C.+
Routing:
- net 5V: track 326.9 -> 0.00 mm
- net 3.3V: track 311.1 -> 0.00 mm
- net VIN: track 147.6 -> 0.00 mm
- net SCK_NRF: track 90.6 -> 0.00 mm
- net SDA_GY521: track 83.6 -> 0.00 mm
- net MOSI_NRF: track 66.0 -> 0.00 mm
- net SHIELD_IN: track 63.7 -> 0.00 mm
- net CSN_NRF: track 58.8 -> 0.00 mm
- net A5: track 57.5 -> 0.00 mm
- net CE_NRF: track 56.5 -> 0.00 mm
- net MISO_NRF: track 33.8 -> 0.00 mm
- net N$5: track 20.5 -> 0.00 mm
- net A7: track 20.5 -> 0.00 mm
- net N$24: track 20.2 -> 0.00 mm
- net N$18: track 20.2 -> 0.00 mm
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