File: _PCB/_NANO prototype board/board.sch (EAGLE design)
At the start: 36 parts, among them T1_5MM 5mm, T2_5MM 5mm, T3_5MM 5mm

Commit message: prototype board optimization
Parts:
- removed BREAD_450: BREADBOARDMINI, SparkFun-Boards:BREADBOARDMINI
- added PIEZO: F/CM12P, buzzer:F/CM12P
- added P_HIGH: (no value), pinhead_v2:PINHD-1X1/OCT
- D_5PIN, D_B: device pinhead:PINHD-1X2 -> SparkFun-Connectors:CONN_02LOCK
Connections:
- removed net D+_B: D_B.1, USB_B.D+
- removed net D-_B: D_B.2, USB_B.D-
- new net N$34: PIEZO.1, P_HIGH.1
- new net N$35: D_B.1, USB_B.D-
- new net N$36: D_B.2, USB_B.D+
- net D+_5PIN: now also D_5PIN.2; no longer D_5PIN.1
- net D-_5PIN: now also D_5PIN.1; no longer D_5PIN.2
- net GND: now also PIEZO.2
Other:
- moved on the sheet: D_5PIN, D_B, H1, H2, H3

Commit message: prototype board update
Parts:
- removed H2, H3: MOUNT-HOLE3.0, holes:MOUNT-HOLE3.0
- removed IRQ: LSP10, solpad:LSP10
- removed P_HIGH: (no value), pinhead_v2:PINHD-1X1/OCT
- removed RAW-D13_1, RAW-D13_2, TX0-D12_1, TX0-D12_2: (no value), pinhead:PINHD-1X15
- removed RAW_C: (no value), resistor:CPOL-EUE3.5-8
- added B1: BREADBOARDMINI, SparkFun-Boards:BREADBOARDMINI
- added J2: (no value), SparkFun-Connectors:CONN_02LOCK
- added PH1, PH2: (no value), pinhead:PINHD-2X15
- added U$1: LORA-RA-02-433MHZ, LikeCircuit:LORA-RA-02-433MHZ
- ES32-433T20D: device con-lsta:FE07-1 -> SparkFun-Connectors:CONN_07LOCK
- GY-521: value DIP-BLACK-FEMALE-HEADER-VERT(8P-2.54) -> (none); device Seeed-Connector:DIP-BLACK-FEMALE-HEADER-VERT(8P-2.54) -> SparkFun-Connectors:CONN_08LOCK
- GY_4-8: device SparkFun-Connectors:CONN_04 -> SparkFun-Connectors:CONN_04LOCK
- J1: device SparkFun-Connectors:CONN_05 -> SparkFun-Connectors:CONN_05LOCK
- R_SHIELD: device resistor:R-US_0204/5 -> rcl:R-US_0207/7
Connections:
- net 3.3V: now also PH1.3, PH1.4; no longer RAW-D13_1.2, RAW-D13_2.2
- net 5V: now also PH1.23, PH1.24; no longer RAW-D13_1.12, RAW-D13_2.12
- net A5: now also PH1.17, PH1.18; no longer RAW-D13_1.9, RAW-D13_2.9
- net A6: now also PH1.19, PH1.20; no longer RAW-D13_1.10, RAW-D13_2.10
- net A7: now also PH1.21, PH1.22; no longer RAW-D13_1.11, RAW-D13_2.11
- net CE_NRF: now also PH2.13, PH2.14; no longer TX0-D12_1.7, TX0-D12_2.7
- net CSN_NRF: now also PH2.15, PH2.16; no longer TX0-D12_1.8, TX0-D12_2.8
- net GND: now also PH1.27, PH1.28, RAW.GNDBREAK; no longer RAW-D13_1.14, RAW-D13_2.14, RAW.GND, RAW_C.-
- net MISO_NRF: now also PH2.23, PH2.24; no longer TX0-D12_1.12, TX0-D12_2.12
- net MOSI_NRF: now also PH2.21, PH2.22; no longer TX0-D12_1.11, TX0-D12_2.11
- net N$1: now also U$1.GND.1, U$1.GND.2; no longer IRQ.MP, NRF24L01.8
- net N$16: now also PH2.1, PH2.2; no longer TX0-D12_1.1, TX0-D12_2.1
- net N$17: now also PH2.3, PH2.4; no longer TX0-D12_1.2, TX0-D12_2.2
- net N$18: now also PH2.5, PH2.6; no longer TX0-D12_1.3, TX0-D12_2.3
- net N$19: now also PH2.7, PH2.8; no longer TX0-D12_1.4, TX0-D12_2.4
- net N$20: now also PH2.10, PH2.9; no longer TX0-D12_1.5, TX0-D12_2.5
- net N$21: now also PH2.11, PH2.12; no longer TX0-D12_1.6, TX0-D12_2.6
- net N$24: now also PH2.17, PH2.18; no longer TX0-D12_1.9, TX0-D12_2.9
- net N$25: now also PH2.19, PH2.20; no longer TX0-D12_1.10, TX0-D12_2.10
- net N$28: now also PH2.25, PH2.26; no longer TX0-D12_1.13, TX0-D12_2.13
- net N$29: now also PH2.27, PH2.28; no longer TX0-D12_1.14, TX0-D12_2.14
- net N$3: now also PH1.5, PH1.6; no longer RAW-D13_1.3, RAW-D13_2.3
- net N$30: now also PH2.29, PH2.30; no longer TX0-D12_1.15, TX0-D12_2.15
- net N$34: now also J2.1, J2.2; no longer P_HIGH.1
- net N$4: now also PH1.7, PH1.8; no longer RAW-D13_1.4, RAW-D13_2.4
- net N$5: now also PH1.10, PH1.9; no longer RAW-D13_1.5, RAW-D13_2.5
- net N$6: now also PH1.11, PH1.12; no longer RAW-D13_1.6, RAW-D13_2.6
- net N$7: now also PH1.13, PH1.14; no longer RAW-D13_1.7, RAW-D13_2.7
- net RST: now also PH1.25, PH1.26; no longer RAW-D13_1.13, RAW-D13_2.13
- net SCK_NRF: now also PH1.1, PH1.2; no longer RAW-D13_1.1, RAW-D13_2.1
- net SDA_GY521: now also PH1.15, PH1.16; no longer RAW-D13_1.8, RAW-D13_2.8
- net VIN: now also PH1.29, PH1.30; no longer RAW-D13_1.15, RAW-D13_2.15, RAW_C.+
Other:
- moved on the sheet: 3.3/5, 3.3V_C, 5PIN1, 5PIN2, 5V, 5V_C, D_5PIN, D_B, ES32-433T20D, GND, H1, J1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
