File: _PCB/_pro mini prototype board/board.brd (EAGLE design)
At the start: 85.1 x 100 mm, 36 parts, among them T1_5MM 5mm, T2_5MM 5mm, T3_5MM 5mm

Commit message: checkpoint
Parts:
- removed RAW-D13_1, RAW-D13_2, TX0-D12_1, TX0-D12_2: (no value), pinhead:1X15
- removed U$1: ABK-PRO-MINI, Arduino-clone:ABK-PRO-MINI
- added D1: 1N4004, Seeed-Diode:DO-41
- added D1-D9_1, D1-D9_2, D13-RAW_1, D13-RAW_2: (no value), pinhead:1X12
- added PRO_MINI: (no value), SparkFun-Boards:ARDUINO_PRO_MINI
- moved BREAD_450 66.8 mm to (57.8, 64.6)
- moved 3.3V_C 3.92 mm to (30.1, 82.0)
- moved D_B 3.86 mm to (28.7, 72.1)
- moved R_SHIELD 3.68 mm to (22.0, 66.4), turned to 0 degrees
- moved 3.3V 3.00 mm to (77.5, 28.4)
- moved 5V 3.00 mm to (77.5, 22.1)
- moved GND 3.00 mm to (77.5, 15.7)
- moved VIN 3.00 mm to (77.5, 34.8)
- moved 5V_C 0.72 mm to (20.2, 78.1)
Connections:
- removed net N$28: TX0-D12_1.13, TX0-D12_2.13
- removed net N$29: TX0-D12_1.14, TX0-D12_2.14
- removed net N$30: TX0-D12_1.15, TX0-D12_2.15
- removed net RST: RAW-D13_1.13, RAW-D13_2.13
- net 3.3V: now also D1-D9_1.2, D1-D9_2.2, PRO_MINI.2; no longer RAW-D13_1.2, RAW-D13_2.2
- net 5V: now also D1-D9_1.12, D1-D9_2.12, PRO_MINI.12; no longer RAW-D13_1.12, RAW-D13_2.12
- net A5: now also D1-D9_1.9, D1-D9_2.9, PRO_MINI.9; no longer RAW-D13_1.9, RAW-D13_2.9
- net A6: now also D1-D9_1.10, D1-D9_2.10, PRO_MINI.10; no longer RAW-D13_1.10, RAW-D13_2.10
- net A7: now also D1-D9_1.11, D1-D9_2.11, PRO_MINI.11; no longer RAW-D13_1.11, RAW-D13_2.11
- net CE_NRF: now also D13-RAW_1.7, D13-RAW_2.7, PRO_MINI.18; no longer TX0-D12_1.7, TX0-D12_2.7
- net CSN_NRF: now also D13-RAW_1.8, D13-RAW_2.8, PRO_MINI.17; no longer TX0-D12_1.8, TX0-D12_2.8
- net GND: no longer RAW-D13_1.14, RAW-D13_2.14
- net MISO_NRF: now also D13-RAW_1.12, D13-RAW_2.12, PRO_MINI.13; no longer TX0-D12_1.12, TX0-D12_2.12
- net MOSI_NRF: now also D13-RAW_1.11, D13-RAW_2.11, PRO_MINI.14; no longer TX0-D12_1.11, TX0-D12_2.11
- net N$16: now also D13-RAW_1.1, D13-RAW_2.1, PRO_MINI.24; no longer TX0-D12_1.1, TX0-D12_2.1
- net N$17: now also D13-RAW_1.2, D13-RAW_2.2, PRO_MINI.23; no longer TX0-D12_1.2, TX0-D12_2.2
- net N$18: now also D13-RAW_1.3, D13-RAW_2.3, PRO_MINI.22; no longer TX0-D12_1.3, TX0-D12_2.3
- net N$19: now also D13-RAW_1.4, D13-RAW_2.4, PRO_MINI.21; no longer TX0-D12_1.4, TX0-D12_2.4
- net N$20: now also D13-RAW_1.5, D13-RAW_2.5, PRO_MINI.20; no longer TX0-D12_1.5, TX0-D12_2.5
- net N$21: now also D13-RAW_1.6, D13-RAW_2.6, PRO_MINI.19; no longer TX0-D12_1.6, TX0-D12_2.6
- net N$24: now also D13-RAW_1.9, D13-RAW_2.9, PRO_MINI.16; no longer TX0-D12_1.9, TX0-D12_2.9
- net N$25: now also D13-RAW_1.10, D13-RAW_2.10, PRO_MINI.15; no longer TX0-D12_1.10, TX0-D12_2.10
- net N$3: now also D1-D9_1.3, D1-D9_2.3, PRO_MINI.3; no longer RAW-D13_1.3, RAW-D13_2.3
- net N$4: now also D1-D9_1.4, D1-D9_2.4, PRO_MINI.4; no longer RAW-D13_1.4, RAW-D13_2.4
- net N$5: now also D1-D9_1.5, D1-D9_2.5, PRO_MINI.5; no longer RAW-D13_1.5, RAW-D13_2.5
- net N$6: now also D1-D9_1.6, D1-D9_2.6, PRO_MINI.6; no longer RAW-D13_1.6, RAW-D13_2.6
- net N$7: now also D1-D9_1.7, D1-D9_2.7, PRO_MINI.7; no longer RAW-D13_1.7, RAW-D13_2.7
- net SCK_NRF: now also D1-D9_1.1, D1-D9_2.1, PRO_MINI.1; no longer RAW-D13_1.1, RAW-D13_2.1
- net SDA_GY521: now also D1-D9_1.8, D1-D9_2.8, PRO_MINI.8; no longer RAW-D13_1.8, RAW-D13_2.8
- net VIN: no longer RAW-D13_1.15, RAW-D13_2.15
Routing:
- net 3.3V: track 167.4 -> 0.00 mm
- net 5V: track 97.9 -> 0.00 mm
- net SCK_NRF: track 90.8 -> 0.00 mm
- net VIN: track 89.6 -> 0.00 mm
- net SHIELD_IN: track 62.7 -> 0.00 mm
- net SDA_GY521: track 47.7 -> 0.00 mm
- net CSN_NRF: track 41.1 -> 0.00 mm
- net CE_NRF: track 41.0 -> 0.00 mm
- net A5: track 33.3 -> 0.00 mm
- net D+_5PIN: track 18.9 -> 0.00 mm
- net D+_B: track 14.6 -> 0.00 mm
- net N$5: track 13.3 -> 0.00 mm
- net A7: track 13.3 -> 0.00 mm
- net RST: track 13.2 -> 0.00 mm
- net N$7: track 13.2 -> 0.00 mm
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Other:
- board text added: "A0"
- board text added: "A1"
- board text added: "A2"
- board text added: "A3"
- board text added: "A6"
- board text added: "A7"
- board text added: "AREF"
- board text added: "D0_RX"
- board text added: "D10_SS"
- board text added: "D11_MOSI"
- board text added: "D12_MISO"
- board text added: "D1_TX"
- board text added: "D2_INT0"
- board text added: "D3_INT1"
- board text added: "D4"
- board text added: "D5"
- board text added: "D6"
- board text added: "D7"
- board text added: "D8"
- board text added: "D9"
- board text added: "I2C"
- board text added: "PWM"
- board text added: "PWM_SPI"
- board text added: "RST"
- board text added: "SCK_D13"
- board text added: "SCL_A5"
- board text added: "SDA_A4"
- board text added: "SPI"
- board text added: "SPI_LED"
- board text added: "VIN"
