File: _PCB/_pro mini prototype board/board.brd (EAGLE design)
At the start: 85.1 x 100 mm, 37 parts, among them T1_5MM 5mm, T2_5MM 5mm, T3_5MM 5mm

Commit message: library update
Parts:
- removed PRO_MINI: (no value), SparkFun-Boards:ARDUINO_PRO_MINI
- added U$1: ABK-PRO-MINI, Arduino-clone:ABK-PRO-MINI
Connections:
- new net N$28: U$1.A1
- new net N$29: U$1.D13
- net 3.3V: now also U$1.RX1; no longer PRO_MINI.2
- net 5V: now also U$1.D9; no longer PRO_MINI.12
- net A5: now also U$1.D6; no longer PRO_MINI.9
- net A6: now also U$1.D7; no longer PRO_MINI.10
- net A7: now also U$1.D8; no longer PRO_MINI.11
- net CE_NRF: no longer PRO_MINI.18
- net CSN_NRF: now also U$1.A0; no longer PRO_MINI.17
- net MISO_NRF: now also U$1.D10; no longer PRO_MINI.13
- net MOSI_NRF: now also U$1.D11; no longer PRO_MINI.14
- net N$16: now also U$1.RAW; no longer PRO_MINI.24
- net N$17: now also U$1.GND; no longer PRO_MINI.23
- net N$18: now also U$1.RST; no longer PRO_MINI.22
- net N$19: now also U$1.VCC; no longer PRO_MINI.21
- net N$20: now also U$1.A3; no longer PRO_MINI.20
- net N$21: now also U$1.A2; no longer PRO_MINI.19
- net N$24: no longer PRO_MINI.16
- net N$25: now also U$1.D12; no longer PRO_MINI.15
- net N$3: now also U$1.RST1; no longer PRO_MINI.3
- net N$4: now also U$1.GND1; no longer PRO_MINI.4
- net N$5: now also U$1.D2; no longer PRO_MINI.5
- net N$6: now also U$1.D3; no longer PRO_MINI.6
- net N$7: now also U$1.D4; no longer PRO_MINI.7
- net SCK_NRF: now also U$1.TX0; no longer PRO_MINI.1
- net SDA_GY521: now also U$1.D5; no longer PRO_MINI.8
Other:
- board text added: "A4_SDA"
- board text added: "A5_SCL"
- board text removed: "SCL_A5"
- board text removed: "SDA_A4"

Commit message: board update
Parts:
- moved D13-RAW_1 5.72 mm to (58.1, 16.9)
- moved D13-RAW_2 5.72 mm to (55.1, 16.9)
- moved U$1 5.09 mm to (36.6, 24.5)
- moved D1-D9_1 1.55 mm to (21.2, 16.9)
- moved D1-D9_2 1.55 mm to (24.2, 16.9)
Connections:
- removed net N$24: D13-RAW_1.9, D13-RAW_2.9
- removed net N$28: U$1.A1
- net CE_NRF: now also U$1.A2
- net CSN_NRF: now also U$1.A3; no longer U$1.A0
- net GND: now also U$1.GND2, U$1.GND3, U$1.GND4
- net N$20: now also U$1.A0; no longer U$1.A3
- net N$21: now also U$1.A1; no longer U$1.A2
- net N$29: now also D13-RAW_1.9, D13-RAW_2.9
Other:
- board text added: "40mA/PIN 20mA recomme 200mA-MAX 150mA-RAW"
- board text added: "D0"
- board text added: "D1"
- board text added: "D12"
- board text added: "D2"
- board text added: "D3_~"
- board text added: "D5_~"
- board text added: "D6_~"
- board text added: "D9_~"
- board text added: "DTR"
- board text added: "INT0"
- board text added: "INT1"
- board text added: "L_D13"
- board text added: "RX"
- board text added: "SCL_A5"
- board text added: "SDA_A4"
- board text added: "SS"
- board text added: "TX"
- board text added: "~_D10"
- board text added: "~_D11"
- board text removed: "A4_SDA"
- board text removed: "A5_SCL"
- board text removed: "AREF"
- board text removed: "D0_RX"
- board text removed: "D10_SS"
- board text removed: "D11_MOSI"
- board text removed: "D12_MISO"
- board text removed: "D1_TX"
- board text removed: "D2_INT0"
- board text removed: "D3_INT1"
- board text removed: "D5"
- board text removed: "D6"
- board text removed: "D9"
- board text removed: "I2C"
- board text removed: "PWM"
- board text removed: "PWM_SPI"
- board text removed: "SCK_D13"
- board text removed: "SPI"

Commit message: prototype board optimization
Parts:
- added J2: 2p-2.54, Seeed-Connector:H2-2.54
- added J3: 2p-2.0, Seeed-Connector:H2-2.0-6X4.5MM
- moved D1 47.7 mm to (23.1, 37.5)
Connections:
- new net N$28: D1.1, J2.2, J3.+
- net GND: now also J2.1, J3.-, RAW.GND@1
- net VIN: now also D1.2
Changed lines of the file:
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@@
 <attribute name="VALUE" x="51.917" y="32.169" size="1.27" layer="27" rot="R270"/>
 </element>
-<element name="D1" library="Seeed-Diode" library_urn="urn:adsk.eagle:library:467" package="DO-41" package3d_urn="urn:adsk.eagle:package:32521/1" value="1N4004" x="-24.097" y="44.108">
-<attribute name="MPN" value="1N4004" x="-24.097" y="44.108" size="1.778" layer="27" display="off"/>
+<element name="D1" library="Seeed-Diode" library_urn="urn:adsk.eagle:library:467" package="DO-41" package3d_urn="urn:adsk.eagle:package:32521/1" value="1N4004" x="23.147" y="37.504">
+<attribute name="MPN" value="1N4004" x="23.147" y="37.504" size="1.778" layer="27" display="off"/>
 </element>
 <element name="U$1" library="Arduino-clone" package="ABK-PRO-MINI" value="ABK-PRO-MINI" x="36.62" y="24.546"/>
+<element name="J2" library="Seeed-Connector" library_urn="urn:adsk.eagle:library:478" package="H2-2.54" package3d_urn="urn:adsk.eagle:package:33132/1" value="2p-2.54" x="31.369" y="45.212">
+<attribute name="MPN" value="P125-1102A0BS116A1" x="31.369" y="45.212" size="1.1176" layer="27" font="vector" display="off"/>
+</element>
+<element name="J3" library="Seeed-Connector" library_urn="urn:adsk.eagle:library:478" package="H2-2.0-6X4.5MM" package3d_urn="urn:adsk.eagle:package:33112/1" value="2p-2.0" x="24.511" y="44.196"/>
 </elements>
 <signals>
@@
 <contactref element="VIN" pad="2"/>
 <contactref element="RAW" pad="PWR"/>
+<contactref element="D1" pad="2"/>
 <wire x1="78.74" y1="34.75" x2="81.28" y2="34.75" width="0" layer="19" extent="1-1"/>
 <wire x1="76.2" y1="34.75" x2="78.74" y2="34.75" width="0" layer="19" extent="1-1"/>
 <wire x1="73.66" y1="34.75" x2="76.2" y2="34.75" width="0" layer="19" extent="1-1"/>
-<wire x1="19.685" y1="85.852" x2="73.66" y2="34.75" width="0" layer="19" extent="1-1"/>
+<wire x1="27.592" y1="37.504" x2="73.66" y2="34.75" width="0" layer="19" extent="1-1"/>
+<wire x1="19.685" y1="85.852" x2="27.592" y2="37.504" width="0" layer="19" extent="1-1"/>
 <wire x1="13.165" y1="88.225" x2="19.685" y2="85.852" width="0" layer="19" extent="1-1"/>
 </signal>
@@
 <contactref element="U$1" pad="GND3"/>
 <contactref element="U$1" pad="GND4"/>
+<contactref element="J2" pad="1"/>
+<contactref element="RAW" pad="GND@1"/>
+<contactref element="J3" pad="-"/>
 <wire x1="19.685" y1="89.408" x2="25.878" y2="93.795" width="0" layer="19" extent="1-1"/>
 <wire x1="13.178" y1="93.795" x2="19.685" y2="89.408" width="0" layer="19" extent="1-1"/>
@@
 <wire x1="46.78" y1="10.576" x2="55.092" y2="10.579" width="0" layer="19" extent="1-1"/>
 </signal>
+<signal name="N$28" class="1">
+<contactref element="J2" pad="2"/>
+<contactref element="D1" pad="1"/>
+<contactref element="J3" pad="+"/>
+<wire x1="23.511" y1="44.946" x2="31.369" y2="43.942" width="0" layer="19" extent="1-1"/>
+<wire x1="18.702" y1="37.504" x2="23.511" y2="44.946" width="0" layer="19" extent="1-1"/>
+</signal>
 </signals>

Commit message: PCB optimization
Parts:
- removed J3: 2p-2.0, Seeed-Connector:H2-2.0-6X4.5MM
- moved BREAD_450 74.1 mm to (131.3, 73.9)
- moved D1 42.5 mm to (29.1, 79.6), turned to 270 degrees
- moved J2 34.5 mm to (33.4, 79.6), turned to 180 degrees
- moved 3.3V_C 16.6 mm to (19.2, 69.6), turned to 90 degrees
- moved R_SHIELD 5.43 mm to (16.9, 64.5)
- moved GY-521 4.96 mm to (8.89, 35.4)
- moved GY_4-8 4.96 mm to (15.0, 44.3)
- moved H1 4.45 mm to (76.5, 95.8)
- moved H2 4.45 mm to (76.5, 4.19)
- moved T3_5MM 4.45 mm to (65.9, 95.2)
- moved PIN1 4.45 mm to (39.2, 87.6)
- moved PIN2 4.45 mm to (53.2, 87.6)
- moved T1_5MM 4.45 mm to (38.0, 95.2)
- moved T2_5MM 4.45 mm to (51.9, 95.2)
- moved 3.3V 4.44 mm to (73.0, 28.4)
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Connections:
- removed net N$28: D1.1, J2.2, J3.+
- new net N$24: D1.1, J2.2
- net GND: no longer J3.-, RAW.GND@1
Other:
- board size 85.1 x 100 mm -> 80.6 x 100 mm
- board text removed: "SPI_LED"

Commit message: PCB optimization
Parts:
- removed H1: MOUNT-HOLE3.0, holes:3,0
- moved 3.3V 32.5 mm to (53.7, 54.6)
- moved 5V 32.5 mm to (53.7, 48.2)
- moved GND 32.5 mm to (53.7, 41.9)
- moved VIN 32.5 mm to (53.7, 60.9)
- moved H2 8.13 mm to (68.3, 4.32)
Other:
- board size 80.6 x 100 mm -> 72.6 x 100 mm
Changed lines of the file:
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@@
 <fusionsync huburn="a.cGVyc29uYWw6dWUyYTRmMGNk" projecturn="a.cGVyc29uYWw6dWUyYTRmMGNkIzIwMTgwMTAyMTEwNTQ5ODMx" f3durn="urn:adsk.wipprod:dm.lineage:Bxu1HE7lTUeaXPtey1c6dw" pcbguid="eda9b9f7-04f8-461a-b123-4fdb15b2374b" lastpulledtime="" lastsyncedchangeguid="1f1fda12-eeed-9165-c6f5-a847dca60c4a"/>
 <plain>
-<wire x1="0" y1="0" x2="80.625" y2="0" width="0" layer="20"/>
-<wire x1="80.625" y1="0" x2="80.625" y2="100" width="0" layer="20"/>
-<wire x1="80.625" y1="100" x2="0" y2="100" width="0" layer="20"/>
+<wire x1="0" y1="0" x2="72.624" y2="0" width="0" layer="20"/>
+<wire x1="72.624" y1="0" x2="72.624" y2="100" width="0" layer="20"/>
+<wire x1="72.624" y1="100" x2="0" y2="100" width="0" layer="20"/>
 <wire x1="0" y1="100" x2="0" y2="0" width="0" layer="20"/>
 <text x="2.286" y="87.63" size="1.778" layer="136">TOP</text>
@@
 <text x="10.541" y="26.162" size="1.1176" layer="21" font="vector">VCC</text>
 <text x="7.493" y="93.218" size="1.1176" layer="21" font="vector" rot="R90">M3_3MM</text>
-<text x="74.676" y="93.091" size="1.1176" layer="21" font="vector" rot="R90">M3_3MM</text>
-<text x="79.502" y="1.524" size="1.1176" layer="21" font="vector" rot="R90">M3_3MM</text>
+<text x="71.374" y="1.651" size="1.1176" layer="21" font="vector" rot="R90">M3_3MM</text>
 <polygon width="0.1524" layer="41">
 <vertex x="0.508" y="61.6712"/>
@@
 </autorouter>
 <elements>
-<element name="3.3V" library="pinhead" library_urn="urn:adsk.eagle:library:325" package="1X04" package3d_urn="urn:adsk.eagle:package:22407/2" value="" x="73.025" y="28.4" smashed="yes" rot="R180">
-<attribute name="NAME" x="78.1812" y="26.5712" size="1.27" layer="25" ratio="10" rot="R180"/>
-<attribute name="VALUE" x="78.105" y="31.575" size="1.27" layer="27" rot="R180"/>
+<element name="3.3V" library="pinhead" library_urn="urn:adsk.eagle:library:325" package="1X04" package3d_urn="urn:adsk.eagle:package:22407/2" value="" x="53.721" y="54.562" smashed="yes" rot="R180">
+<attribute name="NAME" x="58.8772" y="52.7332" size="1.27" layer="25" ratio="10" rot="R180"/>
+<attribute name="VALUE" x="58.801" y="57.737" size="1.27" layer="27" rot="R180"/>
 </element>
 <element name="3.3V_C" library="rcl" library_urn="urn:adsk.eagle:library:334" package="E2,5-5" package3d_urn="urn:adsk.eagle:package:23344/1" value="" x="19.177" y="69.596" smashed="yes" rot="R90">
@@
 <attribute name="VALUE" x="21.59" y="72.009" size="1.27" layer="27" ratio="10" rot="R90"/>
 </element>
-<element name="5V" library="pinhead" library_urn="urn:adsk.eagle:library:325" package="1X04" package3d_urn="urn:adsk.eagle:package:22407/2" value="" x="73.025" y="22.05" smashed="yes" rot="R180">
-<attribute name="NAME" x="78.1812" y="20.2212" size="1.27" layer="25" ratio="10" rot="R180"/>
-<attribute name="VALUE" x="78.105" y="25.225" size="1.27" layer="27" rot="R180"/>
+<element name="5V" library="pinhead" library_urn="urn:adsk.eagle:library:325" package="1X04" package3d_urn="urn:adsk.eagle:package:22407/2" value="" x="53.721" y="48.212" smashed="yes" rot="R180">
+<attribute name="NAME" x="58.8772" y="46.3832" size="1.27" layer="25" ratio="10" rot="R180"/>
+<attribute name="VALUE" x="58.801" y="51.387" size="1.27" layer="27" rot="R180"/>
 </element>
 <element name="5V_C" library="resistor" library_urn="urn:adsk.eagle:library:348" package="E3,5-8" package3d_urn="urn:adsk.eagle:package:25842/1" value="" x="20.828" y="77.851" smashed="yes">
@@
 <attribute name="VALUE" x="6.858" y="2.667" size="1.27" layer="27" ratio="10" rot="R90"/>
 </element>
-<element name="GND" library="pinhead" library_urn="urn:adsk.eagle:library:325" package="1X04" package3d_urn="urn:adsk.eagle:package:22407/2" value="" x="73.025" y="15.7" smashed="yes" rot="R180">
-<attribute name="NAME" x="78.1812" y="13.8712" size="1.27" layer="25" ratio="10" rot="R180"/>
-<attribute name="VALUE" x="78.105" y="18.875" size="1.27" layer="27" rot="R180"/>
+<element name="GND" library="pinhead" library_urn="urn:adsk.eagle:library:325" package="1X04" package3d_urn="urn:adsk.eagle:package:22407/2" value="" x="53.721" y="41.862" smashed="yes" rot="R180">
+<attribute name="NAME" x="58.8772" y="40.0332" size="1.27" layer="25" ratio="10" rot="R180"/>
+<attribute name="VALUE" x="58.801" y="45.037" size="1.27" layer="27" rot="R180"/>
 </element>
 <element name="GY-521" library="Seeed-Connector" library_urn="urn:adsk.eagle:library:478" package="H8-2.54" package3d_urn="urn:adsk.eagle:package:33113/1" value="" x="8.89" y="35.433" smashed="yes" rot="R180">
@@
 <attribute name="VALUE" x="0.571" y="65.786" size="0.6096" layer="27" font="vector" ratio="20" align="top-left"/>
 </element>
-<element name="VIN" library="pinhead" library_urn="urn:adsk.eagle:library:325" package="1X04" package3d_urn="urn:adsk.eagle:package:22407/2" value="" x="73.025" y="34.75" smashed="yes" rot="R180">
-<attribute name="NAME" x="78.1812" y="32.9212" size="1.27" layer="25" ratio="10" rot="R180"/>
-<attribute name="VALUE" x="78.105" y="37.925" size="1.27" layer="27" rot="R180"/>
+<element name="VIN" library="pinhead" library_urn="urn:adsk.eagle:library:325" package="1X04" package3d_urn="urn:adsk.eagle:package:22407/2" value="" x="53.721" y="60.912" smashed="yes" rot="R180">
+<attribute name="NAME" x="58.8772" y="59.0832" size="1.27" layer="25" ratio="10" rot="R180"/>
+<attribute name="VALUE" x="58.801" y="64.087" size="1.27" layer="27" rot="R180"/>
 </element>
 <element name="5PIN1" library="SparkFun-Connectors" library_urn="urn:adsk.eagle:library:513" package="USB-B-MICRO-SMD" package3d_urn="urn:adsk.eagle:package:38238/1" value="" x="13.716" y="96.52" smashed="yes" rot="R270">
@@
 <attribute name="VALUE" x="20.193" y="47.879" size="0.0254" layer="27" rot="R180"/>
 </element>
-<element name="H1" library="holes" library_urn="urn:adsk.eagle:library:237" package="3,0" package3d_urn="urn:adsk.eagle:package:14277/1" value="MOUNT-HOLE3.0" x="76.454" y="95.758"/>
-<element name="H2" library="holes" library_urn="urn:adsk.eagle:library:237" package="3,0" package3d_urn="urn:adsk.eagle:package:14277/1" value="MOUNT-HOLE3.0" x="76.454" y="4.191"/>
+<element name="H2" library="holes" library_urn="urn:adsk.eagle:library:237" package="3,0" package3d_urn="urn:adsk.eagle:package:14277/1" value="MOUNT-HOLE3.0" x="68.326" y="4.318"/>
 <element name="H3" library="holes" library_urn="urn:adsk.eagle:library:237" package="3,0" package3d_urn="urn:adsk.eagle:package:14277/1" value="MOUNT-HOLE3.0" x="4.0386" y="95.9612"/>
 <element name="GY_4-8" library="SparkFun-Connectors" library_urn="urn:adsk.eagle:library:513" package="1X04" package3d_urn="urn:adsk.eagle:package:38085/1" value="" x="14.986" y="44.323" smashed="yes" rot="R270">
@@
 <contactref element="RAW" pad="PWR"/>
 <contactref element="D1" pad="2"/>
-<wire x1="74.295" y1="34.75" x2="76.835" y2="34.75" width="0" layer="19" extent="1-1"/>
-<wire x1="71.755" y1="34.75" x2="74.295" y2="34.75" width="0" layer="19" extent="1-1"/>
-<wire x1="69.215" y1="34.75" x2="71.755" y2="34.75" width="0" layer="19" extent="1-1"/>
-<wire x1="29.122" y1="75.151" x2="69.215" y2="34.75" width="0" layer="19" extent="1-1"/>
+<wire x1="54.991" y1="60.912" x2="57.531" y2="60.912" width="0" layer="19" extent="1-1"/>
+<wire x1="52.451" y1="60.912" x2="54.991" y2="60.912" width="0" layer="19" extent="1-1"/>
+<wire x1="49.911" y1="60.912" x2="52.451" y2="60.912" width="0" layer="19" extent="1-1"/>
+<wire x1="29.122" y1="75.151" x2="49.911" y2="60.912" width="0" layer="19" extent="1-1"/>
 <wire x1="18.415" y1="87.249" x2="29.122" y2="75.151" width="0" layer="19" extent="1-1"/>
 <wire x1="13.165" y1="88.225" x2="18.415" y2="87.249" width="0" layer="19" extent="1-1"/>
@@
 <contactref element="D1-D9_2" pad="2"/>
 <contactref element="U$1" pad="RX1"/>
-<wire x1="74.295" y1="28.4" x2="76.835" y2="28.4" width="0" layer="19" extent="1-1"/>
-<wire x1="71.755" y1="28.4" x2="74.295" y2="28.4" width="0" layer="19" extent="1-1"/>
-<wire x1="69.215" y1="28.4" x2="71.755" y2="28.4" width="0" layer="19" extent="1-1"/>
-<wire x1="31.54" y1="28.356" x2="69.215" y2="28.4" width="0" layer="19" extent="1-1"/>
+<wire x1="54.991" y1="54.562" x2="57.531" y2="54.562" width="0" layer="19" extent="1-1"/>
+<wire x1="52.451" y1="54.562" x2="54.991" y2="54.562" width="0" layer="19" extent="1-1"/>
+<wire x1="49.911" y1="54.562" x2="52.451" y2="54.562" width="0" layer="19" extent="1-1"/>
+<wire x1="31.54" y1="28.356" x2="49.911" y2="54.562" width="0" layer="19" extent="1-1"/>
 <wire x1="24.205" y1="28.359" x2="31.54" y2="28.356" width="0" layer="19" extent="1-1"/>
 <wire x1="21.166" y1="28.359" x2="24.205" y2="28.359" width="0" layer="19" extent="1-1"/>
@@
 <wire x1="24.205" y1="2.959" x2="21.166" y2="2.959" width="0" layer="19" extent="1-1"/>
 <wire x1="31.54" y1="2.956" x2="24.205" y2="2.959" width="0" layer="19" extent="1-1"/>
-<wire x1="69.215" y1="22.05" x2="31.54" y2="2.956" width="0" layer="19" extent="1-1"/>
-<wire x1="71.755" y1="22.05" x2="69.215" y2="22.05" width="0" layer="19" extent="1-1"/>
-<wire x1="74.295" y1="22.05" x2="71.755" y2="22.05" width="0" layer="19" extent="1-1"/>
-<wire x1="76.835" y1="22.05" x2="74.295" y2="22.05" width="0" layer="19" extent="1-1"/>
+<wire x1="49.911" y1="48.212" x2="31.54" y2="2.956" width="0" layer="19" extent="1-1"/>
+<wire x1="52.451" y1="48.212" x2="49.911" y2="48.212" width="0" layer="19" extent="1-1"/>
+<wire x1="54.991" y1="48.212" x2="52.451" y2="48.212" width="0" layer="19" extent="1-1"/>
+<wire x1="57.531" y1="48.212" x2="54.991" y2="48.212" width="0" layer="19" extent="1-1"/>
 </signal>
 <signal name="GND" class="1">
