File: _PCB/_pro mini prototype board/board.sch (EAGLE design)
At the start: 37 parts, among them T1_5MM 5mm, T2_5MM 5mm, T3_5MM 5mm

Commit message: library update
Parts:
- removed PRO_MINI: ARDUINO_PRO_MINI, SparkFun-Boards:ARDUINO_PRO_MINI
- added U$1: ABK-PRO-MINI, Arduino-clone:ABK-PRO-MINI
Connections:
- new net N$28: U$1.A1
- new net N$29: U$1.D13
- net 3.3V: now also U$1.RX1; no longer PRO_MINI.RXI
- net 5V: now also U$1.D9; no longer PRO_MINI.*9
- net A5: now also U$1.D6; no longer PRO_MINI.*6
- net A6: now also U$1.D7; no longer PRO_MINI.7
- net A7: now also U$1.D8; no longer PRO_MINI.8
- net CE_NRF: no longer PRO_MINI.A1
- net CSN_NRF: now also U$1.A0; no longer PRO_MINI.A0
- net MISO_NRF: now also U$1.D10; no longer PRO_MINI.*10
- net MOSI_NRF: now also U$1.D11; no longer PRO_MINI.*11
- net N$16: now also U$1.RAW; no longer PRO_MINI.RAW
- net N$17: now also U$1.GND; no longer PRO_MINI.GND@2
- net N$18: now also U$1.RST; no longer PRO_MINI.RST@2
- net N$19: now also U$1.VCC; no longer PRO_MINI.VCC
- net N$20: now also U$1.A3; no longer PRO_MINI.A3
- net N$21: now also U$1.A2; no longer PRO_MINI.A2
- net N$24: no longer PRO_MINI.13
- net N$25: now also U$1.D12; no longer PRO_MINI.12
- net N$3: now also U$1.RST1; no longer PRO_MINI.RST
- net N$4: now also U$1.GND2; no longer PRO_MINI.GND
- net N$5: now also U$1.D2; no longer PRO_MINI.2
- net N$6: now also U$1.D3; no longer PRO_MINI.*3
- net N$7: now also U$1.D4; no longer PRO_MINI.4
- net SCK_NRF: now also U$1.TX0; no longer PRO_MINI.TXO
- net SDA_GY521: now also U$1.D5; no longer PRO_MINI.*5
Other:
- moved on the sheet: D1-D9_1, D1-D9_2, D13-RAW_1, D13-RAW_2

Commit message: board update
Connections:
- removed net N$24: D13-RAW_1.9, D13-RAW_2.9
- removed net N$28: U$1.A1
- net CE_NRF: now also U$1.A2
- net CSN_NRF: now also U$1.A3; no longer U$1.A0
- net GND: now also U$1.GND1, U$1.GND3, U$1.GND4
- net N$20: now also U$1.A0; no longer U$1.A3
- net N$21: now also U$1.A1; no longer U$1.A2
- net N$29: now also D13-RAW_1.9, D13-RAW_2.9
Changed lines of the file:
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@@
 <part name="D1" library="Seeed-Diode" library_urn="urn:adsk.eagle:library:467" deviceset="DIP-DIODE-400V-1A(DO-41)" device="" package3d_urn="urn:adsk.eagle:package:32521/1" value="1N4004"/>
 <part name="U$1" library="Arduino-clone" deviceset="ABK-PRO-MINI" device=""/>
+<part name="GND1" library="SparkFun-PowerSymbols" library_urn="urn:adsk.eagle:library:530" deviceset="GND" device=""/>
+<part name="GND4" library="SparkFun-PowerSymbols" library_urn="urn:adsk.eagle:library:530" deviceset="GND" device=""/>
 </parts>
 <sheets>
@@
 <instance part="D1" gate="G$1" x="-88.9" y="-53.34"/>
 <instance part="U$1" gate="G$1" x="0" y="7.62"/>
+<instance part="GND1" gate="1" x="-5.08" y="-22.86"/>
+<instance part="GND4" gate="1" x="-17.78" y="35.56"/>
 </instances>
 <busses>
@@
 <wire x1="50.8" y1="10.16" x2="30.48" y2="10.16" width="0.1524" layer="91"/>
 <pinref part="D13-RAW_1" gate="G$1" pin="5"/>
+<pinref part="D13-RAW_2" gate="G$1" pin="5"/>
+<pinref part="U$1" gate="G$1" pin="A0"/>
+<wire x1="15.24" y1="2.54" x2="22.86" y2="2.54" width="0.1524" layer="91"/>
+<wire x1="22.86" y1="2.54" x2="30.48" y2="10.16" width="0.1524" layer="91"/>
 <junction x="30.48" y="10.16"/>
-<wire x1="15.24" y1="10.16" x2="25.4" y2="10.16" width="0.1524" layer="91"/>
-<wire x1="30.48" y1="10.16" x2="15.24" y2="10.16" width="0.1524" layer="91"/>
-<pinref part="D13-RAW_2" gate="G$1" pin="5"/>
-<pinref part="U$1" gate="G$1" pin="A3"/>
-<wire x1="15.24" y1="10.16" x2="20.32" y2="10.16" width="0.1524" layer="91"/>
 </segment>
 </net>
@@
 <wire x1="50.8" y1="7.62" x2="30.48" y2="7.62" width="0.1524" layer="91"/>
 <pinref part="D13-RAW_1" gate="G$1" pin="6"/>
+<pinref part="D13-RAW_2" gate="G$1" pin="6"/>
+<pinref part="U$1" gate="G$1" pin="A1"/>
+<wire x1="15.24" y1="5.08" x2="27.94" y2="5.08" width="0.1524" layer="91"/>
+<wire x1="27.94" y1="5.08" x2="30.48" y2="7.62" width="0.1524" layer="91"/>
 <junction x="30.48" y="7.62"/>
-<wire x1="15.24" y1="7.62" x2="25.4" y2="7.62" width="0.1524" layer="91"/>
-<wire x1="30.48" y1="7.62" x2="15.24" y2="7.62" width="0.1524" layer="91"/>
-<pinref part="D13-RAW_2" gate="G$1" pin="6"/>
-<pinref part="U$1" gate="G$1" pin="A2"/>
-<wire x1="15.24" y1="7.62" x2="20.32" y2="7.62" width="0.1524" layer="91"/>
 </segment>
 </net>
@@
 <pinref part="D13-RAW_2" gate="G$1" pin="7"/>
 <junction x="50.8" y="5.08"/>
+<pinref part="U$1" gate="G$1" pin="A2"/>
+<wire x1="15.24" y1="7.62" x2="27.94" y2="7.62" width="0.1524" layer="91"/>
+<wire x1="27.94" y1="7.62" x2="30.48" y2="5.08" width="0.1524" layer="91"/>
+<junction x="30.48" y="5.08"/>
 </segment>
 </net>
@@
 <segment>
 <pinref part="NRF24L01" gate="G$1" pin="4"/>
-<wire x1="15.24" y1="2.54" x2="25.4" y2="2.54" width="0.1524" layer="91"/>
 <wire x1="77.47" y1="-31.75" x2="88.9" y2="-31.75" width="0.1524" layer="91"/>
 <wire x1="88.9" y1="-31.75" x2="88.9" y2="2.54" width="0.1524" layer="91"/>
 <wire x1="88.9" y1="2.54" x2="50.8" y2="2.54" width="0.1524" layer="91"/>
 <pinref part="D13-RAW_1" gate="G$1" pin="8"/>
-<junction x="30.48" y="2.54"/>
 <wire x1="50.8" y1="2.54" x2="30.48" y2="2.54" width="0.1524" layer="91"/>
-<wire x1="30.48" y1="2.54" x2="15.24" y2="2.54" width="0.1524" layer="91"/>
 <pinref part="D13-RAW_2" gate="G$1" pin="8"/>
 <junction x="50.8" y="2.54"/>
-<pinref part="U$1" gate="G$1" pin="A0"/>
-</segment>
-</net>
-<net name="N$24" class="0">
-<segment>
-<wire x1="50.8" y1="0" x2="30.48" y2="0" width="0.1524" layer="91"/>
-<pinref part="D13-RAW_1" gate="G$1" pin="9"/>
-<pinref part="D13-RAW_2" gate="G$1" pin="9"/>
+<pinref part="U$1" gate="G$1" pin="A3"/>
+<wire x1="15.24" y1="10.16" x2="22.86" y2="10.16" width="0.1524" layer="91"/>
+<wire x1="22.86" y1="10.16" x2="30.48" y2="2.54" width="0.1524" layer="91"/>
+<junction x="30.48" y="2.54"/>
 </segment>
 </net>
@@
 <pinref part="U$1" gate="G$1" pin="D10"/>
 <wire x1="15.24" y1="-7.62" x2="20.32" y2="-7.62" width="0.1524" layer="91"/>
-<junction x="15.24" y="-7.62"/>
 </segment>
 </net>
@@
 <wire x1="100.33" y1="19.05" x2="107.95" y2="19.05" width="0.1524" layer="91"/>
 </segment>
+<segment>
+<pinref part="GND4" gate="1" pin="GND"/>
+<wire x1="-17.78" y1="38.1" x2="-17.78" y2="40.64" width="0.1524" layer="91"/>
+<wire x1="-17.78" y1="40.64" x2="-10.16" y2="40.64" width="0.1524" layer="91"/>
+<pinref part="U$1" gate="G$1" pin="GND3"/>
+<wire x1="-10.16" y1="40.64" x2="-10.16" y2="35.56" width="0.1524" layer="91"/>
+<pinref part="U$1" gate="G$1" pin="GND4"/>
+<wire x1="-10.16" y1="35.56" x2="-7.62" y2="35.56" width="0.1524" layer="91"/>
+<junction x="-10.16" y="35.56"/>
+</segment>
+<segment>
+<pinref part="U$1" gate="G$1" pin="GND1"/>
+<pinref part="GND1" gate="1" pin="GND"/>
+<wire x1="-5.08" y1="-17.78" x2="-5.08" y2="-20.32" width="0.1524" layer="91"/>
+</segment>
 </net>
 <net name="SHIELD_IN" class="1">
@@
 </segment>
 </net>
-<net name="N$28" class="0">
-<segment>
-<wire x1="15.24" y1="5.08" x2="25.4" y2="5.08" width="0.1524" layer="91"/>
-<pinref part="U$1" gate="G$1" pin="A1"/>
-</segment>
-</net>
 <net name="N$29" class="0">
 <segment>
 <wire x1="15.24" y1="0" x2="25.4" y2="0" width="0.1524" layer="91"/>
 <pinref part="U$1" gate="G$1" pin="D13"/>
-</segment>
-</net>
+<wire x1="50.8" y1="0" x2="30.48" y2="0" width="0.1524" layer="91"/>
+<pinref part="D13-RAW_1" gate="G$1" pin="9"/>
+<pinref part="D13-RAW_2" gate="G$1" pin="9"/>
+<wire x1="25.4" y1="0" x2="30.48" y2="0" width="0.1524" layer="91"/>
+<junction x="30.48" y="0"/>
+</segment>
+</net>

Commit message: prototype board optimization
Parts:
- added J2: 2p-2.54, Seeed-Connector:DIP-BLACK-MALE-HEADER-VERT(2P-2.54)
- added J3: 2p-2.0, Seeed-Connector:DIP-JST-2P-2.0
Connections:
- new net N$28: D1.+, J2.2, J3.P$1
- net GND: now also J2.1, J3.P$2, RAW.GNDBREAK
- net VIN: now also D1.-
Other:
- moved on the sheet: D1
Changed lines of the file:
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@@
 <setting verticaltext="up"/>
 </settings>
-<grid distance="0.1" unitdist="inch" unit="inch" style="lines" multiple="1" display="no" altdistance="0.01" altunitdist="inch" altunit="inch"/>
+<grid distance="0.05" unitdist="inch" unit="inch" style="lines" multiple="1" display="no" altdistance="0.01" altunitdist="inch" altunit="inch"/>
 <layers>
 <layer number="1" name="Top" color="4" fill="1" visible="no" active="no"/>
@@
 <part name="GND1" library="SparkFun-PowerSymbols" library_urn="urn:adsk.eagle:library:530" deviceset="GND" device=""/>
 <part name="GND4" library="SparkFun-PowerSymbols" library_urn="urn:adsk.eagle:library:530" deviceset="GND" device=""/>
+<part name="J2" library="Seeed-Connector" library_urn="urn:adsk.eagle:library:478" deviceset="DIP-BLACK-MALE-HEADER-VERT(2P-2.54)" device="" package3d_urn="urn:adsk.eagle:package:33132/1" value="2p-2.54"/>
+<part name="J3" library="Seeed-Connector" library_urn="urn:adsk.eagle:library:478" deviceset="DIP-JST-2P-2.0" device="" package3d_urn="urn:adsk.eagle:package:33112/1" value="2p-2.0"/>
 </parts>
 <sheets>
@@
 <instance part="D13-RAW_1" gate="G$1" x="33.02" y="7.62"/>
 <instance part="D13-RAW_2" gate="G$1" x="53.34" y="7.62"/>
-<instance part="D1" gate="G$1" x="-88.9" y="-53.34"/>
+<instance part="D1" gate="G$1" x="-93.98" y="-53.34" rot="R90"/>
 <instance part="U$1" gate="G$1" x="0" y="7.62"/>
 <instance part="GND1" gate="1" x="-5.08" y="-22.86"/>
 <instance part="GND4" gate="1" x="-17.78" y="35.56"/>
+<instance part="J2" gate="G$1" x="-73.66" y="-58.42"/>
+<instance part="J3" gate="G$1" x="-78.74" y="-71.12"/>
 </instances>
 <busses>
@@
 <label x="-158.75" y="-53.34" size="1.778" layer="95"/>
 <pinref part="RAW" gate="G$1" pin="PWR"/>
-<wire x1="-85.09" y1="-45.72" x2="-100.33" y2="-45.72" width="0.1524" layer="91"/>
+<wire x1="-85.09" y1="-45.72" x2="-88.9" y2="-45.72" width="0.1524" layer="91"/>
+<wire x1="-88.9" y1="-45.72" x2="-93.98" y2="-45.72" width="0.1524" layer="91"/>
+<wire x1="-93.98" y1="-45.72" x2="-100.33" y2="-45.72" width="0.1524" layer="91"/>
 <wire x1="-100.33" y1="-45.72" x2="-100.33" y2="-25.4" width="0.1524" layer="91"/>
 <wire x1="-100.33" y1="-25.4" x2="-60.96" y2="-25.4" width="0.1524" layer="91"/>
 <junction x="-100.33" y="-25.4"/>
+<pinref part="D1" gate="G$1" pin="-"/>
+<wire x1="-93.98" y1="-49.53" x2="-93.98" y2="-45.72" width="0.1524" layer="91"/>
+<junction x="-93.98" y="-45.72"/>
 </segment>
 </net>
@@
 <wire x1="-175.26" y1="52.07" x2="-149.86" y2="52.07" width="0.1524" layer="91"/>
 <junction x="-149.86" y="52.07"/>
+<pinref part="J2" gate="G$1" pin="1"/>
+<wire x1="-81.28" y1="-55.88" x2="-85.09" y2="-52.07" width="0.1524" layer="91"/>
+<wire x1="-85.09" y1="-52.07" x2="-85.09" y2="-51.816" width="0.1524" layer="91"/>
+<junction x="-85.09" y="-40.64"/>
+<pinref part="RAW" gate="G$1" pin="GNDBREAK"/>
+<wire x1="-85.09" y1="-51.816" x2="-85.09" y2="-43.18" width="0.1524" layer="91"/>
+<wire x1="-85.09" y1="-43.18" x2="-85.09" y2="-40.64" width="0.1524" layer="91"/>
+<junction x="-85.09" y="-43.18"/>
+<pinref part="J3" gate="G$1" pin="P$2"/>
+<wire x1="-81.28" y1="-72.39" x2="-85.09" y2="-68.58" width="0.1524" layer="91"/>
+<wire x1="-85.09" y1="-68.58" x2="-85.09" y2="-51.816" width="0.1524" layer="91"/>
+<junction x="-85.09" y="-51.816"/>
 </segment>
 <segment>
@@
 </segment>
 </net>
+<net name="N$28" class="1">
+<segment>
+<pinref part="J2" gate="G$1" pin="2"/>
+<pinref part="D1" gate="G$1" pin="+"/>
+<wire x1="-93.98" y1="-57.15" x2="-90.17" y2="-60.96" width="0.1524" layer="91"/>
+<wire x1="-90.17" y1="-60.96" x2="-89.916" y2="-60.96" width="0.1524" layer="91"/>
+<pinref part="J3" gate="G$1" pin="P$1"/>
+<wire x1="-89.916" y1="-60.96" x2="-81.28" y2="-60.96" width="0.1524" layer="91"/>
+<wire x1="-81.28" y1="-69.85" x2="-89.916" y2="-61.214" width="0.1524" layer="91"/>
+<wire x1="-89.916" y1="-61.214" x2="-89.916" y2="-60.96" width="0.1524" layer="91"/>
+<junction x="-89.916" y="-60.96"/>
+</segment>
+</net>

Commit message: PCB optimization
Parts:
- removed J3: 2p-2.0, Seeed-Connector:DIP-JST-2P-2.0
Connections:
- removed net N$28: D1.+, J2.2, J3.P$1
- new net N$24: D1.+, J2.2
- net GND: no longer J3.P$2, RAW.GNDBREAK
Other:
- moved on the sheet: D1, J2
Changed lines of the file:
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@@
 <part name="GND4" library="SparkFun-PowerSymbols" library_urn="urn:adsk.eagle:library:530" deviceset="GND" device=""/>
 <part name="J2" library="Seeed-Connector" library_urn="urn:adsk.eagle:library:478" deviceset="DIP-BLACK-MALE-HEADER-VERT(2P-2.54)" device="" package3d_urn="urn:adsk.eagle:package:33132/1" value="2p-2.54"/>
-<part name="J3" library="Seeed-Connector" library_urn="urn:adsk.eagle:library:478" deviceset="DIP-JST-2P-2.0" device="" package3d_urn="urn:adsk.eagle:package:33112/1" value="2p-2.0"/>
 </parts>
 <sheets>
@@
 <instance part="D13-RAW_1" gate="G$1" x="33.02" y="7.62"/>
 <instance part="D13-RAW_2" gate="G$1" x="53.34" y="7.62"/>
-<instance part="D1" gate="G$1" x="-93.98" y="-53.34" rot="R90"/>
+<instance part="D1" gate="G$1" x="-92.71" y="-58.42" rot="R90"/>
 <instance part="U$1" gate="G$1" x="0" y="7.62"/>
 <instance part="GND1" gate="1" x="-5.08" y="-22.86"/>
 <instance part="GND4" gate="1" x="-17.78" y="35.56"/>
-<instance part="J2" gate="G$1" x="-73.66" y="-58.42"/>
-<instance part="J3" gate="G$1" x="-78.74" y="-71.12"/>
+<instance part="J2" gate="G$1" x="-72.39" y="-63.5"/>
 </instances>
 <busses>
@@
 <label x="-158.75" y="-53.34" size="1.778" layer="95"/>
 <pinref part="RAW" gate="G$1" pin="PWR"/>
-<wire x1="-85.09" y1="-45.72" x2="-88.9" y2="-45.72" width="0.1524" layer="91"/>
-<wire x1="-88.9" y1="-45.72" x2="-93.98" y2="-45.72" width="0.1524" layer="91"/>
-<wire x1="-93.98" y1="-45.72" x2="-100.33" y2="-45.72" width="0.1524" layer="91"/>
+<wire x1="-85.09" y1="-45.72" x2="-92.71" y2="-45.72" width="0.1524" layer="91"/>
+<wire x1="-92.71" y1="-45.72" x2="-100.33" y2="-45.72" width="0.1524" layer="91"/>
 <wire x1="-100.33" y1="-45.72" x2="-100.33" y2="-25.4" width="0.1524" layer="91"/>
 <wire x1="-100.33" y1="-25.4" x2="-60.96" y2="-25.4" width="0.1524" layer="91"/>
 <junction x="-100.33" y="-25.4"/>
 <pinref part="D1" gate="G$1" pin="-"/>
-<wire x1="-93.98" y1="-49.53" x2="-93.98" y2="-45.72" width="0.1524" layer="91"/>
-<junction x="-93.98" y="-45.72"/>
+<wire x1="-92.71" y1="-54.61" x2="-92.71" y2="-45.72" width="0.1524" layer="91"/>
+<junction x="-92.71" y="-45.72"/>
 </segment>
 </net>
@@
 <junction x="-95.25" y="-15.24"/>
 <pinref part="RAW" gate="G$1" pin="GND"/>
-<wire x1="-85.09" y1="-40.64" x2="-95.25" y2="-40.64" width="0.1524" layer="91"/>
+<wire x1="-85.09" y1="-40.64" x2="-87.63" y2="-40.64" width="0.1524" layer="91"/>
+<wire x1="-87.63" y1="-40.64" x2="-95.25" y2="-40.64" width="0.1524" layer="91"/>
 <wire x1="-95.25" y1="-40.64" x2="-95.25" y2="-15.24" width="0.1524" layer="91"/>
 <pinref part="USB_B" gate="G$1" pin="GND"/>
@@
 <junction x="-149.86" y="52.07"/>
 <pinref part="J2" gate="G$1" pin="1"/>
-<wire x1="-81.28" y1="-55.88" x2="-85.09" y2="-52.07" width="0.1524" layer="91"/>
-<wire x1="-85.09" y1="-52.07" x2="-85.09" y2="-51.816" width="0.1524" layer="91"/>
-<junction x="-85.09" y="-40.64"/>
-<pinref part="RAW" gate="G$1" pin="GNDBREAK"/>
-<wire x1="-85.09" y1="-51.816" x2="-85.09" y2="-43.18" width="0.1524" layer="91"/>
-<wire x1="-85.09" y1="-43.18" x2="-85.09" y2="-40.64" width="0.1524" layer="91"/>
-<junction x="-85.09" y="-43.18"/>
-<pinref part="J3" gate="G$1" pin="P$2"/>
-<wire x1="-81.28" y1="-72.39" x2="-85.09" y2="-68.58" width="0.1524" layer="91"/>
-<wire x1="-85.09" y1="-68.58" x2="-85.09" y2="-51.816" width="0.1524" layer="91"/>
-<junction x="-85.09" y="-51.816"/>
+<wire x1="-80.01" y1="-60.96" x2="-87.63" y2="-53.34" width="0.1524" layer="91"/>
+<wire x1="-87.63" y1="-53.34" x2="-87.63" y2="-40.64" width="0.1524" layer="91"/>
+<junction x="-87.63" y="-40.64"/>
 </segment>
 <segment>
@@
 </segment>
 </net>
-<net name="N$28" class="1">
-<segment>
+<net name="N$24" class="0">
+<segment>
+<pinref part="D1" gate="G$1" pin="+"/>
 <pinref part="J2" gate="G$1" pin="2"/>
-<pinref part="D1" gate="G$1" pin="+"/>
-<wire x1="-93.98" y1="-57.15" x2="-90.17" y2="-60.96" width="0.1524" layer="91"/>
-<wire x1="-90.17" y1="-60.96" x2="-89.916" y2="-60.96" width="0.1524" layer="91"/>
-<pinref part="J3" gate="G$1" pin="P$1"/>
-<wire x1="-89.916" y1="-60.96" x2="-81.28" y2="-60.96" width="0.1524" layer="91"/>
-<wire x1="-81.28" y1="-69.85" x2="-89.916" y2="-61.214" width="0.1524" layer="91"/>
-<wire x1="-89.916" y1="-61.214" x2="-89.916" y2="-60.96" width="0.1524" layer="91"/>
-<junction x="-89.916" y="-60.96"/>
-</segment>
-</net>
+<wire x1="-92.71" y1="-62.23" x2="-88.9" y2="-66.04" width="0.1524" layer="91"/>
+<wire x1="-88.9" y1="-66.04" x2="-80.01" y2="-66.04" width="0.1524" layer="91"/>
+</segment>
+</net>

Commit message: PCB optimization
Parts:
- removed H1: MOUNT-HOLE3.0, holes:MOUNT-HOLE3.0
Changed lines of the file:
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@@
 <part name="BREAD_450" library="SparkFun-Boards" library_urn="urn:adsk.eagle:library:509" deviceset="BREADBOARD" device="MINI" package3d_urn="urn:adsk.eagle:package:37314/1"/>
 <part name="IRQ" library="solpad" library_urn="urn:adsk.eagle:library:364" deviceset="LSP10" device="" package3d_urn="urn:adsk.eagle:package:26501/1"/>
-<part name="H1" library="holes" library_urn="urn:adsk.eagle:library:237" deviceset="MOUNT-HOLE" device="3.0" package3d_urn="urn:adsk.eagle:package:14277/1"/>
 <part name="H2" library="holes" library_urn="urn:adsk.eagle:library:237" deviceset="MOUNT-HOLE" device="3.0" package3d_urn="urn:adsk.eagle:package:14277/1"/>
 <part name="H3" library="holes" library_urn="urn:adsk.eagle:library:237" deviceset="MOUNT-HOLE" device="3.0" package3d_urn="urn:adsk.eagle:package:14277/1"/>
@@
 <instance part="BREAD_450" gate="G$1" x="81.28" y="63.5"/>
 <instance part="IRQ" gate="1" x="52.23" y="-45.88" rot="R180"/>
-<instance part="H1" gate="G$1" x="-30.48" y="66.04"/>
 <instance part="H2" gate="G$1" x="-30.48" y="60.96"/>
 <instance part="H3" gate="G$1" x="-30.48" y="55.88"/>
