File: _PCB/Air Mouse-521/schematic.brd (EAGLE design)
At the start: 160 x 100 mm, 0 parts

Commit message: library update
Parts:
- added D1: (no value), SparkFun-LED:LED_3MM
- added J1, J2, J3, J4: (no value), SparkFun-Connectors:1X02_LOCK
- added M1: WIRELESS-NRF24L01, diy-modules:WIRELESS-NRF24L01
- added R1: (no value), resistor:0207/10
- added U$1: ABK-PRO-MINI, Arduino-clone:ABK-PRO-MINI
- added U1: GY-521MPU6050, gy-521:GY-521
Connections:
- new net GND: M1.1
- new net VCC: M1.2
