File: _PCB/Air Mouse-521/schematic.sch (EAGLE design)
At the start: 0 parts

Commit message: library update
Parts:
- added D1: (no value), SparkFun-LED:LED3MM
- added J1, J2, J3, J4: (no value), SparkFun-Connectors:CONN_02LOCK
- added M1: WIRELESS-NRF24L01, diy-modules:WIRELESS-NRF24L01
- added R1: (no value), resistor:R-EU_0207/10
- added U$1: ABK-PRO-MINI, Arduino-clone:ABK-PRO-MINI
- added U1: GY-521MPU6050, gy-521:GY-521MPU6050

Commit message: air mouse project added
Parts:
- added M2: ARDUINO-NANO-3.0#ISP, diy-modules:ARDUINO-NANO-3.0#ISP
- added R2, R3: (no value), resistor:R-EU_0207/10
- added S1, S2: MOMENTARY-SWITCH-SPST-PTH-6.0MM, SparkFun-Switches:MOMENTARY-SWITCH-SPST-PTH-6.0MM
Connections:
- new net N$1: R3.1, S1.2
- new net N$2: R2.1, S2.2
- new net N$3: R2.2, R3.2, U$1.VCC, U1.VCC
- new net N$4: U$1.GND, U1.GND
- new net N$5: M1.GND, U$1.GND2
Other:
- moved on the sheet: M1
Changed lines of the file:
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@@
 <part name="D1" library="SparkFun-LED" library_urn="urn:adsk.eagle:library:529" deviceset="LED" device="3MM" package3d_urn="urn:adsk.eagle:package:39361/1"/>
 <part name="R1" library="resistor" library_urn="urn:adsk.eagle:library:348" deviceset="R-EU_" device="0207/10" package3d_urn="urn:adsk.eagle:package:23491/1"/>
+<part name="S1" library="SparkFun-Switches" library_urn="urn:adsk.eagle:library:535" deviceset="MOMENTARY-SWITCH-SPST" device="-PTH-6.0MM" package3d_urn="urn:adsk.eagle:package:40163/1"/>
+<part name="S2" library="SparkFun-Switches" library_urn="urn:adsk.eagle:library:535" deviceset="MOMENTARY-SWITCH-SPST" device="-PTH-6.0MM" package3d_urn="urn:adsk.eagle:package:40163/1"/>
+<part name="R2" library="resistor" library_urn="urn:adsk.eagle:library:348" deviceset="R-EU_" device="0207/10" package3d_urn="urn:adsk.eagle:package:23491/1"/>
+<part name="R3" library="resistor" library_urn="urn:adsk.eagle:library:348" deviceset="R-EU_" device="0207/10" package3d_urn="urn:adsk.eagle:package:23491/1"/>
+<part name="M2" library="diy-modules" deviceset="ARDUINO-NANO-3.0#ISP" device=""/>
 </parts>
 <sheets>
@@
 </plain>
 <instances>
-<instance part="U1" gate="G$1" x="116.84" y="66.04"/>
-<instance part="U$1" gate="G$1" x="45.72" y="60.96"/>
-<instance part="M1" gate="G$1" x="43.18" y="7.62"/>
+<instance part="U1" gate="G$1" x="134.62" y="63.5"/>
+<instance part="U$1" gate="G$1" x="66.04" y="60.96"/>
+<instance part="M1" gate="G$1" x="-7.62" y="60.96" rot="R180"/>
 <instance part="J1" gate="G$1" x="172.72" y="78.74"/>
 <instance part="J2" gate="G$1" x="172.72" y="66.04"/>
@@
 <instance part="D1" gate="G$1" x="203.2" y="81.28"/>
 <instance part="R1" gate="G$1" x="203.2" y="68.58"/>
+<instance part="S1" gate="G$1" x="66.04" y="129.54"/>
+<instance part="S2" gate="G$1" x="66.04" y="119.38"/>
+<instance part="R2" gate="G$1" x="104.14" y="119.38"/>
+<instance part="R3" gate="G$1" x="104.14" y="129.54"/>
+<instance part="M2" gate="G$1" x="63.5" y="-5.08"/>
 </instances>
 <busses>
 </busses>
 <nets>
+<net name="N$1" class="0">
+<segment>
+<pinref part="S1" gate="G$1" pin="2"/>
+<pinref part="R3" gate="G$1" pin="1"/>
+<wire x1="71.12" y1="129.54" x2="99.06" y2="129.54" width="0.1524" layer="91"/>
+</segment>
+</net>
+<net name="N$2" class="0">
+<segment>
+<pinref part="R2" gate="G$1" pin="1"/>
+<pinref part="S2" gate="G$1" pin="2"/>
+<wire x1="99.06" y1="119.38" x2="71.12" y2="119.38" width="0.1524" layer="91"/>
+</segment>
+</net>
+<net name="N$3" class="0">
+<segment>
+<pinref part="R2" gate="G$1" pin="2"/>
+<pinref part="R3" gate="G$1" pin="2"/>
+<wire x1="109.22" y1="119.38" x2="109.22" y2="129.54" width="0.1524" layer="91"/>
+<pinref part="U$1" gate="G$1" pin="VCC"/>
+<wire x1="109.22" y1="119.38" x2="109.22" y2="68.58" width="0.1524" layer="91"/>
+<wire x1="109.22" y1="68.58" x2="109.22" y2="66.04" width="0.1524" layer="91"/>
+<wire x1="109.22" y1="66.04" x2="81.28" y2="66.04" width="0.1524" layer="91"/>
+<junction x="109.22" y="119.38"/>
+<pinref part="U1" gate="G$1" pin="VCC"/>
+<wire x1="119.38" y1="78.74" x2="109.22" y2="68.58" width="0.1524" layer="91"/>
+<junction x="109.22" y="68.58"/>
+</segment>
+</net>
+<net name="N$4" class="0">
+<segment>
+<pinref part="U1" gate="G$1" pin="GND"/>
+<pinref part="U$1" gate="G$1" pin="GND"/>
+<wire x1="119.38" y1="73.66" x2="116.84" y2="71.12" width="0.1524" layer="91"/>
+<wire x1="116.84" y1="71.12" x2="81.28" y2="71.12" width="0.1524" layer="91"/>
+</segment>
+</net>
+<net name="N$5" class="0">
+<segment>
+<pinref part="M1" gate="G$1" pin="GND"/>
+<pinref part="U$1" gate="G$1" pin="GND2"/>
+<wire x1="15.24" y1="50.8" x2="30.48" y2="66.04" width="0.1524" layer="91"/>
+<wire x1="30.48" y1="66.04" x2="43.18" y2="66.04" width="0.1524" layer="91"/>
+</segment>
+</net>
 </nets>
 </sheet>
