File: _PCB/NANO.ProMini prototype board/board.brd (EAGLE design)
At the start: 93.2 x 100.1 mm, 59 parts, among them T1_5MM 5mm, T2_5MM 5mm, T3_5MM 5mm

Commit message: final prototype
Parts:
- added PAD1, PAD10, PAD2, PAD3, PAD4, PAD5, PAD6, PAD7, PAD8, PAD9: (no value), wirepad:SMD1,27-2,54
- added U$1: USB-SERIAL-FT232R, diy-modules:USB-SERIAL-FT232R
- CP2102_USB-SERIAL: value (none) -> USB-SERIAL-CP2102
- moved VIN 71.4 mm to (32.4, 86.4), turned to 0 degrees
- moved H3 57.5 mm to (71.7, 63.1), turned to 90 degrees
- moved GND 38.8 mm to (79.4, 3.76), turned to 180 degrees
- moved CP2102_USB-SERIAL 36.4 mm to (97.5, 37.1), turned to 180 degrees
- moved 5V 34.9 mm to (79.4, 9.09), turned to 180 degrees
- moved 3.3V 32.2 mm to (79.4, 14.4), turned to 180 degrees
- moved J8 30.4 mm to (65.2, 34.7), turned to 90 degrees
- moved J2 24.0 mm to (65.9, 28.0), turned to 180 degrees
- moved H4 20.3 mm to (34.7, 63.1)
- moved ESP_C 16.6 mm to (89.3, 88.1), turned to 90 degrees
- moved J7 14.6 mm to (78.7, 30.6), turned to 90 degrees
- moved S2 13.1 mm to (73.6, 22.4), turned to 180 degrees
- moved S4 13.1 mm to (73.6, 22.4), turned to 90 degrees
- moved S1 11.1 mm to (83.2, 22.5), turned to 180 degrees
- moved S3 11.1 mm to (83.2, 22.5), turned to 90 degrees
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Connections:
- removed net N$56: CP2102_USB-SERIAL.2, J7.2, J9.2, PROMINI_H.6
- new net N$65: BOARD_POWER.1, PAD10.1
- new net N$66: CP2102_USB-SERIAL.2, J7.6, J9.2, PROMINI_H.6, U$1.1
- net 3.3V: now also J7.2, PAD1.1, PAD3.1, PAD5.1, PAD7.1; no longer J7.1
- net 5V: now also J7.3, PAD8.1, U$1.4; no longer J7.6
- net GND: now also J7.1, U$1.6; no longer J7.5
- net N$36: now also PAD9.1
- net N$55: now also PAD2.1, PAD6.1
- net N$57: now also J7.5, U$1.2; no longer J7.3
- net N$62: now also U$1.3
- net N$76: now also PAD4.1
Routing:
- net 3.3V: track 307.6 -> 0.00 mm
- net 5V: track 235.7 -> 0.00 mm, vias 4 -> 0
- net N$36: track 181.7 -> 0.00 mm, vias 2 -> 0
- net D+_5PIN: track 165.9 -> 0.00 mm, vias 1 -> 0
- net D-_5PIN: track 149.1 -> 0.00 mm
- net VIN: track 110.8 -> 0.00 mm
- net SCK_NRF: track 70.0 -> 0.00 mm
- net A5: track 61.6 -> 0.00 mm
- net SDA_GY521: track 59.6 -> 0.00 mm
- net CE_NRF: track 56.5 -> 0.00 mm
- net CSN_NRF: track 51.3 -> 0.00 mm
- net N$57: track 39.9 -> 0.00 mm
- net N$62: track 39.7 -> 0.00 mm
- net N$56: track 38.9 -> 0.00 mm
- net MOSI_NRF: track 37.0 -> 0.00 mm
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
Commit message: really final prototype
Routing:
- net 3.3V: track 0.00 -> 342.6 mm, vias 0 -> 2
- net 5V: track 0.00 -> 283.5 mm, vias 0 -> 3
- net D+_5PIN: track 0.00 -> 148.0 mm
- net N$36: track 0.00 -> 144.1 mm, vias 0 -> 3
- net D-_5PIN: track 0.00 -> 119.1 mm
- net VIN: track 0.00 -> 86.6 mm
- net SCK_NRF: track 0.00 -> 77.3 mm
- net N$66: track 0.00 -> 67.4 mm
- net A5: track 0.00 -> 62.3 mm
- net SDA_GY521: track 0.00 -> 61.5 mm
- net N$57: track 0.00 -> 60.8 mm
- net CE_NRF: track 0.00 -> 56.6 mm
- net CSN_NRF: track 0.00 -> 53.3 mm
- net N$62: track 0.00 -> 47.1 mm
- net MOSI_NRF: track 0.00 -> 37.8 mm
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
Commit message: update
Parts:
- added ESP1_1, ESP2_1, R1_1, R2_1: (no value), rcl:R2012
- moved ESP1 2.44 mm to (85.2, 88.4)
- moved ESP2 2.44 mm to (82.2, 88.4)
- moved R1 0.41 mm to (47.1, 22.3)
Connections:
- net GND: now also ESP2_1.1
- net N$13: now also R1_1.1
- net N$14: now also R2_1.1
- net N$15: now also R1_1.2
- net N$38: now also R2_1.2
- net N$58: now also ESP1_1.1, ESP2_1.2
- net N$61: now also ESP1_1.2
Routing:
- net N$58: track 17.4 -> 26.5 mm
- net N$15: track 37.4 -> 42.1 mm
- net N$14: track 27.5 -> 32.1 mm, vias 0 -> 1
- net N$13: track 31.2 -> 35.4 mm, vias 0 -> 1
- net N$61: track 18.9 -> 22.9 mm
- net N$38: track 33.8 -> 37.7 mm, vias 0 -> 1
- net CE_NRF: track 56.6 -> 59.4 mm
