File: _PCB/NANO.ProMini prototype board/board.sch (EAGLE design)
At the start: 70 parts, among them T1_5MM 5mm, T2_5MM 5mm, T3_5MM 5mm

Commit message: update
Parts:
- added ESP1_1, ESP2_1, R1_1, R2_1: (no value), rcl:R-US_R2012
Connections:
- net GND: now also ESP2_1.1
- net N$13: now also R1_1.1
- net N$14: now also R2_1.1
- net N$15: now also R1_1.2
- net N$38: now also R2_1.2
- net N$58: now also ESP1_1.1, ESP2_1.2
- net N$61: now also ESP1_1.2
Changed lines of the file:
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@@
 <?xml version="1.0" encoding="utf-8"?>
 <!DOCTYPE eagle SYSTEM "eagle.dtd">
-<eagle version="9.1.1">
+<eagle version="9.1.2">
 <drawing>
 <settings>
@@
 <part name="U$1" library="diy-modules" deviceset="USB-SERIAL-FT232R" device=""/>
 <part name="J7" library="SparkFun-Connectors" library_urn="urn:adsk.eagle:library:513" deviceset="CONN_06" device="LOCK" package3d_urn="urn:adsk.eagle:package:38002/1"/>
+<part name="ESP2_1" library="rcl" library_urn="urn:adsk.eagle:library:334" deviceset="R-US_" device="R2012" package3d_urn="urn:adsk.eagle:package:23543/2"/>
+<part name="ESP1_1" library="rcl" library_urn="urn:adsk.eagle:library:334" deviceset="R-US_" device="R2012" package3d_urn="urn:adsk.eagle:package:23543/2"/>
+<part name="R1_1" library="rcl" library_urn="urn:adsk.eagle:library:334" deviceset="R-US_" device="R2012" package3d_urn="urn:adsk.eagle:package:23543/2"/>
+<part name="R2_1" library="rcl" library_urn="urn:adsk.eagle:library:334" deviceset="R-US_" device="R2012" package3d_urn="urn:adsk.eagle:package:23543/2"/>
 </parts>
 <sheets>
@@
 <instance part="U$1" gate="G$1" x="-76.2" y="73.66"/>
 <instance part="J7" gate="G$1" x="12.7" y="76.2" rot="R180"/>
+<instance part="ESP2_1" gate="G$1" x="-134.62" y="-76.2"/>
+<instance part="ESP1_1" gate="G$1" x="-114.3" y="-76.2"/>
+<instance part="R1_1" gate="G$1" x="116.84" y="-7.62"/>
+<instance part="R2_1" gate="G$1" x="116.84" y="0"/>
 </instances>
 <busses>
@@
 <wire x1="-139.7" y1="-111.76" x2="-116.84" y2="-111.76" width="0.1524" layer="91"/>
 <junction x="-116.84" y="-111.76"/>
+<pinref part="ESP2_1" gate="G$1" pin="1"/>
+<wire x1="-139.7" y1="-83.82" x2="-139.7" y2="-76.2" width="0.1524" layer="91"/>
+<junction x="-139.7" y="-83.82"/>
 </segment>
 </net>
@@
 <pinref part="J1" gate="G$1" pin="4"/>
 <wire x1="111.76" y1="-10.16" x2="104.14" y2="-17.78" width="0.1524" layer="91"/>
+<pinref part="R1_1" gate="G$1" pin="1"/>
+<wire x1="111.76" y1="-7.62" x2="111.76" y2="-10.16" width="0.1524" layer="91"/>
+<junction x="111.76" y="-10.16"/>
 </segment>
 </net>
@@
 <pinref part="J1" gate="G$1" pin="3"/>
 <wire x1="106.68" y1="-17.78" x2="104.14" y2="-20.32" width="0.1524" layer="91"/>
+<pinref part="R2_1" gate="G$1" pin="1"/>
+<wire x1="111.76" y1="0" x2="111.76" y2="-2.54" width="0.1524" layer="91"/>
+<junction x="111.76" y="-2.54"/>
 </segment>
 </net>
@@
 <wire x1="121.92" y1="-10.16" x2="121.92" y2="-15.24" width="0.1524" layer="91"/>
 <wire x1="121.92" y1="-15.24" x2="129.54" y2="-22.86" width="0.1524" layer="91"/>
+<pinref part="R1_1" gate="G$1" pin="2"/>
+<wire x1="121.92" y1="-7.62" x2="121.92" y2="-10.16" width="0.1524" layer="91"/>
+<junction x="121.92" y="-10.16"/>
 </segment>
 </net>
@@
 <pinref part="R2" gate="G$1" pin="2"/>
 <wire x1="121.92" y1="-2.54" x2="124.46" y2="-5.08" width="0.1524" layer="91"/>
-<wire x1="124.46" y1="-5.08" x2="124.46" y2="-12.7" width="0.1524" layer="91"/>
+<wire x1="124.46" y1="-5.08" x2="124.46" y2="-15.24" width="0.1524" layer="91"/>
 <pinref part="ES32-433T20D" gate="G$1" pin="3"/>
-<wire x1="124.46" y1="-12.7" x2="124.46" y2="-15.24" width="0.1524" layer="91"/>
 <wire x1="124.46" y1="-15.24" x2="129.54" y2="-20.32" width="0.1524" layer="91"/>
+<pinref part="R2_1" gate="G$1" pin="2"/>
+<wire x1="121.92" y1="-2.54" x2="121.92" y2="0" width="0.1524" layer="91"/>
+<junction x="121.92" y="-2.54"/>
 </segment>
 </net>
@@
 <wire x1="-119.38" y1="-83.82" x2="-129.54" y2="-83.82" width="0.1524" layer="91"/>
 <junction x="-119.38" y="-83.82"/>
+<pinref part="ESP2_1" gate="G$1" pin="2"/>
+<wire x1="-129.54" y1="-83.82" x2="-129.54" y2="-76.2" width="0.1524" layer="91"/>
+<junction x="-129.54" y="-83.82"/>
+<wire x1="-119.38" y1="-83.82" x2="-119.38" y2="-76.2" width="0.1524" layer="91"/>
+<pinref part="ESP1_1" gate="G$1" pin="1"/>
 </segment>
 </net>
@@
 <wire x1="-116.84" y1="-93.98" x2="-109.22" y2="-86.36" width="0.1524" layer="91"/>
 <wire x1="-109.22" y1="-86.36" x2="-109.22" y2="-83.82" width="0.1524" layer="91"/>
-</segment>
-</net>
+<pinref part="ESP1_1" gate="G$1" pin="2"/>
+<wire x1="-109.22" y1="-83.82" x2="-109.22" y2="-76.2" width="0.1524" layer="91"/>
+<junction x="-109.22" y="-83.82"/>
+</segment>
+</net>
