File: _PCB/NANO.ProMini_MINI prototype board/board.brd (EAGLE design)
At the start: 93.2 x 100.1 mm, 48 parts, among them T1_5MM 5mm, T2_5MM 5mm

Commit message: update
Parts:
- removed BOARD_POWER: (no value), SparkFun-Connectors:1X04_LOCK_LONGPADS
- removed CP2102_USB-SERIAL: USB-SERIAL-CP2102, diy-modules:USB-SERIAL-CP2102
- removed ESP1: 1k, rcl:R2012
- removed ESP2: 2k, rcl:R2012
- removed ESP8266: (no value), diy-modules:WIRELESS-WIFI-ESP-01
- removed ESP_C: (no value), rcl:E2,5-5
- removed ESP_H: (no value), SparkFun-Connectors:2X3
- removed ESP_POW, PIEZO, PIN2: (no value), SparkFun-Connectors:1X02_LOCK
- removed H1, H2, H3, H4: MOUNT-HOLE3.0, holes:3,0
- removed J2: (no value), SparkFun-Connectors:1X02_LOCK_LONGPADS
- removed J7, J9: (no value), SparkFun-Connectors:1X06_LOCK
- removed MICRO_2: (no value), SparkFun-Connectors:USB-MICROB
- removed PC1, PC2: 47u, rcl:PANASONIC_D
- removed PIEZO_: (no value), buzzer:F/CM12P
- removed PROMINI_H: (no value), pinhead_v2:1X06/OCT
- removed RAW: (no value), SparkFun-Connectors:POWER_JACK_SLOT
- removed S1, S2: MOMENTARY-SWITCH-SPST-PTH-6.0MM, SparkFun-Switches:TACTILE_SWITCH_PTH_6.0MM
- removed S3, S4: DTS-3, switch-tact:DTS-3
- removed T2_5MM: 5mm, Seeed-Connector:H2-5.0-10.5X8.0MM
- removed U$1: USB-SERIAL-FT232R, diy-modules:USB-SERIAL-FT232R
- removed USB_B: (no value), SparkFun-Connectors:USB-B-PTH
- removed VIN: (no value), SparkFun-Connectors:1X03_LOCK
- added POWER: (no value), SparkFun-Connectors:1X03_LOCK
- 3.3V_C: device rcl:E2,5-5 -> rcl:PANASONIC_D
- 5V_C: device resistor:E3,5-8 -> rcl:PANASONIC_D
- moved T1_5MM 91.6 mm to (53.0, 4.19), turned to 270 degrees
- moved SW1 82.2 mm to (6.22, 34.2), turned to 90 degrees
- moved PIN1 78.4 mm to (53.1, 9.78), turned to 0 degrees
- moved J4 71.4 mm to (13.7, 38.0), turned to 270 degrees
- moved 3.3V_C 62.2 mm to (30.4, 17.2)
- moved 5V_C 58.3 mm to (31.9, 28.8)
- moved NRF24L01 39.7 mm to (1.93, 19.7)
- moved ES32-433T20D 39.3 mm to (53.4, 38.7), turned to 270 degrees
- moved J1 33.6 mm to (50.3, 38.7), turned to 270 degrees
- moved 5V 19.9 mm to (11.6, 10.0), turned to 180 degrees
- moved GND 17.0 mm to (11.4, 2.79), turned to 180 degrees
- moved 3.3V 14.5 mm to (11.6, 6.35), turned to 180 degrees
- moved PH1 14.0 mm to (43.4, 20.1)
- moved NANO 14.0 mm to (29.4, 29.0)
- moved PH2 14.0 mm to (20.5, 20.1)
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Connections:
- removed net N$27: PIN2.2, T2_5MM.1
- removed net N$31: PIN2.1, T2_5MM.2
- removed net N$32: MICRO_2.D+, USB_B.D+
- removed net N$33: MICRO_2.D-, USB_B.D-
- removed net N$34: PIEZO.1, PIEZO.2, PIEZO_.+
- removed net N$35: GND.1, GND.2, GND.4
- removed net N$37: J2.1, S1.3, S3.2
- removed net N$43: J2.2, S2.3, S4.1
- removed net N$55: ESP8266.B2, ESP_POW.2
- removed net N$57: CP2102_USB-SERIAL.3, J7.5, J9.3, PROMINI_H.4, U$1.2
- removed net N$58: ESP1.1, ESP2.2, ESP8266.D1
- removed net N$59: ESP8266.C2, ESP_H.2
- removed net N$60: ESP8266.C1, ESP_H.3
- removed net N$61: ESP1.2, ESP_H.1
- removed net N$62: CP2102_USB-SERIAL.4, J7.4, J9.4, PROMINI_H.5, U$1.3
- removed net N$63: ESP8266.B1, ESP_H.5
- removed net N$64: ESP8266.A2, ESP_H.6
- removed net N$66: CP2102_USB-SERIAL.2, J7.6, J9.2, PROMINI_H.6, U$1.1
- net 3.3V: now also POWER.3; no longer BOARD_POWER.4, CP2102_USB-SERIAL.1, ESP8266.D2, ESP_C.+, ESP_POW.1, J7.2, J9.1
- net 5V: now also POWER.1; no longer BOARD_POWER.2, CP2102_USB-SERIAL.6, J7.3, J9.6, MICRO_2.VBUS, U$1.4, USB_B.VBUS
- net GND: now also GND.1, GND.2, GND.4; no longer CP2102_USB-SERIAL.5, ESP2.1, ESP8266.A1, ESP_C.-, J7.1, J9.5, MICRO_2.GND, PIEZO_.-, PROMINI_H.1, RAW.GND@1, U$1.6, USB_B.GND
- net N$36: now also POWER.2; no longer BOARD_POWER.3, PROMINI_H.3, S1.1, S2.1, S3.1, S4.2
- net VIN: no longer RAW.PWR, VIN.1, VIN.2, VIN.3
Routing:
- net 3.3V: track 317.9 -> 112.3 mm, vias 2 -> 3
- net 5V: track 236.7 -> 91.3 mm, vias 3 -> 1
- net VIN: track 75.8 -> 5.13 mm
- net N$66: track 67.4 -> 0.00 mm
- net N$57: track 60.8 -> 0.00 mm
- net A5: track 62.3 -> 5.13 mm
- net SDA_GY521: track 61.5 -> 5.13 mm
- net N$36: track 143.7 -> 87.8 mm, vias 3 -> 0
- net CE_NRF: track 59.4 -> 10.4 mm
- net N$62: track 47.1 -> 0.00 mm
- net SCK_NRF: track 77.3 -> 36.7 mm
- net CSN_NRF: track 53.3 -> 14.0 mm
- net N$55: track 28.1 -> 0.00 mm
- net N$38: track 35.1 -> 11.2 mm, vias 1 -> 0
- net N$37: track 22.0 -> 0.00 mm
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Other:
- board size 93.2 x 100.1 mm -> 58.2 x 41 mm
- board text removed: "0"
- board text removed: "1k"
- board text removed: "2k"
- board text removed: "3V3"
- board text removed: "ADO"
- board text removed: "BOARD_POWER"
- board text removed: "CE"
- board text removed: "CSN"
- board text removed: "D+"
- board text removed: "D-"
- board text removed: "DTR"
- board text removed: "DTR_RST"
- board text removed: "ESP_POWER"
- board text removed: "GPIO0"
- board text removed: "GPIO2"
- board text removed: "INT"
- board text removed: "IRQ"
- board text removed: "LoRa"
- board text removed: "MOSI"
- board text removed: "NC"
- board text removed: "NSS"
- board text removed: "OFF"
- board text removed: "RA02 POW"
- board text removed: "SWITCH"
- board text removed: "VCC"
- board text removed: "XCL"
- board text removed: "XDA"
- board text removed: "connected to board _power"
