File: _PCB/NANO.ProMini_MINI prototype board/board.sch (EAGLE design)
At the start: 48 parts, among them T1_5MM 5mm, T2_5MM 5mm

Commit message: update
Parts:
- removed BOARD_POWER: (no value), SparkFun-Connectors:CONN_04LOCK_LONGPADS
- removed CP2102_USB-SERIAL: USB-SERIAL-CP2102, diy-modules:USB-SERIAL-CP2102
- removed ESP1: 1k, rcl:R-US_R2012
- removed ESP2: 2k, rcl:R-US_R2012
- removed ESP8266: WIRELESS-WIFI-ESP-01, diy-modules:WIRELESS-WIFI-ESP-01
- removed ESP_C: (no value), rcl:CPOL-EUE2.5-5
- removed ESP_H: (no value), SparkFun-Connectors:CONN_03X2FEMALE
- removed ESP_POW, PIEZO, PIN2: (no value), SparkFun-Connectors:CONN_02LOCK
- removed H1, H2, H3, H4: MOUNT-HOLE3.0, holes:MOUNT-HOLE3.0
- removed J2: (no value), SparkFun-Connectors:CONN_02LOCK_LONGPADS
- removed J7, J9: (no value), SparkFun-Connectors:CONN_06LOCK
- removed MICRO_2: (no value), SparkFun-Connectors:USB_MICRO-B_SMT
- removed PC1, PC2: 47u, rcl:CPOL-EUD
- removed PIEZO_: F/CM12P, buzzer:F/CM12P
- removed PROMINI_H: (no value), pinhead_v2:PINHD-1X6/OCT
- removed RAW: POWER_JACKSLT, SparkFun-Connectors:POWER_JACKSLT
- removed S1, S2: MOMENTARY-SWITCH-SPST-PTH-6.0MM, SparkFun-Switches:MOMENTARY-SWITCH-SPST-PTH-6.0MM
- removed S3, S4: DTS-3, switch-tact:DTS-3
- removed T2_5MM: 5mm, Seeed-Connector:SCREW-TERMINAL-GREEN(2P-5.0)
- removed U$1: USB-SERIAL-FT232R, diy-modules:USB-SERIAL-FT232R
- removed USB_B: USB_B_PTH, SparkFun-Connectors:USB_B_PTH
- removed VIN: (no value), SparkFun-Connectors:CONN_03LOCK
- added POWER: (no value), SparkFun-Connectors:CONN_03LOCK
- 3.3V_C: device rcl:CPOL-EUE2.5-5 -> rcl:CPOL-EUD
- 5V_C: device resistor:CPOL-EUE3.5-8 -> rcl:CPOL-EUD
Connections:
- removed net N$27: PIN2.2, T2_5MM.1
- removed net N$31: PIN2.1, T2_5MM.2
- removed net N$32: MICRO_2.D+, USB_B.D+
- removed net N$33: MICRO_2.D-, USB_B.D-
- removed net N$34: PIEZO.1, PIEZO.2, PIEZO_.1
- removed net N$35: GND.1, GND.2, GND.4
- removed net N$37: J2.1, S1.2, S3.2
- removed net N$43: J2.2, S2.2, S4.1
- removed net N$55: ESP8266.CH_PD, ESP_POW.2
- removed net N$57: CP2102_USB-SERIAL.RXI, J7.5, J9.3, PROMINI_H.4, U$1.RX
- removed net N$58: ESP1.1, ESP2.2, ESP8266.URXD
- removed net N$59: ESP8266.RST, ESP_H.2
- removed net N$60: ESP8266.GPIO0, ESP_H.3
- removed net N$61: ESP1.2, ESP_H.1
- removed net N$62: CP2102_USB-SERIAL.TDO, J7.4, J9.4, PROMINI_H.5, U$1.TX
- removed net N$63: ESP8266.GPIO2, ESP_H.5
- removed net N$64: ESP8266.UTXD, ESP_H.6
- removed net N$66: CP2102_USB-SERIAL.DTR, J7.6, J9.2, PROMINI_H.6, U$1.DTR
- net 3.3V: now also POWER.3; no longer BOARD_POWER.4, CP2102_USB-SERIAL.3V3, ESP8266.VCC, ESP_C.+, ESP_POW.1, J7.2, J9.1
- net 5V: now also POWER.1; no longer BOARD_POWER.2, CP2102_USB-SERIAL.+5V, J7.3, J9.6, MICRO_2.VBUS, U$1.VCC, USB_B.VBUS
- net GND: now also GND.1, GND.2, GND.4; no longer CP2102_USB-SERIAL.GND, ESP2.1, ESP8266.GND, ESP_C.-, J7.1, J9.5, MICRO_2.GND, PIEZO_.2, PROMINI_H.1, RAW.GNDBREAK, U$1.GND, USB_B.GND
- net N$36: now also POWER.2; no longer BOARD_POWER.3, PROMINI_H.3, S1.1, S2.1, S3.1, S4.2
- net VIN: no longer RAW.PWR, VIN.1, VIN.2, VIN.3
Other:
- moved on the sheet: 3.3V, 3.3V_C, 5V, 5V_C, GND, PIN1, T1_5MM
