File: _PCB/_Prototyping Boards/NANO.ProMini_prototype board/board.brd (EAGLE design)
At the start: 93.2 x 100.1 mm, 74 parts, among them T1_5MM 5mm, T2_5MM 5mm, T3_5MM 5mm

Commit message: IMU + proto board update
Parts:
- removed 3.3/5: (no value), SparkFun-Connectors:1X03_LOCK
- removed BOARD_POWER: (no value), SparkFun-Connectors:1X04_LOCK_LONGPADS
- removed PAD10, PAD7, PAD8, PAD9: (no value), wirepad:SMD1,27-2,54
Connections:
- removed net N$11: 3.3/5.2, ES32-433T20D.6
- removed net N$36: BOARD_POWER.3, NANO.5V, PAD9.1, PH1.23, PH1.24, PROMINI_H.3, S1.1, S2.1, S3.1, S4.2, SW1.5, SW1.6, SW1.7, SW1.8
- removed net N$65: BOARD_POWER.1, PAD10.1
- net 3.3V: now also ES32-433T20D.6, NRF24L01.2; no longer 3.3/5.3, BOARD_POWER.4, PAD7.1
- net 5V: now also NANO.5V, PH1.23, PH1.24, PROMINI_H.3; no longer 3.3/5.1, BOARD_POWER.2, NRF24L01.2, PAD8.1
- net GND: now also S1.1, S2.1, S3.1, S4.2, SW1.5, SW1.6, SW1.7, SW1.8
Routing:
- net N$36: track 144.1 -> 0.00 mm, vias 3 -> 0
- net 5V: track 283.5 -> 374.6 mm, vias 3 -> 6
- net GND: track 0.00 -> 36.5 mm
- net 3.3V: track 342.6 -> 350.5 mm
- net N$11: track 4.99 -> 0.00 mm
- net N$65: track 3.82 -> 0.00 mm
