File: _PCB/_Prototyping Boards/NANO.ProMini_prototype board/board.sch (EAGLE design)
At the start: 74 parts, among them T1_5MM 5mm, T2_5MM 5mm, T3_5MM 5mm

Commit message: IMU + proto board update
Parts:
- removed 3.3/5: (no value), SparkFun-Connectors:CONN_03LOCK
- removed BOARD_POWER: (no value), SparkFun-Connectors:CONN_04LOCK_LONGPADS
- removed PAD10, PAD7, PAD8, PAD9: (no value), wirepad:SMD2
Connections:
- removed net N$11: 3.3/5.2, ES32-433T20D.6
- removed net N$36: BOARD_POWER.3, NANO.5.5V, PAD9.P, PH1.23, PH1.24, PROMINI_H.3, S1.1, S2.1, S3.1, S4.2, SW1.5, SW1.6, SW1.7, SW1.8
- removed net N$65: BOARD_POWER.1, PAD10.P
- net 3.3V: now also ES32-433T20D.6, NRF24L01.VCC; no longer 3.3/5.3, BOARD_POWER.4, PAD7.P
- net 5V: now also NANO.5.5V, PH1.23, PH1.24, PROMINI_H.3; no longer 3.3/5.1, BOARD_POWER.2, NRF24L01.VCC, PAD8.P
- net GND: now also S1.1, S2.1, S3.1, S4.2, SW1.5, SW1.6, SW1.7, SW1.8
