File: _PCB/_Prototyping Boards/NANO.ProMini_MINI prototype board/board.brd (EAGLE design)
At the start: 57.2 x 41 mm, 26 parts, among them T1_5MM 5mm

Commit message: prototype board complete
Parts:
- removed R2: 4.7k, rcl:R2012
- added 3.3V_C1: (no value), rcl:PANASONIC_D
- added MICRO_3: (no value), SparkFun-Connectors:USB-MICROB
- moved 5V_C 12.2 mm to (30.7, 15.6), turned to 0 degrees
- moved 3.3REG 5.96 mm to (29.5, 2.41), turned to 180 degrees
- moved 3.3V_C 4.40 mm to (30.7, 22.4), turned to 0 degrees
- moved C3.3 4.05 mm to (25.7, 5.84), turned to 90 degrees
- moved C5 1.20 mm to (34.0, 2.16)
- moved I2C_1 1.09 mm to (52.6, 10.5)
- moved REG3.3 0.81 mm to (30.7, 7.87)
- moved SW1 0.13 mm to (6.86, 35.2)
- moved J4 0.13 mm to (14.1, 39.0)
- renumbered 3.3V to 3V3, ES32-433T20D to ES32-TTL
Connections:
- net A5 renamed SCL
- net 3.3V: now also 3.3V_C1.+
- net 5V: now also MICRO_3.VBUS
- net GND: now also 3.3V_C1.-, MICRO_3.GND
Routing:
- net 5V: track 0.00 -> 149.0 mm, vias 0 -> 2
- net 3.3V: track 0.00 -> 110.3 mm, vias 0 -> 1
- net ES32_TXD: track 0.00 -> 54.3 mm
- net N$17: track 0.00 -> 53.8 mm
- net M1: track 0.00 -> 39.1 mm
- net SCK_NRF: track 0.00 -> 38.6 mm, vias 0 -> 1
- net M0: track 0.00 -> 38.2 mm
- net SCL: track 0.00 -> 37.1 mm
- net ES32_AUX: track 0.00 -> 35.1 mm
- net SDA: track 0.00 -> 21.2 mm, vias 0 -> 1
- net MOSI_NRF: track 0.00 -> 18.0 mm
- net MISO_NRF: track 0.00 -> 14.1 mm
- net CSN_NRF: track 0.00 -> 12.7 mm
- net ES32_RXD: track 0.00 -> 9.54 mm
- net CE_NRF: track 0.00 -> 9.45 mm
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Other:
- board text removed: "3.3"
- board text removed: "A1"
- board text removed: "A2"
- board text removed: "A3"
- board text removed: "A4"
- board text removed: "A5"
- board text removed: "A6"
- board text removed: "A7"
- board text removed: "D0"
- board text removed: "D10"
- board text removed: "D11"
- board text removed: "D13"
- board text removed: "D2"
- board text removed: "D5"
- board text removed: "D6"
- board text removed: "D7"
- board text removed: "RST"

Commit message: PCB update
Parts:
- moved R1 60.8 mm to (4.26, 1.69), turned to 270 degrees
- moved JP1 56.7 mm to (4.06, 5.59), turned to 0 degrees
- moved ES32-TTL 55.3 mm to (8.71, 0.79), turned to 90 degrees
- moved NRF24L01 54.9 mm to (55.7, 18.8), turned to 0 degrees
- moved T1_5MM 54.6 mm to (52.3, 33.3), turned to 0 degrees
- moved JP2 54.1 mm to (4.06, 8.26), turned to 0 degrees
- moved 5.GND 53.1 mm to (5.84, 34.4), turned to 0 degrees
- moved MICRO_3 52.6 mm to (2.54, 15.1), turned to 180 degrees
- moved SW1 52.3 mm to (50.0, 5.59), turned to 270 degrees
- moved I2C_1 52.3 mm to (4.06, 30.0), turned to 270 degrees
- moved 3V3 51.8 mm to (9.65, 38.2), turned to 180 degrees
- moved MICRO_1 50.9 mm to (53.8, 19.4), turned to 0 degrees
- moved J4 46.8 mm to (42.4, 1.78), turned to 90 degrees
- moved PAD2 45.2 mm to (10.9, 5.84), turned to 180 degrees
- moved PAD1 42.1 mm to (10.9, 8.38), turned to 180 degrees
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Other:
- outline, holes or cut-outs redrawn
