File: _PCB/_Prototyping Boards/NANO.ProMini_MINI prototype board/board.sch (EAGLE design)
At the start: 20 parts, among them T1_5MM 5mm

Commit message: fixed errors
Parts:
- removed POWER: (no value), SparkFun-Connectors:CONN_03LOCK
Connections:
- removed net N$36: NANO.5.5V, PH1.23, PH1.24, POWER.2, SW1.5, SW1.6, SW1.7, SW1.8
- net 3.3V: no longer POWER.3
- net 5V: now also NANO.5.5V, PH1.23, PH1.24, SW1.5, SW1.6, SW1.7, SW1.8; no longer POWER.1
Changed lines of the file:
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@@
 <?xml version="1.0" encoding="utf-8"?>
 <!DOCTYPE eagle SYSTEM "eagle.dtd">
-<eagle version="9.1.2">
+<eagle version="9.1.3">
 <drawing>
 <settings>
@@
 <part name="5V_C" library="rcl" deviceset="CPOL-EU" device="D"/>
 <part name="3.3V_C" library="rcl" deviceset="CPOL-EU" device="D"/>
-<part name="POWER" library="SparkFun-Connectors" library_urn="urn:adsk.eagle:library:513" deviceset="CONN_03" device="LOCK" package3d_urn="urn:adsk.eagle:package:38071/1"/>
 <part name="GND" library="SparkFun-Connectors" library_urn="urn:adsk.eagle:library:513" deviceset="CONN_04" device="LOCK" package3d_urn="urn:adsk.eagle:package:38089/1"/>
 <part name="MICRO_1" library="SparkFun-Connectors" library_urn="urn:adsk.eagle:library:513" deviceset="USB_MICRO-B" device="_SMT" package3d_urn="urn:adsk.eagle:package:38240/1"/>
@@
 <attribute name="VALUE" x="-83.82" y="2.54" size="1.778" layer="96"/>
 </instance>
-<instance part="POWER" gate="J$1" x="-48.26" y="-38.1"/>
 <instance part="GND" gate="G$1" x="-106.68" y="-27.94"/>
 <instance part="MICRO_1" gate="G$1" x="-99.06" y="-76.2" rot="R180"/>
@@
 <wire x1="-20.32" y1="17.78" x2="-15.24" y2="17.78" width="0.1524" layer="91"/>
 <wire x1="-76.2" y1="7.62" x2="-66.04" y2="17.78" width="0.1524" layer="91"/>
-<wire x1="-66.04" y1="17.78" x2="-33.02" y2="17.78" width="0.1524" layer="91"/>
+<wire x1="-66.04" y1="17.78" x2="-27.94" y2="17.78" width="0.1524" layer="91"/>
 <pinref part="PH1" gate="A" pin="3"/>
-<wire x1="-33.02" y1="17.78" x2="-27.94" y2="17.78" width="0.1524" layer="91"/>
 <wire x1="-27.94" y1="17.78" x2="-20.32" y2="17.78" width="0.1524" layer="91"/>
 <junction x="-27.94" y="17.78"/>
 <pinref part="PH1" gate="A" pin="4"/>
 <junction x="-20.32" y="17.78"/>
-<junction x="-33.02" y="17.78"/>
 <junction x="-101.6" y="7.62"/>
-<wire x1="-33.02" y1="-27.94" x2="-33.02" y2="17.78" width="0.1524" layer="91"/>
-<wire x1="-40.64" y1="-35.56" x2="-33.02" y2="-27.94" width="0.1524" layer="91"/>
 <wire x1="-101.6" y1="7.62" x2="-101.6" y2="5.08" width="0.1524" layer="91"/>
 <pinref part="3.3V" gate="G$1" pin="1"/>
@@
 <junction x="-101.6" y="10.16"/>
 <pinref part="3.3V" gate="G$1" pin="4"/>
-<pinref part="POWER" gate="J$1" pin="3"/>
 <pinref part="3.3V_C" gate="G$1" pin="+"/>
 <junction x="-76.2" y="7.62"/>
@@
 <net name="5V" class="1">
 <segment>
-<wire x1="-76.2" y1="-5.08" x2="-71.12" y2="-5.08" width="0.1524" layer="91"/>
 <wire x1="-76.2" y1="-5.08" x2="-101.6" y2="-5.08" width="0.1524" layer="91"/>
 <wire x1="-101.6" y1="-10.16" x2="-101.6" y2="-12.7" width="0.1524" layer="91"/>
 <wire x1="-101.6" y1="-10.16" x2="-101.6" y2="-7.62" width="0.1524" layer="91"/>
 <wire x1="-101.6" y1="-5.08" x2="-101.6" y2="-7.62" width="0.1524" layer="91"/>
-<wire x1="-71.12" y1="-5.08" x2="-38.1" y2="-5.08" width="0.1524" layer="91"/>
-<wire x1="-38.1" y1="-5.08" x2="-38.1" y2="-40.64" width="0.1524" layer="91"/>
-<wire x1="-38.1" y1="-40.64" x2="-40.64" y2="-40.64" width="0.1524" layer="91"/>
+<wire x1="-76.2" y1="-5.08" x2="-48.26" y2="-5.08" width="0.1524" layer="91"/>
 <pinref part="5V" gate="G$1" pin="1"/>
 <pinref part="5V" gate="G$1" pin="2"/>
@@
 <pinref part="5V" gate="G$1" pin="4"/>
 <junction x="-101.6" y="-5.08"/>
-<pinref part="POWER" gate="J$1" pin="1"/>
 <pinref part="5V_C" gate="G$1" pin="+"/>
 <junction x="-76.2" y="-5.08"/>
+<pinref part="NANO" gate="G$1" pin="5.5V"/>
+<pinref part="PH1" gate="A" pin="23"/>
+<wire x1="-27.94" y1="-7.62" x2="-20.32" y2="-7.62" width="0.1524" layer="91"/>
+<pinref part="PH1" gate="A" pin="24"/>
+<junction x="-20.32" y="-7.62"/>
+<wire x1="-20.32" y1="-7.62" x2="-15.24" y2="-7.62" width="0.1524" layer="91"/>
+<wire x1="-48.26" y1="-5.08" x2="-45.72" y2="-7.62" width="0.1524" layer="91"/>
+<wire x1="-45.72" y1="-7.62" x2="-27.94" y2="-7.62" width="0.1524" layer="91"/>
+<junction x="-27.94" y="-7.62"/>
+<pinref part="SW1" gate="A" pin="5"/>
+<pinref part="SW1" gate="A" pin="6"/>
+<wire x1="-25.4" y1="-35.56" x2="-25.4" y2="-38.1" width="0.1524" layer="91"/>
+<pinref part="SW1" gate="A" pin="7"/>
+<wire x1="-25.4" y1="-38.1" x2="-25.4" y2="-40.64" width="0.1524" layer="91"/>
+<junction x="-25.4" y="-38.1"/>
+<pinref part="SW1" gate="A" pin="8"/>
+<wire x1="-25.4" y1="-40.64" x2="-25.4" y2="-43.18" width="0.1524" layer="91"/>
+<junction x="-25.4" y="-40.64"/>
+<wire x1="-25.4" y1="-38.1" x2="-40.64" y2="-38.1" width="0.1524" layer="91"/>
+<wire x1="-45.72" y1="-7.62" x2="-45.72" y2="-33.02" width="0.1524" layer="91"/>
+<wire x1="-45.72" y1="-33.02" x2="-40.64" y2="-38.1" width="0.1524" layer="91"/>
+<junction x="-45.72" y="-7.62"/>
 </segment>
 <segment>
@@
 </segment>
 </net>
-<net name="N$36" class="1">
-<segment>
-<pinref part="SW1" gate="A" pin="5"/>
-<pinref part="SW1" gate="A" pin="6"/>
-<wire x1="-25.4" y1="-35.56" x2="-25.4" y2="-38.1" width="0.1524" layer="91"/>
-<pinref part="SW1" gate="A" pin="7"/>
-<wire x1="-25.4" y1="-38.1" x2="-25.4" y2="-40.64" width="0.1524" layer="91"/>
-<junction x="-25.4" y="-38.1"/>
-<pinref part="SW1" gate="A" pin="8"/>
-<wire x1="-25.4" y1="-40.64" x2="-25.4" y2="-43.18" width="0.1524" layer="91"/>
-<junction x="-25.4" y="-40.64"/>
-<pinref part="NANO" gate="G$1" pin="5.5V"/>
-<pinref part="PH1" gate="A" pin="23"/>
-<wire x1="-27.94" y1="-7.62" x2="-20.32" y2="-7.62" width="0.1524" layer="91"/>
-<pinref part="PH1" gate="A" pin="24"/>
-<junction x="-20.32" y="-7.62"/>
-<wire x1="-20.32" y1="-7.62" x2="-15.24" y2="-7.62" width="0.1524" layer="91"/>
-<wire x1="-40.64" y1="-38.1" x2="-35.56" y2="-38.1" width="0.1524" layer="91"/>
-<wire x1="-35.56" y1="-38.1" x2="-35.56" y2="-7.62" width="0.1524" layer="91"/>
-<wire x1="-35.56" y1="-7.62" x2="-27.94" y2="-7.62" width="0.1524" layer="91"/>
-<junction x="-27.94" y="-7.62"/>
-<wire x1="-25.4" y1="-38.1" x2="-27.94" y2="-38.1" width="0.1524" layer="91"/>
-<junction x="-35.56" y="-38.1"/>
-<wire x1="-27.94" y1="-38.1" x2="-35.56" y2="-38.1" width="0.1524" layer="91"/>
-<pinref part="POWER" gate="J$1" pin="2"/>
-</segment>
-</net>

Commit message: proto board update
Parts:
- added C3.3, C5: (no value), rcl:C-EUC0805
- added I2C_1: (no value), SparkFun-Connectors:CONN_04LOCK
- added R3, R4, R5, R6: 10k, rcl:R-US_R2012
- added REG3.3: REG1117, burr-brown:REG1117
- 3.3V: device SparkFun-Connectors:CONN_04LOCK -> SparkFun-Connectors:CONN_03LOCK
- NANO: value NANO -> ARDUINO-NANO-3.0; device Arduino-clone:NANO -> diy-modules:ARDUINO-NANO-3.0
Connections:
- net N$1 renamed M1
- net N$12 renamed M0
- net N$15 renamed ES32_TXD
- net N$22 renamed ES32_AUX
- net N$38 renamed ES32_RXD
- removed net SDA_GY521: NANO.A4, PH1.15, PH1.16
- new net SDA: I2C_1.4, NANO.A4, PH1.15, PH1.16
- net 3.3V: now also C3.3.2, NANO.3V3, REG3.3.VOUT; no longer 3.3V.4, NANO.3.3V
- net 5V: now also C5.1, I2C_1.2, NANO.5V, REG3.3.VIN; no longer NANO.5.5V
- net A5: now also I2C_1.3
- net GND: now also C3.3.1, C5.2, I2C_1.1, NANO.GND.2, R3.1, R4.1, R5.1, R6.1, REG3.3.GND; no longer NANO.GND, NANO.ICSP6
- net MISO_NRF: now also NANO.GND.1; no longer NANO.GND2
- net N$16: now also NANO.D12/MISO; no longer NANO.D12
- net N$17: now also NANO.D11/MOSI; no longer NANO.D11
- net N$28: now also NANO.RST.1; no longer NANO.RST1
- net N$29: now also NANO.D0/RX; no longer NANO.RX1
- net N$30: now also NANO.D1/TX; no longer NANO.TX0
- net N$39: now also R3.2
- net N$40: now also R4.2
- net N$41: now also R5.2
- net N$42: now also R6.2
- net RST: now also NANO.RST.2; no longer NANO.RST
- net SCK_NRF: now also NANO.D13/SCK; no longer NANO.D13
- net VIN: now also NANO.VIN; no longer NANO.RAW
Other:
- moved on the sheet: MICRO_1, MICRO_2

Commit message: IMU + proto board update
Parts:
- removed R3, R4, R5, R6: 10k, rcl:R-US_R2012
Connections:
- net 3.3V: now also NRF24L01.VCC
- net 5V: no longer NRF24L01.VCC, SW1.5, SW1.6, SW1.7, SW1.8
- net GND: now also SW1.5, SW1.6, SW1.7, SW1.8; no longer R3.1, R4.1, R5.1, R6.1
- net N$39: no longer R3.2
- net N$40: no longer R4.2
- net N$41: no longer R5.2
- net N$42: no longer R6.2
Other:
- moved on the sheet: J4, PIN1, SW1, T1_5MM
Changed lines of the file:
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@@
 <parts>
 <part name="ES32-433T20D" library="SparkFun-Connectors" library_urn="urn:adsk.eagle:library:513" deviceset="CONN_07" device="LOCK" package3d_urn="urn:adsk.eagle:package:38132/1"/>
-<part name="SUPPLY2" library="SparkFun-PowerSymbols" library_urn="urn:adsk.eagle:library:530" deviceset="5V" device=""/>
 <part name="GND1" library="SparkFun-PowerSymbols" library_urn="urn:adsk.eagle:library:530" deviceset="GND" device=""/>
 <part name="GND3" library="SparkFun-PowerSymbols" library_urn="urn:adsk.eagle:library:530" deviceset="GND" device=""/>
@@
 <part name="GND7" library="SparkFun-PowerSymbols" library_urn="urn:adsk.eagle:library:530" deviceset="GND" device=""/>
 <part name="SUPPLY8" library="SparkFun-PowerSymbols" library_urn="urn:adsk.eagle:library:530" deviceset="3.3V" device=""/>
-<part name="R3" library="rcl" library_urn="urn:adsk.eagle:library:334" deviceset="R-US_" device="R2012" package3d_urn="urn:adsk.eagle:package:23543/2" value="10k"/>
-<part name="R4" library="rcl" library_urn="urn:adsk.eagle:library:334" deviceset="R-US_" device="R2012" package3d_urn="urn:adsk.eagle:package:23543/2" value="10k"/>
-<part name="R5" library="rcl" library_urn="urn:adsk.eagle:library:334" deviceset="R-US_" device="R2012" package3d_urn="urn:adsk.eagle:package:23543/2" value="10k"/>
-<part name="R6" library="rcl" library_urn="urn:adsk.eagle:library:334" deviceset="R-US_" device="R2012" package3d_urn="urn:adsk.eagle:package:23543/2" value="10k"/>
 </parts>
 <sheets>
@@
 <instances>
 <instance part="ES32-433T20D" gate="G$1" x="134.62" y="-20.32" rot="R180"/>
-<instance part="SUPPLY2" gate="G$1" x="91.44" y="-50.8" rot="R180"/>
-<instance part="GND1" gate="1" x="22.86" y="-45.72"/>
+<instance part="GND1" gate="1" x="81.28" y="-106.68"/>
 <instance part="GND3" gate="1" x="83.82" y="-53.34"/>
-<instance part="T1_5MM" gate="G$1" x="-68.58" y="-35.56"/>
+<instance part="T1_5MM" gate="G$1" x="-17.78" y="-53.34"/>
 <instance part="SUPPLY3" gate="G$1" x="119.38" y="-53.34" rot="R180"/>
 <instance part="J1" gate="G$1" x="96.52" y="-20.32"/>
-<instance part="PIN1" gate="G$1" x="-83.82" y="-38.1"/>
+<instance part="PIN1" gate="G$1" x="-33.02" y="-55.88"/>
 <instance part="PH1" gate="A" x="-25.4" y="2.54"/>
 <instance part="PH2" gate="A" x="25.4" y="2.54"/>
-<instance part="SW1" gate="A" x="-17.78" y="-38.1"/>
-<instance part="J4" gate="G$1" x="-2.54" y="-38.1" rot="R180"/>
+<instance part="SW1" gate="A" x="96.52" y="-93.98"/>
+<instance part="J4" gate="G$1" x="111.76" y="-93.98" rot="R180"/>
 <instance part="NRF24L01" gate="G$1" x="58.42" y="-53.34" rot="R270"/>
 <instance part="R1" gate="G$1" x="116.84" y="-10.16"/>
@@
 <instance part="GND7" gate="1" x="-20.32" y="-109.22"/>
 <instance part="SUPPLY8" gate="G$1" x="2.54" y="-106.68" rot="R180"/>
-<instance part="R3" gate="G$1" x="10.16" y="-35.56" rot="R180"/>
-<instance part="R4" gate="G$1" x="10.16" y="-38.1" rot="R180"/>
-<instance part="R5" gate="G$1" x="10.16" y="-40.64" rot="R180"/>
-<instance part="R6" gate="G$1" x="10.16" y="-43.18" rot="R180"/>
 </instances>
 <busses>
@@
 <wire x1="121.92" y1="-27.94" x2="119.38" y2="-30.48" width="0.1524" layer="91"/>
 <pinref part="SUPPLY3" gate="G$1" pin="3.3V"/>
-<wire x1="119.38" y1="-30.48" x2="119.38" y2="-53.34" width="0.1524" layer="91"/>
+<wire x1="119.38" y1="-30.48" x2="119.38" y2="-45.72" width="0.1524" layer="91"/>
+<wire x1="119.38" y1="-45.72" x2="119.38" y2="-53.34" width="0.1524" layer="91"/>
+<wire x1="91.44" y1="-27.94" x2="66.04" y2="-27.94" width="0.1524" layer="91"/>
+<pinref part="NRF24L01" gate="G$1" pin="VCC"/>
+<wire x1="66.04" y1="-27.94" x2="66.04" y2="-30.48" width="0.1524" layer="91"/>
+<wire x1="91.44" y1="-27.94" x2="91.44" y2="-45.72" width="0.1524" layer="91"/>
+<wire x1="91.44" y1="-45.72" x2="119.38" y2="-45.72" width="0.1524" layer="91"/>
+<junction x="119.38" y="-45.72"/>
 </segment>
 <segment>
@@
 <wire x1="-45.72" y1="-7.62" x2="-27.94" y2="-7.62" width="0.1524" layer="91"/>
 <junction x="-27.94" y="-7.62"/>
-<pinref part="SW1" gate="A" pin="5"/>
-<pinref part="SW1" gate="A" pin="6"/>
-<wire x1="-25.4" y1="-35.56" x2="-25.4" y2="-38.1" width="0.1524" layer="91"/>
-<pinref part="SW1" gate="A" pin="7"/>
-<wire x1="-25.4" y1="-38.1" x2="-25.4" y2="-40.64" width="0.1524" layer="91"/>
-<junction x="-25.4" y="-38.1"/>
-<pinref part="SW1" gate="A" pin="8"/>
-<wire x1="-25.4" y1="-40.64" x2="-25.4" y2="-43.18" width="0.1524" layer="91"/>
-<junction x="-25.4" y="-40.64"/>
-<wire x1="-25.4" y1="-38.1" x2="-40.64" y2="-38.1" width="0.1524" layer="91"/>
-<wire x1="-45.72" y1="-7.62" x2="-45.72" y2="-33.02" width="0.1524" layer="91"/>
-<wire x1="-45.72" y1="-33.02" x2="-40.64" y2="-38.1" width="0.1524" layer="91"/>
-<junction x="-45.72" y="-7.62"/>
 <pinref part="NANO" gate="G$1" pin="5V"/>
 <junction x="-17.78" y="-7.62"/>
 <wire x1="-17.78" y1="-7.62" x2="-20.32" y2="-7.62" width="0.1524" layer="91"/>
-</segment>
-<segment>
-<pinref part="SUPPLY2" gate="G$1" pin="5V"/>
-<wire x1="91.44" y1="-27.94" x2="91.44" y2="-50.8" width="0.1524" layer="91"/>
-<wire x1="91.44" y1="-27.94" x2="66.04" y2="-27.94" width="0.1524" layer="91"/>
-<pinref part="NRF24L01" gate="G$1" pin="VCC"/>
-<wire x1="66.04" y1="-27.94" x2="66.04" y2="-30.48" width="0.1524" layer="91"/>
 </segment>
 <segment>
@@
 </segment>
 <segment>
-<pinref part="R3" gate="G$1" pin="1"/>
+<pinref part="SW1" gate="A" pin="8"/>
+<pinref part="SW1" gate="A" pin="7"/>
+<wire x1="88.9" y1="-96.52" x2="88.9" y2="-99.06" width="0.1524" layer="91"/>
+<junction x="88.9" y="-96.52"/>
+<pinref part="SW1" gate="A" pin="6"/>
+<wire x1="88.9" y1="-93.98" x2="88.9" y2="-96.52" width="0.1524" layer="91"/>
+<junction x="88.9" y="-93.98"/>
+<pinref part="SW1" gate="A" pin="5"/>
+<wire x1="88.9" y1="-91.44" x2="88.9" y2="-93.98" width="0.1524" layer="91"/>
 <pinref part="GND1" gate="1" pin="GND"/>
-<wire x1="15.24" y1="-35.56" x2="22.86" y2="-35.56" width="0.1524" layer="91"/>
-<wire x1="22.86" y1="-35.56" x2="22.86" y2="-43.18" width="0.1524" layer="91"/>
-<pinref part="R4" gate="G$1" pin="1"/>
-<wire x1="15.24" y1="-35.56" x2="15.24" y2="-38.1" width="0.1524" layer="91"/>
-<junction x="15.24" y="-35.56"/>
-<pinref part="R5" gate="G$1" pin="1"/>
-<wire x1="15.24" y1="-38.1" x2="15.24" y2="-40.64" width="0.1524" layer="91"/>
-<junction x="15.24" y="-38.1"/>
-<pinref part="R6" gate="G$1" pin="1"/>
-<wire x1="15.24" y1="-40.64" x2="15.24" y2="-43.18" width="0.1524" layer="91"/>
-<junction x="15.24" y="-40.64"/>
+<wire x1="88.9" y1="-99.06" x2="81.28" y2="-99.06" width="0.1524" layer="91"/>
+<wire x1="81.28" y1="-99.06" x2="81.28" y2="-104.14" width="0.1524" layer="91"/>
+<junction x="88.9" y="-99.06"/>
 </segment>
 </net>
@@
 <pinref part="PIN1" gate="G$1" pin="2"/>
 <pinref part="T1_5MM" gate="G$1" pin="1"/>
-<wire x1="-76.2" y1="-35.56" x2="-73.66" y2="-33.02" width="0.1524" layer="91"/>
+<wire x1="-25.4" y1="-53.34" x2="-22.86" y2="-50.8" width="0.1524" layer="91"/>
 </segment>
 </net>
@@
 <pinref part="PIN1" gate="G$1" pin="1"/>
 <pinref part="T1_5MM" gate="G$1" pin="2"/>
-<wire x1="-76.2" y1="-38.1" x2="-73.66" y2="-38.1" width="0.1524" layer="91"/>
+<wire x1="-25.4" y1="-55.88" x2="-22.86" y2="-55.88" width="0.1524" layer="91"/>
 </segment>
 </net>
@@
 <pinref part="SW1" gate="A" pin="4"/>
 <pinref part="J4" gate="G$1" pin="1"/>
-<wire x1="-7.62" y1="-35.56" x2="-10.16" y2="-35.56" width="0.1524" layer="91"/>
-<pinref part="R3" gate="G$1" pin="2"/>
-<wire x1="-7.62" y1="-35.56" x2="5.08" y2="-35.56" width="0.1524" layer="91"/>
-<junction x="-7.62" y="-35.56"/>
+<wire x1="106.68" y1="-91.44" x2="104.14" y2="-91.44" width="0.1524" layer="91"/>
 </segment>
 </net>
@@
 <pinref part="SW1" gate="A" pin="3"/>
 <pinref part="J4" gate="G$1" pin="2"/>
-<wire x1="-7.62" y1="-38.1" x2="-10.16" y2="-38.1" width="0.1524" layer="91"/>
-<pinref part="R4" gate="G$1" pin="2"/>
-<wire x1="5.08" y1="-38.1" x2="-7.62" y2="-38.1" width="0.1524" layer="91"/>
-<junction x="-7.62" y="-38.1"/>
+<wire x1="106.68" y1="-93.98" x2="104.14" y2="-93.98" width="0.1524" layer="91"/>
 </segment>
 </net>
@@
 <pinref part="SW1" gate="A" pin="2"/>
 <pinref part="J4" gate="G$1" pin="3"/>
-<wire x1="-7.62" y1="-40.64" x2="-10.16" y2="-40.64" width="0.1524" layer="91"/>
-<pinref part="R5" gate="G$1" pin="2"/>
-<wire x1="-7.62" y1="-40.64" x2="5.08" y2="-40.64" width="0.1524" layer="91"/>
-<junction x="-7.62" y="-40.64"/>
+<wire x1="106.68" y1="-96.52" x2="104.14" y2="-96.52" width="0.1524" layer="91"/>
 </segment>
 </net>
@@
 <pinref part="SW1" gate="A" pin="1"/>
 <pinref part="J4" gate="G$1" pin="4"/>
-<wire x1="-7.62" y1="-43.18" x2="-10.16" y2="-43.18" width="0.1524" layer="91"/>
-<pinref part="R6" gate="G$1" pin="2"/>
-<wire x1="5.08" y1="-43.18" x2="-7.62" y2="-43.18" width="0.1524" layer="91"/>
-<junction x="-7.62" y="-43.18"/>
-</segment>
-</net>
+<wire x1="106.68" y1="-99.06" x2="104.14" y2="-99.06" width="0.1524" layer="91"/>
+</segment>
+</net>

Commit message: update
Parts:
- removed 5V, GND: (no value), SparkFun-Connectors:CONN_04LOCK
- added 3.3REG: JUMPER-SMT_2_NO_NO-SILK, SparkFun-Jumpers:JUMPER-SMT_2_NO_NO-SILK
- added 5.GND: (no value), SparkFun-Connectors:CONN_04X2
- C3.3, C5: value (none) -> 100nF
Connections:
- new net N$2: 3.3REG.1, C3.3.2, REG3.3.VOUT
- net 3.3V: now also 3.3REG.2; no longer C3.3.2, REG3.3.VOUT
- net 5V: now also 5.GND.2, 5.GND.4, 5.GND.6, 5.GND.8; no longer 5V.1, 5V.2, 5V.3, 5V.4, I2C_1.2
- net A5: now also I2C_1.1
- net GND: now also 5.GND.1, 5.GND.3, 5.GND.5, 5.GND.7; no longer GND.1, GND.2, GND.3, GND.4, I2C_1.1
- net SDA: now also I2C_1.2
