File: _PCB/_Prototyping Boards/NANO.ProMini_MINI prototype board/board.sch (EAGLE design)
At the start: 26 parts, among them T1_5MM 5mm

Commit message: prototype board complete
Parts:
- removed R2: 4.7k, rcl:R-US_R2012
- added 3.3V_C1: (no value), rcl:CPOL-EUD
- added MICRO_3: (no value), SparkFun-Connectors:USB_MICRO-B_SMT
- renumbered 3.3V to 3V3, ES32-433T20D to ES32-TTL
Connections:
- net A5 renamed SCL
- net 3.3V: now also 3.3V_C1.+
- net 5V: now also MICRO_3.VBUS
- net GND: now also 3.3V_C1.-, MICRO_3.GND
Other:
- moved on the sheet: MICRO_1, MICRO_2
