File: _PCB/_Prototyping Boards/IM_L400_prototype board/schematics.brd (EAGLE design)
At the start: 29.7 x 21.8 mm, 10 parts

Commit message: IM-L400 prototype board
Parts:
- removed C2: (no value), rcl:C0805
- removed J3: (no value), SparkFun-Connectors:1X04_LOCK
- removed R1, R2, R3, R4: 4.7k, rcl:R2012
- added RST, WAKE: 6.0X3.5mm, SparkFun-Switches:TACTILE_SWITCH_SMD_6.0X3.5MM
- moved C1 7.74 mm to (21.3, 6.86), turned to 0 degrees
- moved J1 5.85 mm to (25.9, 20.3)
- moved U$1 5.09 mm to (13.7, 13.7)
- moved J2 3.30 mm to (1.78, 5.08)
Connections:
- removed net N$14: J3.3, R2.2
- removed net N$15: J3.2, R3.2
- removed net N$16: J3.1, R4.2
- removed net N$4: J3.4, R1.2
- net GND: now also RST.2, WAKE.2; no longer C2.1
- net N$10: no longer R1.1
- net N$12: now also RST.1
- net N$2: no longer R4.1
- net N$3: no longer R3.1
- net N$6: now also WAKE.1
- net N$9: no longer R2.1
- net VCC: no longer C2.2
Routing:
- net N$6: track 3.27 -> 22.3 mm, vias 0 -> 1
- net N$12: track 3.84 -> 19.8 mm, vias 0 -> 1
- net N$2: track 19.2 -> 3.94 mm, vias 1 -> 0
- net N$9: track 16.5 -> 3.72 mm
- net N$3: track 14.6 -> 3.47 mm
- net N$10: track 13.8 -> 3.22 mm
- net N$15: track 8.35 -> 0.00 mm
- net N$16: track 8.03 -> 0.00 mm
- net N$14: track 7.81 -> 0.00 mm
- net N$4: track 7.48 -> 0.00 mm
- net VCC: track 34.1 -> 29.2 mm
- net N$13: track 4.34 -> 3.52 mm
Other:
- board size 29.7 x 21.8 mm -> 27.4 x 21.8 mm
