File: _PCB/LoRa_Node/board.brd (EAGLE design)
At the start: 79.9 x 70 mm, 24 parts

Commit message: prototype board complete
Parts:
- moved H2 70.1 mm to (39.1, -14.2), turned to 180 degrees
Routing:
- net GND: track 0.00 -> 142.9 mm
- net 5V: track 0.00 -> 96.8 mm
- net 3.3V: track 0.00 -> 51.2 mm
- net N$2: track 0.00 -> 18.3 mm
- net N$1: track 0.00 -> 7.54 mm
- net N$11: track 0.00 -> 2.61 mm
- net N$16: track 0.00 -> 2.61 mm
- net N$5: track 0.00 -> 2.60 mm
- net N$32: track 0.00 -> 2.60 mm
- net N$28: track 0.00 -> 2.59 mm
- net N$27: track 0.00 -> 2.58 mm
- net N$15: track 0.00 -> 2.58 mm
- net N$12: track 0.00 -> 2.58 mm
- net N$33: track 0.00 -> 2.57 mm
- net N$6: track 0.00 -> 2.57 mm
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Other:
- board size 79.9 x 70 mm -> 79.9 x 76.3 mm

Commit message: PCB update
Parts:
- added J4: (no value), SparkFun-Connectors:1X04_LOCK
- added SW1: (no value), special:EDG-04
- moved H2 89.2 mm to (123.4, 15.0), turned to 270 degrees
Connections:
- new net N$39: J4.1, SW1.4
- new net N$40: J4.2, SW1.3
- new net N$41: J4.3, SW1.2
- new net N$42: J4.4, SW1.1
- net GND: now also SW1.5, SW1.6, SW1.7, SW1.8
Changed lines of the file:
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@@
 <text x="53.848" y="1.27" size="1.4224" layer="21" font="vector" rot="R180">1</text>
 <text x="68.072" y="1.27" size="1.4224" layer="21" font="vector" rot="R180">5</text>
-<wire x1="73.406" y1="-24.13" x2="5.334" y2="-24.13" width="0.1524" layer="21"/>
-<wire x1="5.334" y1="-24.13" x2="5.334" y2="-5.334" width="0.1524" layer="21"/>
-<wire x1="5.334" y1="-5.334" x2="73.406" y2="-5.334" width="0.1524" layer="21"/>
-<wire x1="73.406" y1="-5.334" x2="73.406" y2="-24.13" width="0.1524" layer="21"/>
-<text x="72.136" y="-20.066" size="2.54" layer="21" font="vector" rot="R180">18650</text>
+<wire x1="133.35" y1="49.276" x2="133.35" y2="-18.796" width="0.1524" layer="21"/>
+<wire x1="133.35" y1="-18.796" x2="114.554" y2="-18.796" width="0.1524" layer="21"/>
+<wire x1="114.554" y1="-18.796" x2="114.554" y2="49.276" width="0.1524" layer="21"/>
+<wire x1="114.554" y1="49.276" x2="133.35" y2="49.276" width="0.1524" layer="21"/>
+<text x="129.286" y="48.006" size="2.54" layer="21" font="vector" rot="R270">18650</text>
 <text x="75.946" y="48.006" size="2.54" layer="21" font="vector" rot="R270">GP2Y1023AU0F</text>
 </plain>
@@
 </class>
 <class number="1" name="power" width="0.762" drill="0">
-<clearance class="0" value="0.205"/>
 <clearance class="1" value="0.254"/>
 </class>
@@
 <attribute name="VALUE" x="54.2036" y="-1.397" size="0.6096" layer="27" font="vector" ratio="20"/>
 </element>
-<element name="H2" library="holes" package="2,8" value="18650" x="39.116" y="-14.224" smashed="yes" rot="R180"/>
+<element name="H2" library="holes" package="2,8" value="18650" x="123.444" y="14.986" smashed="yes" rot="R270"/>
 <element name="H3" library="holes" package="3,0" value="ANT" x="38.1" y="2.54" smashed="yes"/>
+<element name="SW1" library="special" library_urn="urn:adsk.eagle:library:367" package="EDG-04" package3d_urn="urn:adsk.eagle:package:26655/2" value="" x="10.16" y="-1.27" smashed="yes">
+<attribute name="NAME" x="4.318" y="4.064" size="1.27" layer="25" ratio="10"/>
+<attribute name="VALUE" x="4.318" y="-7.874" size="1.27" layer="27" ratio="10"/>
+</element>
+<element name="J4" library="SparkFun-Connectors" library_urn="urn:adsk.eagle:library:513" package="1X04_LOCK" package3d_urn="urn:adsk.eagle:package:38089/1" value="" x="13.97" y="-8.89" smashed="yes" rot="R180">
+<attribute name="NAME" x="15.24" y="-10.287" size="0.6096" layer="25" font="vector" ratio="20" rot="R180"/>
+<attribute name="PROD_ID" value="CONN-09696" x="26.67" y="-22.86" size="1.778" layer="27" rot="R180" display="off"/>
+<attribute name="VALUE" x="15.24" y="-6.858" size="0.6096" layer="27" font="vector" ratio="20" rot="R180"/>
+</element>
 </elements>
 <signals>
-<signal name="GND">
+<signal name="GND" class="1">
 <contactref element="GP2Y10" pad="3"/>
 <contactref element="GP2Y10" pad="2"/>
@@
 <wire x1="44.3176" y1="18.9422" x2="44.45" y2="19.05" width="0.1524" layer="16"/>
 <wire x1="21.6227" y1="3.9314" x2="21.59" y2="3.81" width="0.1524" layer="16"/>
-</signal>
-<signal name="5V">
+<contactref element="SW1" pad="8"/>
+<contactref element="SW1" pad="7"/>
+<contactref element="SW1" pad="6"/>
+<contactref element="SW1" pad="5"/>
+<wire x1="13.97" y1="2.54" x2="18.9422" y2="3.9314" width="0" layer="19" extent="16-16"/>
+<wire x1="11.43" y1="2.54" x2="13.97" y2="2.54" width="0" layer="19" extent="1-1"/>
+<wire x1="8.89" y1="2.54" x2="11.43" y2="2.54" width="0" layer="19" extent="1-1"/>
+<wire x1="6.35" y1="2.54" x2="8.89" y2="2.54" width="0" layer="19" extent="1-1"/>
+</signal>
+<signal name="5V" class="1">
 <contactref element="GP2Y10" pad="5"/>
 <contactref element="R1" pad="2"/>
@@
 <wire x1="44.3176" y1="16.6191" x2="44.45" y2="16.51" width="0.1524" layer="1"/>
 </signal>
-<signal name="N$2">
+<signal name="N$2" class="1">
 <contactref element="R1" pad="1"/>
 <contactref element="C6" pad="+"/>
@@
 <wire x1="21.444" y1="31.8086" x2="21.59" y2="31.75" width="0.1524" layer="1"/>
 </signal>
-<signal name="3.3V">
+<signal name="3.3V" class="1">
 <contactref element="JP2" pad="3"/>
 <contactref element="JP2" pad="4"/>
@@
 <wire x1="55.5757" y1="-1.787" x2="55.472" y2="-1.902" width="0.1524" layer="1"/>
 </signal>
+<signal name="N$39" class="1">
+<contactref element="SW1" pad="4"/>
+<contactref element="J4" pad="1"/>
+<wire x1="13.97" y1="-9.017" x2="13.97" y2="-5.08" width="0" layer="19" extent="1-1"/>
+</signal>
+<signal name="N$40" class="1">
+<contactref element="SW1" pad="3"/>
+<contactref element="J4" pad="2"/>
+<wire x1="11.43" y1="-8.763" x2="11.43" y2="-5.08" width="0" layer="19" extent="1-1"/>
+</signal>
+<signal name="N$41" class="1">
+<contactref element="SW1" pad="2"/>
+<contactref element="J4" pad="3"/>
+<wire x1="8.89" y1="-9.017" x2="8.89" y2="-5.08" width="0" layer="19" extent="1-1"/>
+</signal>
+<signal name="N$42" class="1">
+<contactref element="SW1" pad="1"/>
+<contactref element="J4" pad="4"/>
+<wire x1="6.35" y1="-5.08" x2="6.35" y2="-8.763" width="0" layer="19" extent="1-1"/>
+</signal>
 </signals>

Commit message: LoRa update
Parts:
- added JP4, JP5, JP6, JP7: (no value), SparkFun-Jumpers:SMT-JUMPER_2_NC_TRACE_SILK
- moved H2 86.8 mm to (43.4, -18.8), turned to 0 degrees
- moved J4 15.9 mm to (6.35, 5.08), turned to 0 degrees
- moved BME280_4-6 1.93 mm to (7.11, 13.2)
- moved BME280_1-3 1.93 mm to (7.11, 20.8)
- moved C9 1.30 mm to (7.87, 26.7)
- moved C2 1.27 mm to (11.4, 45.5)
- moved C3 1.27 mm to (4.32, 45.5)
- moved SW1 1.27 mm to (10.2, -2.54), turned to 180 degrees
- moved C1 1.27 mm to (11.4, 37.8)
- moved C8 1.27 mm to (4.32, 37.8), turned to 90 degrees
Connections:
- net N$14: now also JP6.2
- net N$15: now also JP7.2
- net N$18: now also JP5.2
- net N$19: now also JP4.2
- net N$3: now also BME280_4-6.1
- net N$39: now also JP4.1
- net N$40: now also JP5.1
- net N$41: now also JP6.1
- net N$42: now also JP7.1
- net N$6: now also BME280_1-3.3
Routing:
- net GND: track 142.9 -> 0.00 mm
- net 5V: track 96.8 -> 0.00 mm
- net 3.3V: track 51.2 -> 0.00 mm
- net N$2: track 18.3 -> 0.00 mm
- net N$1: track 7.54 -> 0.00 mm
- net N$11: track 2.61 -> 0.00 mm
- net N$16: track 2.61 -> 0.00 mm
- net N$5: track 2.60 -> 0.00 mm
- net N$32: track 2.60 -> 0.00 mm
- net N$28: track 2.59 -> 0.00 mm
- net N$27: track 2.58 -> 0.00 mm
- net N$15: track 2.58 -> 0.00 mm
- net N$20: track 2.58 -> 0.00 mm
- net N$33: track 2.57 -> 0.00 mm
- net N$6: track 2.57 -> 0.00 mm
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- added copper zone on layer 1, net GND
- added copper zone on layer 16, net GND
Other:
- board size 79.9 x 76.3 mm -> 79.9 x 78.9 mm
- board text added: "12"
- board text added: "14"
- board text added: "32"
- board text added: "33"
- board text added: "GND"
- board text added: "NCS"
- board text added: "SCL"
- board text added: "SDA"
- board text added: "SDO"
- board text added: "VCC"
