File: _PCB/LoRa_Node/board.sch (EAGLE design)
At the start: 24 parts

Commit message: PCB update
Parts:
- added J4: (no value), SparkFun-Connectors:CONN_04LOCK
- added SW1: (no value), special:SW_DIP-4
Connections:
- new net N$39: J4.1, SW1.4
- new net N$40: J4.2, SW1.3
- new net N$41: J4.3, SW1.2
- new net N$42: J4.4, SW1.1
- net GND: now also SW1.5, SW1.6, SW1.7, SW1.8
Changed lines of the file:
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@@
 <?xml version="1.0" encoding="utf-8"?>
 <!DOCTYPE eagle SYSTEM "eagle.dtd">
-<eagle version="9.2.1">
+<eagle version="9.2.2">
 <drawing>
 <settings>
@@
 <setting verticaltext="up"/>
 </settings>
-<grid distance="0.05" unitdist="inch" unit="inch" style="lines" multiple="1" display="no" altdistance="0.01" altunitdist="inch" altunit="inch"/>
+<grid distance="0.1" unitdist="inch" unit="inch" style="lines" multiple="1" display="no" altdistance="0.01" altunitdist="inch" altunit="inch"/>
 <layers>
 <layer number="1" name="Top" color="4" fill="1" visible="no" active="no"/>
@@
 </class>
 <class number="1" name="power" width="0.762" drill="0">
-<clearance class="0" value="0.205"/>
 <clearance class="1" value="0.254"/>
 </class>
@@
 <part name="H2" library="holes" deviceset="MOUNT-HOLE" device="2.8" value="18650"/>
 <part name="H3" library="holes" deviceset="MOUNT-HOLE" device="3.0" value="ANT"/>
+<part name="GND7" library="SparkFun-PowerSymbols" library_urn="urn:adsk.eagle:library:530" deviceset="GND" device=""/>
+<part name="SW1" library="special" library_urn="urn:adsk.eagle:library:367" deviceset="SW_DIP-4" device="" package3d_urn="urn:adsk.eagle:package:26655/2"/>
+<part name="J4" library="SparkFun-Connectors" library_urn="urn:adsk.eagle:library:513" deviceset="CONN_04" device="LOCK" package3d_urn="urn:adsk.eagle:package:38089/1"/>
 </parts>
 <sheets>
@@
 <attribute name="VALUE" x="250.952" y="153.7462" size="1.778" layer="96"/>
 </instance>
+<instance part="GND7" gate="1" x="185.42" y="149.86" smashed="yes">
+<attribute name="VALUE" x="185.42" y="149.606" size="1.778" layer="96" align="top-center"/>
+</instance>
+<instance part="SW1" gate="A" x="200.66" y="162.56" smashed="yes">
+<attribute name="NAME" x="195.58" y="168.275" size="1.778" layer="95"/>
+<attribute name="VALUE" x="195.58" y="152.4" size="1.778" layer="96"/>
+</instance>
+<instance part="J4" gate="G$1" x="215.9" y="162.56" smashed="yes" rot="R180">
+<attribute name="VALUE" x="220.98" y="169.926" size="1.778" layer="96" font="vector" rot="R180"/>
+<attribute name="NAME" x="220.98" y="154.432" size="1.778" layer="95" font="vector" rot="R180"/>
+</instance>
 </instances>
 <busses>
 </busses>
 <nets>
-<net name="GND" class="0">
+<net name="GND" class="1">
 <segment>
 <pinref part="GP2Y10" gate="G$1" pin="3"/>
@@
 <junction x="69.85" y="83.82"/>
 </segment>
-</net>
-<net name="5V" class="0">
+<segment>
+<pinref part="SW1" gate="A" pin="8"/>
+<pinref part="SW1" gate="A" pin="7"/>
+<wire x1="193.04" y1="160.02" x2="193.04" y2="157.48" width="0.1524" layer="91"/>
+<junction x="193.04" y="160.02"/>
+<pinref part="SW1" gate="A" pin="6"/>
+<wire x1="193.04" y1="162.56" x2="193.04" y2="160.02" width="0.1524" layer="91"/>
+<junction x="193.04" y="162.56"/>
+<pinref part="SW1" gate="A" pin="5"/>
+<wire x1="193.04" y1="165.1" x2="193.04" y2="162.56" width="0.1524" layer="91"/>
+<pinref part="GND7" gate="1" pin="GND"/>
+<wire x1="193.04" y1="157.48" x2="185.42" y2="157.48" width="0.1524" layer="91"/>
+<wire x1="185.42" y1="157.48" x2="185.42" y2="152.4" width="0.1524" layer="91"/>
+<junction x="193.04" y="157.48"/>
+</segment>
+</net>
+<net name="5V" class="1">
 <segment>
 <pinref part="SUPPLY10" gate="G$1" pin="5V"/>
@@
 </segment>
 </net>
-<net name="N$2" class="0">
+<net name="N$2" class="1">
 <segment>
 <pinref part="R1" gate="G$1" pin="1"/>
@@
 </segment>
 </net>
-<net name="3.3V" class="0">
+<net name="3.3V" class="1">
 <segment>
 <pinref part="JP2" gate="A" pin="3"/>
@@
 </segment>
 </net>
+<net name="N$39" class="1">
+<segment>
+<pinref part="SW1" gate="A" pin="4"/>
+<pinref part="J4" gate="G$1" pin="1"/>
+<wire x1="210.82" y1="165.1" x2="208.28" y2="165.1" width="0.1524" layer="91"/>
+</segment>
+</net>
+<net name="N$40" class="1">
+<segment>
+<pinref part="SW1" gate="A" pin="3"/>
+<pinref part="J4" gate="G$1" pin="2"/>
+<wire x1="210.82" y1="162.56" x2="208.28" y2="162.56" width="0.1524" layer="91"/>
+</segment>
+</net>
+<net name="N$41" class="1">
+<segment>
+<pinref part="SW1" gate="A" pin="2"/>
+<pinref part="J4" gate="G$1" pin="3"/>
+<wire x1="210.82" y1="160.02" x2="208.28" y2="160.02" width="0.1524" layer="91"/>
+</segment>
+</net>
+<net name="N$42" class="1">
+<segment>
+<pinref part="SW1" gate="A" pin="1"/>
+<pinref part="J4" gate="G$1" pin="4"/>
+<wire x1="210.82" y1="157.48" x2="208.28" y2="157.48" width="0.1524" layer="91"/>
+</segment>
+</net>

Commit message: LoRa update
Parts:
- added JP4, JP5, JP6, JP7: JUMPER-SMT_2_NC_TRACE_SILK, SparkFun-Jumpers:JUMPER-SMT_2_NC_TRACE_SILK
Connections:
- net N$14: now also JP6.2
- net N$15: now also JP7.2
- net N$18: now also JP5.2
- net N$19: now also JP4.2
- net N$3: now also BME280_4-6.1
- net N$39: now also JP4.1
- net N$40: now also JP5.1
- net N$41: now also JP6.1
- net N$42: now also JP7.1
- net N$6: now also BME280_1-3.3
Other:
- moved on the sheet: ESP32, H1, H2, H3, J4, REFERENCE, SW1
