File: _PCB/MAKER_LoRa_Node/board.brd (EAGLE design)
At the start: 51.7 x 93.4 mm, 37 parts

Commit message: LoRa update
Parts:
- removed CER: 100nF, rcl:C0805
- removed DIP1: (no value), rcl:0204/7
- removed EL: (no value), rcl:E2,5-5
- removed GP2Y10_1, REFERENCE: (no value), SparkFun-Connectors:1X05
- removed H2: 18650, holes:2,8
- removed H3: ANT, holes:3,0
- removed H4, H5, H6, H7: MOUNT-HOLE3.0, holes:3,0
- removed J4: (no value), SparkFun-Connectors:1X04_LOCK
- removed POWER: (no value), SparkFun-Connectors:2X3
- removed SMD1: (no value), rcl:PANASONIC_D
- added JP8, JP9: (no value), pinhead_v2:2X02
- moved MICRO_1 199.0 mm to (46.0, -2.79), flipped to the bottom, turned to 180 degrees
- moved MICRO_2 171.5 mm to (4.06, -3.81), flipped to the bottom
- moved MICRO_3 54.4 mm to (4.19, 12.8), turned to 180 degrees
- moved JP1 43.8 mm to (45.6, 40.9), turned to 180 degrees
- moved C6 40.2 mm to (46.4, 24.5)
- moved SW1 36.6 mm to (7.11, 38.6), turned to 90 degrees
- moved GP2Y10 27.3 mm to (46.9, 19.2), turned to 270 degrees
- moved JP5 24.3 mm to (20.3, 38.4), turned to 0 degrees
- moved JP6 24.3 mm to (20.3, 35.8), turned to 0 degrees
- moved JP7 24.3 mm to (20.3, 33.3), turned to 0 degrees
- moved JP4 24.3 mm to (20.3, 40.9), turned to 0 degrees
- moved R1 18.3 mm to (40.5, 10.8), turned to 270 degrees
- moved C9 9.14 mm to (8.89, 24.4), turned to 0 degrees
- moved BME280_4-6 8.70 mm to (4.32, 21.3)
- moved BME280_1-3 8.70 mm to (4.32, 29.0)
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Connections:
- net 3.3V: now also JP8.1, JP8.2, JP9.1, JP9.2; no longer POWER.2, POWER.4, POWER.6
- net 5V: no longer GP2Y10_1.5
- net GND: now also JP8.3, JP8.4, JP9.3, JP9.4; no longer GP2Y10_1.2, GP2Y10_1.3, POWER.1, POWER.3, POWER.5
- net N$1: no longer J4.1
- net N$13: no longer J4.3
- net N$2: no longer J4.2
- net N$21: no longer J4.4
- net VLED: no longer GP2Y10_1.4
- net VOUT_1: no longer GP2Y10_1.1
Routing:
- net 5V: track 0.00 -> 145.8 mm, vias 0 -> 2
- net 3.3V: track 0.00 -> 113.7 mm
- net VOUT_1: track 0.00 -> 86.4 mm
- net VLED: track 0.00 -> 68.3 mm
- net SDA: track 0.00 -> 33.9 mm
- net DIP4: track 0.00 -> 30.1 mm, vias 0 -> 2
- net DIP3: track 0.00 -> 30.1 mm, vias 0 -> 2
- net DIP2: track 0.00 -> 30.1 mm, vias 0 -> 2
- net DIP1: track 0.00 -> 27.4 mm
- net SCL: track 0.00 -> 19.4 mm
- net N$21: track 0.00 -> 9.52 mm
- net N$2: track 0.00 -> 9.52 mm
- net N$13: track 0.00 -> 9.52 mm
- net N$1: track 0.00 -> 9.52 mm
- net VOUT: track 0.00 -> 5.22 mm
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Other:
- board size 51.7 x 93.4 mm -> 53.3 x 78.2 mm
- board text added: "ANT"
- board text added: "GP2Y10_HOLE"
