File: _PCB/MAKER_LoRa_Node/board.sch (EAGLE design)
At the start: 37 parts

Commit message: LoRa update
Parts:
- removed CER: 100nF, rcl:C-EUC0805
- removed DIP1: (no value), rcl:R-EU_0204/7
- removed EL: (no value), rcl:CPOL-EUE2.5-5
- removed GP2Y10_1, REFERENCE: (no value), SparkFun-Connectors:CONN_05
- removed H2: 18650, holes:MOUNT-HOLE2.8
- removed H3: ANT, holes:MOUNT-HOLE3.0
- removed H4, H5, H6, H7: MOUNT-HOLE3.0, holes:MOUNT-HOLE3.0
- removed J4: (no value), SparkFun-Connectors:CONN_04LOCK
- removed POWER: (no value), SparkFun-Connectors:CONN_03X22X3_SILK_MALE_PTH
- removed SMD1: (no value), rcl:CPOL-EUD
- added JP8, JP9: (no value), pinhead_v2:PINHD-2X2/OCT
Connections:
- net 3.3V: now also JP8.1, JP8.2, JP9.1, JP9.2; no longer POWER.2, POWER.4, POWER.6
- net 5V: no longer GP2Y10_1.5
- net GND: now also JP8.3, JP8.4, JP9.3, JP9.4; no longer GP2Y10_1.2, GP2Y10_1.3, POWER.1, POWER.3, POWER.5
- net N$1: no longer J4.1
- net N$13: no longer J4.3
- net N$2: no longer J4.2
- net N$21: no longer J4.4
- net VLED: no longer GP2Y10_1.4
- net VOUT_1: no longer GP2Y10_1.1
Other:
- moved on the sheet: GP2Y10_2, JP4, JP5, JP6, JP7
