File: _PCB/RFID_SensorTag/board.brd (EAGLE design)
At the start: 100 x 60 mm, 14 parts, among them X1 53048-02

Commit message: PCB schematic update
Parts:
- removed JP_CURRENT: (no value), pinhead:1X02
- removed OLED: (no value), SparkFun-Connectors:1X04
- added CURRENT: (no value), pinhead:1X02
- added OLED_1, OLED_2: (no value), SparkFun-Connectors:1X04
- moved C1 115.6 mm to (23.8, 49.6)
- moved C2 113.0 mm to (28.9, 49.6)
- moved M2 78.2 mm to (85.8, 16.9), turned to 180 degrees
- moved S1 72.0 mm to (86.2, 3.57)
- moved JP_GND 64.4 mm to (50.0, 47.5), turned to 0 degrees
- moved JP_VBATT 64.1 mm to (50.3, 56.1), turned to 0 degrees
- moved X1 63.3 mm to (66.3, 21.6), turned to 180 degrees
- moved JP_3V3 58.7 mm to (62.2, 56.1), turned to 0 degrees
- moved BAT- 51.7 mm to (65.3, 33.8), turned to 270 degrees
- moved U$1 49.9 mm to (35.2, 52.5)
- moved BAT+ 49.0 mm to (65.3, 30.0), turned to 270 degrees
Connections:
- removed net N$3: BAT+.1, M2.B+
- removed net N$4: BAT-.1, M2.B-
- new net BATT+: BAT+.1, M2.B+, X1.1
- new net BATT-: BAT-.1, M2.B-, X1.2
- net 5V: now also OLED_1.3, OLED_2.4; no longer OLED.3
- net GND: now also OLED_1.4, OLED_2.3; no longer OLED.4
- net I2C_SCL: now also OLED_1.2, OLED_2.2; no longer OLED.2
- net I2C_SDA: now also OLED_1.1, OLED_2.1; no longer OLED.1
- net N$1: now also CURRENT.2; no longer JP_CURRENT.2
- net N$2: now also CURRENT.1; no longer JP_CURRENT.1

Commit message: PCB ver1
Parts:
- removed BAT+, BAT-: (no value), pinhead_v2:1X01
- added C3: 100nF, rcl:C0805
- added JP_BATT: (no value), pinhead:1X02
- added JP_BATT_EN: (no value), SparkFun-Jumpers:SMT-JUMPER_2_NC_PASTE_SILK
- added U1: MAXIM_ELECTRONICS_MAX40200AUK+MAXIM_ELECTRONICS_MAX40200AUK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, Maxim Electronics - MAX40200AUK+:MAXIM_ELECTRONICS_MAX40200AUK+_0
- moved JP_3V3 58.2 mm to (24.6, 11.7), turned to 180 degrees
- moved JP_VBATT 46.1 mm to (24.6, 17.8), turned to 180 degrees
- moved JP_GND 34.3 mm to (24.6, 24.4), turned to 180 degrees
- moved X1 31.4 mm to (57.9, 51.8)
- moved S1 16.8 mm to (69.4, 4.05), turned to 90 degrees
- moved M2 8.00 mm to (77.8, 16.9)
- moved OLED_1 8.00 mm to (87.9, 38.7)
- moved OLED_2 8.00 mm to (65.8, 46.6)
- moved CURRENT 6.73 mm to (81.4, 5.08), turned to 0 degrees
- moved C1 3.35 mm to (26.6, 47.7), turned to 180 degrees
- moved C2 2.83 mm to (26.7, 51.3), turned to 0 degrees
- moved U$1 2.54 mm to (32.6, 52.5)
Connections:
- removed net 5V: OLED_1.3, OLED_2.4
- removed net BATT+: BAT+.1, M2.B+, X1.1
- removed net BATT-: BAT-.1, M2.B-, X1.2
- removed net N$1: CURRENT.2, M2.OUT+, S1.3
- new net BATT_VOUT: S1.2, U1.1, U1.3
- new net N$3: JP_BATT.1, JP_BATT_EN.2, X1.1
- new net N$4: CURRENT.2, S1.3
- new net N$5: JP_BATT.2, M2.B-, X1.2
- new net N$6: JP_BATT_EN.1, M2.B+
- net 3.3V: now also OLED_1.3, OLED_2.4; no longer M2.IN+
- net GND: now also C3.2, U1.2, U1.4
- net N$2: now also M2.OUT+
- net V_BATT: now also C3.1, U1.5; no longer S1.2
Routing:
- net 3.3V: track 0.00 -> 171.9 mm
- net I2C_SDA: track 0.00 -> 86.6 mm
- net I2C_SCL: track 0.00 -> 80.5 mm
- net BATT_VOUT: track 0.00 -> 74.8 mm, vias 0 -> 2
- net V_BATT: track 0.00 -> 59.6 mm, vias 0 -> 1
- net N$5: track 0.00 -> 40.0 mm
- net SPI_MISO: track 0.00 -> 38.8 mm
- net SPI_MOSI: track 0.00 -> 37.1 mm
- net N$6: track 0.00 -> 33.6 mm, vias 0 -> 1
- net SPI_SS: track 0.00 -> 31.3 mm
- net N$2: track 0.00 -> 19.1 mm
- net SPI_SCK: track 0.00 -> 18.0 mm
- net N$3: track 0.00 -> 13.1 mm
- net N$4: track 0.00 -> 12.4 mm
- net GND: track 0.00 -> 0.81 mm, vias 0 -> 27
- added copper zone on layer 1, net GND
- added copper zone on layer 16, net GND
Other:
- board size 100 x 60 mm -> 92 x 60 mm
- board text added: "3.2mm 3mm/3mm spacing"

Commit message: RFID PCB v2
Parts:
- removed C3: 100nF, rcl:C0805
- removed JP_BATT, JP_VBATT: (no value), pinhead:1X02
- added BATT, JP_VBATT/5V: (no value), pinhead:1X02
- added C4: 100nF, rcl:C0805
- moved X1 49.3 mm to (82.5, 9.14), turned to 90 degrees
- moved JP_3V3 47.1 mm to (59.2, 43.7)
- moved JP_GND 47.1 mm to (59.2, 56.4)
- moved JP_BATT_EN 45.7 mm to (80.3, 3.56), turned to 0 degrees
- moved U1 29.2 mm to (64.3, 24.6), turned to 180 degrees
- moved OLED_2 19.1 mm to (82.4, 56.1), turned to 180 degrees
- moved OLED_1 14.2 mm to (74.5, 34.1), turned to 0 degrees
- moved CURRENT 11.9 mm to (69.5, 4.06), turned to 180 degrees
- moved M2 5.97 mm to (81.3, 21.7)
- moved S1 4.35 mm to (69.4, 8.40), turned to 270 degrees
- moved C1 3.63 mm to (26.7, 51.3), turned to 0 degrees
- moved C2 3.63 mm to (26.6, 47.7), turned to 180 degrees
Connections:
- new net BUZZER: U$1.D8
- new net RFID_RST: M1.RST, U$1.D9
- net 3.3V: now also C1.1; no longer C2.1
- net GND: now also C4.2; no longer C3.2
- net N$3: now also BATT.1; no longer JP_BATT.1
- net N$5: now also BATT.2; no longer JP_BATT.2
- net V_BATT: now also C2.1, C4.1, JP_VBATT/5V.1, JP_VBATT/5V.2; no longer C1.1, C3.1, JP_VBATT.1, JP_VBATT.2
Routing:
- net BATT_VOUT: track 74.8 -> 17.0 mm, vias 2 -> 0
- net RFID_RST: track 0.00 -> 49.3 mm
- net 3.3V: track 171.9 -> 134.8 mm, vias 0 -> 1
- net BUZZER: track 0.00 -> 33.4 mm, vias 0 -> 1
- net V_BATT: track 59.6 -> 73.4 mm, vias 1 -> 0
- net N$6: track 33.6 -> 20.5 mm, vias 1 -> 0
- net N$5: track 40.0 -> 29.0 mm
- net N$3: track 13.1 -> 22.4 mm
- net I2C_SDA: track 86.6 -> 79.7 mm, vias 0 -> 1
- net N$4: track 12.4 -> 6.65 mm
- net N$2: track 19.1 -> 13.6 mm
- net I2C_SCL: track 80.5 -> 77.7 mm
- net SPI_SCK: track 18.0 -> 16.5 mm
- net SPI_MOSI: track 37.1 -> 37.6 mm
- net GND: track 0.81 -> 1.31 mm, vias 27 -> 41
Other:
- board size 92 x 60 mm -> 95 x 60 mm

Commit message: RFID tag PCB first production
Routing:
- net GND: vias 41 -> 45
Other:
- board text added: "3mm/3mm spacing"
- board text added: "OFF"
- board text added: "ON"
- board text removed: "3.2mm 3mm/3mm spacing"
Changed lines of the file:
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@@
 <setting verticaltext="up"/>
 </settings>
-<grid distance="20" unitdist="mil" unit="mil" style="lines" multiple="1" display="yes" altdistance="5" altunitdist="mil" altunit="mil"/>
+<grid distance="10" unitdist="mil" unit="mil" style="lines" multiple="1" display="yes" altdistance="5" altunitdist="mil" altunit="mil"/>
 <layers>
 <layer number="1" name="Top" color="4" fill="1" visible="yes" active="yes"/>
@@
 <hole x="92" y="3" drill="3.2"/>
 <hole x="92" y="57" drill="3.2"/>
-<text x="1.43" y="50.084" size="1.27" layer="21" font="vector" align="top-left">3.2mm
-3mm/3mm spacing</text>
+<text x="1.43" y="50.084" size="1.27" layer="21" font="vector" align="top-left">3mm/3mm spacing</text>
 <dimension x1="95" y1="60" x2="0" y2="60" x3="47.5" y3="33" textsize="1.27" layer="21" dtype="vertical"/>
 <dimension x1="94.2" y1="0" x2="94.2" y2="60" x3="44.832" y3="30" textsize="1.27" layer="21" dtype="vertical"/>
@@
 <wire x1="95" y1="2" x2="93" y2="0" width="0.1524" layer="20" curve="-90"/>
 <wire x1="0" y1="2" x2="2" y2="0" width="0.1524" layer="20" curve="90"/>
-<dimension x1="3" y1="3" x2="0" y2="7" x3="1.5" y3="8" textsize="1.27" layer="21" dtype="horizontal"/>
 <dimension x1="4.6" y1="57" x2="1.4" y2="57" x3="3" y3="53" textsize="1.27" layer="21" dtype="diameter"/>
 <circle x="50.1" y="52.908" radius="4.2" width="0.5" layer="21"/>
 <wire x1="48.3" y1="53.308" x2="48.3" y2="54.708" width="0.3" layer="21"/>
 <wire x1="47.6" y1="54.008" x2="49" y2="54.008" width="0.3" layer="21"/>
+<text x="74.676" y="10.922" size="1.651" layer="21" font="vector" rot="R180" align="top-left">ON</text>
+<text x="67.31" y="10.922" size="1.651" layer="21" font="vector" rot="R180" align="top-left">OFF</text>
 </plain>
 <attributes>
@@
 <via x="68.024" y="24.638" extent="1-16" drill="0.35" shape="octagon"/>
 <via x="68.024" y="26.162" extent="1-16" drill="0.35" shape="octagon"/>
+<via x="28.448" y="17.478" extent="1-16" drill="0.35" shape="octagon"/>
+<via x="28.448" y="21.288" extent="1-16" drill="0.35" shape="octagon"/>
+<via x="25.4" y="17.478" extent="1-16" drill="0.35" shape="octagon"/>
+<via x="25.4" y="21.288" extent="1-16" drill="0.35" shape="octagon"/>
 </signal>
 <signal name="V_BATT" class="1">
@@
 </drawing>
 <compatibility>
-<note version="6.3" minversion="6.2.2" severity="warning">
-Since Version 6.2.2 text objects can contain more than one line,
-which will not be processed correctly with this version.
-</note>
 <note version="8.2" severity="warning">
 Since Version 8.2, EAGLE supports online libraries. The ids

Commit message: RFID system update
Routing:
- net GND: track 1.31 -> 19.6 mm
Other:
- board text added: "B+"
- board text added: "B-"
Changed lines of the file:
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@@
 <text x="74.676" y="10.922" size="1.651" layer="21" font="vector" rot="R180" align="top-left">ON</text>
 <text x="67.31" y="10.922" size="1.651" layer="21" font="vector" rot="R180" align="top-left">OFF</text>
+<wire x1="4.826" y1="57.658" x2="4.826" y2="59.182" width="0.3048" layer="22"/>
+<wire x1="4.826" y1="59.182" x2="17.272" y2="59.182" width="0.3048" layer="22"/>
+<wire x1="17.272" y1="59.182" x2="17.272" y2="57.658" width="0.3048" layer="22"/>
+<wire x1="4.826" y1="42.164" x2="4.826" y2="40.64" width="0.3048" layer="22"/>
+<wire x1="4.826" y1="40.64" x2="9.652" y2="40.64" width="0.3048" layer="22"/>
+<wire x1="9.652" y1="40.64" x2="9.652" y2="42.164" width="0.3048" layer="22"/>
+<wire x1="22.606" y1="42.164" x2="22.606" y2="40.64" width="0.3048" layer="22"/>
+<wire x1="22.606" y1="40.64" x2="27.432" y2="40.64" width="0.3048" layer="22"/>
+<wire x1="27.432" y1="40.64" x2="27.432" y2="42.164" width="0.3048" layer="22"/>
+<wire x1="32.766" y1="42.164" x2="32.766" y2="40.64" width="0.3048" layer="22"/>
+<wire x1="32.766" y1="40.64" x2="35.052" y2="40.64" width="0.3048" layer="22"/>
+<wire x1="35.052" y1="40.64" x2="35.052" y2="42.164" width="0.3048" layer="22"/>
+<wire x1="37.846" y1="42.164" x2="37.846" y2="40.64" width="0.3048" layer="22"/>
+<wire x1="37.846" y1="40.64" x2="40.132" y2="40.64" width="0.3048" layer="22"/>
+<wire x1="40.132" y1="40.64" x2="40.132" y2="42.164" width="0.3048" layer="22"/>
+<text x="76.454" y="3.81" size="1.651" layer="21" font="vector" rot="R180" align="top-left">ON</text>
+<text x="65.278" y="3.81" size="1.651" layer="21" font="vector" rot="R180" align="top-left">OFF</text>
+<text x="94.742" y="9.906" size="1.778" layer="21" font="vector" rot="R90">B+</text>
+<text x="94.742" y="6.096" size="1.778" layer="21" font="vector" rot="R90">B-</text>
+<text x="85.852" y="6.096" size="1.778" layer="22" font="vector" rot="MR90">B-</text>
+<text x="85.852" y="9.906" size="1.778" layer="22" font="vector" rot="MR90">B+</text>
 </plain>
 <attributes>
@@
 <via x="90.678" y="19.764" extent="1-16" drill="0.35" shape="octagon"/>
 <via x="90.678" y="23.574" extent="1-16" drill="0.35" shape="octagon"/>
-<wire x1="70.463" y1="28.721" x2="70.463" y2="29.823" width="3.048" layer="16"/>
-<wire x1="70.463" y1="29.823" x2="70.612" y2="29.972" width="3.048" layer="16"/>
 <via x="66.294" y="27.892" extent="1-16" drill="0.35" shape="octagon"/>
 <via x="66.294" y="30.686" extent="1-16" drill="0.35" shape="octagon"/>
@@
 <via x="25.4" y="17.478" extent="1-16" drill="0.35" shape="octagon"/>
 <via x="25.4" y="21.288" extent="1-16" drill="0.35" shape="octagon"/>
+<wire x1="93.323" y1="28.721" x2="93.323" y2="26.416" width="3.048" layer="16"/>
+<wire x1="93.323" y1="26.416" x2="93.218" y2="26.416" width="3.048" layer="16"/>
+<wire x1="93.218" y1="26.416" x2="93.218" y2="30.734" width="3.048" layer="16"/>
+<wire x1="93.323" y1="28.721" x2="91.44" y2="28.721" width="3.048" layer="1"/>
+<wire x1="91.44" y1="28.721" x2="91.44" y2="28.448" width="3.048" layer="1"/>
+<wire x1="91.44" y1="28.721" x2="91.44" y2="29.718" width="3.048" layer="1"/>
+<wire x1="91.44" y1="29.718" x2="93.218" y2="29.718" width="3.048" layer="1"/>
+<wire x1="93.2474" y1="29.718" x2="93.218" y2="29.718" width="3.048" layer="1"/>
+<wire x1="93.218" y1="29.718" x2="93.218" y2="26.924" width="3.048" layer="1"/>
+<wire x1="70.463" y1="28.721" x2="71.628" y2="28.721" width="3.048" layer="1"/>
+<wire x1="71.628" y1="28.721" x2="71.628" y2="28.6756" width="3.048" layer="1"/>
+<wire x1="70.463" y1="28.721" x2="70.463" y2="28.702" width="3.048" layer="1"/>
+<wire x1="70.463" y1="28.702" x2="69.088" y2="28.702" width="3.048" layer="1"/>
+<wire x1="71.628" y1="28.702" x2="70.463" y2="28.702" width="3.048" layer="16"/>
+<wire x1="70.463" y1="28.721" x2="70.463" y2="28.702" width="3.048" layer="16"/>
+<wire x1="70.463" y1="28.702" x2="69.088" y2="28.702" width="3.048" layer="16"/>
 </signal>
 <signal name="V_BATT" class="1">
