File: _PCB/ESP12_DevBoard/ESP-12E Dev Board.brd (EAGLE design)
At the start: 160 x 100 mm, 13 parts, among them U1 ESP-12E

Commit message: update
Parts:
- removed LED2: (no value), adafruit:CHIP-LED0805
- added C1, C4: 100nF, rcl:C0805
- added D1: 1N5819W, Seeed-Diode:SOD-123
- added R10, R6, R7, R8, R9: 470Ω, rcl:R0805
- added R3, R4, R5: 10k, rcl:R0805
- added Y1: 12MHz, Serial-Basic:CRYSTAL-SMD-3.2X2.5
- C3: value 100nF -> 100uF; device rcl:C0805 -> rcl:SMC_A
- LED1: value (none) -> blue
- R1: value 470Ω -> 10k
- R2: value (none) -> 10k
- S1: value MOMENTARY-SWITCH-SPST-SMD-4.5MM -> RST
- S2: value MOMENTARY-SWITCH-SPST-SMD-4.5MM -> FLASH
- moved S2 63.2 mm to (-87.6, -61.0)
- moved LED1 45.8 mm to (-87.6, -39.4)
- moved R2 44.5 mm to (-48.3, -94.0)
- moved C3 44.3 mm to (-87.6, -80.0)
- moved R1 43.6 mm to (-41.9, -87.6)
Connections:
- removed net CH_PD: U1.3
- removed net REST: U1.1
- new net 5V: C3.+, C4.2
- new net EN: R3.2, U1.3
- new net N$2: D1.+, JP1.PWR
- new net N$3: R9.2, U$2.2
- new net N$4: LED1.A, R6.2
- new net N$5: R10.2, U$2.3
- new net N$6: Y1.1
- new net N$7: Y1.3
- new net POWER: R7.2, S1.2, S1.3
- new net POWER1: R8.2, S2.2, S2.3
- new net RST: C1.2, R4.2, R7.1, U1.1
- new net RXD: R9.1
- new net TXD: R10.1
- net 12V: now also D1.-; no longer JP1.PWR
- net 3.3V: now also R2.1, R3.1, R4.1, R6.1
- net GND: now also C1.1, R5.1, S1.1, S1.4, S2.1, S2.4, Y1.2, Y1.4; no longer LED1.C
- net GPIO0: now also R1.2
- net GPIO15: now also R5.2
- net GPIO16: now also LED1.C, R8.1
- net GPIO2: now also R2.2
- net N$1: now also C3.-, C4.1, U$2.16; no longer LED1.A, R1.2

Commit message: PCB update
Parts:
- removed USB1: ST-USB-001G, Seeed-Connector:MICRO-USB5+4P-SMD-0.65-B
- added C5: 100nF, rcl:C0805
- added C6, C7: 22pF, rcl:C0805
- added D2: 1N5819W, Seeed-Diode:SOD-123
- added J1: ZX62-B-5PA(33), SamacSys_Parts:ZX62B5PA33
- moved C2 63.1 mm to (-38.1, 8.89)
- moved JP3 63.1 mm to (-39.4, -3.81)
- moved R2 63.1 mm to (-38.1, -31.8)
- moved R3 63.1 mm to (-33.0, -31.8)
- moved C1 63.1 mm to (-38.1, -25.4)
- moved R1 63.1 mm to (-31.8, -25.4)
- moved R4 63.1 mm to (-38.1, -38.1)
- moved R5 63.1 mm to (-33.0, -38.1)
- moved C3 62.7 mm to (-54.6, -26.7)
- moved R6 62.7 mm to (-54.6, 21.6)
- moved R8 62.7 mm to (-54.6, -14.0)
- moved S2 62.7 mm to (-54.6, -7.62)
- moved C4 62.7 mm to (-54.6, -20.3)
- moved LED1 62.7 mm to (-54.6, 14.0)
- moved R10 62.7 mm to (-54.6, -39.4)
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Connections:
- new net D+_USB: J1.D+, U$2.5
- new net D-_USB: J1.D-, U$2.6
- new net N$8: C5.2, U$2.4
- new net N$9: D2.+, J1.VCC
- net 5V: now also D2.-
- net GND: now also C5.1, C6.1, C7.1, J1.GND, J1.SHIELD_1, J1.SHIELD_2, J1.SHIELD_3, J1.SHIELD_4, J1.SHIELD_5, J1.SHIELD_6
- net N$6: now also C7.2, U$2.8, Y1.3; no longer Y1.1
- net N$7: now also C6.2, U$2.7, Y1.1; no longer Y1.3

Commit message: ESP12E dev board schematic V1
Parts:
- removed JP3: Vout, SparkFun-Jumpers:SMT-JUMPER_2_NC_TRACE_SILK
- removed U$2: CH340G, ch340g:SOIC16
- removed Y1: 12MHz, Serial-Basic:CRYSTAL-SMD-3.2X2.5
- added C10, C12: 100nF, rcl:C0805
- added C11: 100uF, rcl:SMC_B
- added C8: 10uF, rcl:C0805
- added C9: 22uF, rcl:C0805
- added Q1: UMH3N, SamacSys_Parts:SOT65P210X100-6N
- added SJR1: ESP-12E, esp12e:ESP8266-ESP12E
- added U2: 5V_REG, SamacSys_Parts:SOT230P700X170-4N
- added U3: 3V3_REG, SamacSys_Parts:SOT230P700X170-4N
- C1, C4: value 100nF -> 10uF
- C2, C3: value 100uF -> 100nF; device rcl:SMC_A -> rcl:C0805
- C5: value 100nF -> 22uF
- C6: value 22pF -> 100uF; device rcl:C0805 -> rcl:SMC_B
- C7: value 22pF -> 220uF; device rcl:C0805 -> rcl:UD-6,3X7,7_NICHICON
- R1, R2: value 10k -> 470Ω
- R6, R7: value 470Ω -> 10k
- S1, S2: device SparkFun-Switches:TACTILE_SWITCH_SMD_4.5MM -> SparkFun-Switches:TACTILE_SWITCH_SMD_6.0X3.5MM
- U1: value ESP-12E -> CH340C; device esp12e:ESP8266-ESP12E -> ch340g:SOIC16
- moved C7 114.9 mm to (16.0, 16.5), turned to 90 degrees
- moved R10 114.5 mm to (29.5, 38.4)
- moved C3 102.5 mm to (29.5, 32.0)
- moved D1 98.6 mm to (-17.5, 5.33), turned to 90 degrees
- moved D2 88.5 mm to (-35.6, 8.64), turned to 90 degrees
- moved C5 85.8 mm to (-105.7, 32.8)
- moved C4 83.3 mm to (-105.7, 45.5)
- moved C2 82.9 mm to (35.8, 46.5)
- moved R9 81.9 mm to (-87.6, 41.9)
- moved R2 81.0 mm to (29.5, 13.0)
- moved C6 81.0 mm to (-43.7, 24.1)
- moved J1 77.8 mm to (-30.5, 2.54)
- moved R8 77.3 mm to (-87.6, 55.9)
- moved R1 75.8 mm to (29.5, 19.3)
- moved R4 75.4 mm to (-94.5, 11.9)
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Connections:
- net N$2 renamed 12V_INPUT
- net N$9 renamed 5V_INPUT
- removed net N$6: C7.2, U$2.8, Y1.3
- removed net N$7: C6.2, U$2.7, Y1.1
- removed net N$8: C5.2, U$2.4
- new net DTR: Q1.2, Q1.4, U1.13
- new net RTS: Q1.1, Q1.5, U1.14
- net 12V: now also C1.2, C4.1, U2.3
- net 3.3V: now also C11.+, C12.2, C9.2, R5.1, R8.1, SJR1.8, U3.2, U3.4; no longer C2.+, R1.1, R2.1, U1.8
- net 5V: now also C3.2, C5.1, C6.+, C7.+, C8.1, U1.16, U2.2, U2.4, U3.3; no longer C3.+, C4.2
- net ADC: now also SJR1.2; no longer U1.2
- net CS0_ESP: now also SJR1.17; no longer U1.17
- net D+_USB: now also U1.5; no longer U$2.5
- net D-_USB: now also U1.6; no longer U$2.6
- net EN: now also R5.2, SJR1.3; no longer R3.2, U1.3
- net GND: now also C10.1, C11.-, C12.1, C2.1, C3.1, C4.2, C5.2, C6.-, C7.-, C8.2, C9.1, R7.1, S1.2, S2.2, SJR1.9, U1.1, U2.1, U3.1; no longer C2.-, C5.1, C6.1, C7.1, R5.1, S1.1, S1.4, S2.1, S2.4, U1.9, Y1.2, Y1.4
- net GPIO0: now also Q1.3, R3.2, SJR1.12; no longer R1.2, U1.12
- net GPIO10: now also SJR1.20; no longer U1.20
- net GPIO12: now also SJR1.6; no longer U1.6
- net GPIO13: now also SJR1.7; no longer U1.7
- net GPIO14: now also SJR1.5; no longer U1.5
- net GPIO15: now also R7.2, SJR1.10; no longer R5.2, U1.10
- net GPIO16: now also R10.1, SJR1.4; no longer R8.1, U1.4
- net GPIO2: now also R4.2, SJR1.11; no longer R2.2, U1.11
- net GPIO4: now also SJR1.13; no longer U1.13
- net GPIO5: now also SJR1.14; no longer U1.14
- net GPIO9: now also SJR1.19; no longer U1.19
- net MISO_ESP: now also SJR1.18; no longer U1.18
- net MOSI_ESP: now also SJR1.21; no longer U1.21
- net N$1: now also C2.2, U1.4; no longer C3.-, C4.1, U$2.16
- net N$3: now also R1.2, U1.2; no longer R9.2, U$2.2
- net N$4: now also R8.2; no longer R6.2
- net N$5: now also R2.2, U1.3; no longer R10.2, U$2.3
- net POWER: now also R9.2, S1.1; no longer R7.2, S1.2, S1.3
- net POWER1: now also R10.2, S2.1; no longer R8.2, S2.2, S2.3
- net RST: now also C10.2, Q1.6, R6.2, R9.1, SJR1.1; no longer C1.2, R4.2, R7.1, U1.1
- net RXD: now also R1.1; no longer R9.1
- net RXD_ESP: now also SJR1.15; no longer U1.15
- net SCLK_ESP: now also SJR1.22; no longer U1.22
- net TXD: now also R2.1; no longer R10.1
- net TXD_ESP: now also SJR1.16; no longer U1.16
Other:
- board size 160 x 100 mm -> 70 x 75 mm

Commit message: PCB schematic final V1
Parts:
- added J10: BUTTON1, con-molex-spox:5267-3
- added J11: DUST_SENSOR, con-molex-spox:5267-4
- added J2: LCD_CONN, con-molex-spox:5267-8
- added J3, J5: I2C, con-molex-spox:5267-4
- added J4: LCD_BACKLIGHT, con-molex-spox:5267-2
- added J6: RADON_SENSOR, con-molex-spox:5267-4
- added J8: ADC, con-molex-spox:5267-3
- added J9: TEMP/HUM SENSOR, con-molex-spox:5267-4
- added R11: 47k(1%), rcl:R0805
- added R12: 10k(1%), rcl:R0805
- added R13: 470Ω, rcl:R0805
- added U4: TXB0104, SparkFun-IC-Comms:TSSOP14
- added VR1: RK09K1130AAU, SamacSys_Parts:RK09K1130BGM
- C3: value 100nF -> 10uF
- C4, C8: value 10uF -> 22uF
- C5: value 22uF -> 100uF; device rcl:C0805 -> rcl:SMC_B
- C6: value 100uF -> 220uF(optional); device rcl:SMC_B -> rcl:UD-6,3X7,7_NICHICON
- C7: value 220uF -> 10uF; device rcl:UD-6,3X7,7_NICHICON -> rcl:C0805
- C9: value 22uF -> 100nF
- LED1: value blue -> green
- R1, R2: value 470Ω -> 10k
- R6, R7: value 10k -> 470Ω
- U1: value CH340C -> 5V_REG; device ch340g:SOIC16 -> SamacSys_Parts:SOT230P700X170-4N
- U2: value 5V_REG -> 3.3V_REG
- U3: value 3V3_REG -> CH340C; device SamacSys_Parts:SOT230P700X170-4N -> ch340g:SOIC16
- moved R10 102.6 mm to (-68.6, 68.6)
- moved R2 102.4 mm to (-52.1, 74.9)
- moved R1 94.5 mm to (-47.0, 74.9)
- moved C9 91.8 mm to (-24.1, 68.6)
- moved C1 87.7 mm to (-16.5, 74.9)
- moved S2 87.2 mm to (-17.8, 81.3), turned to 0 degrees
- moved C4 81.9 mm to (-29.2, 74.9)
- moved C10 81.4 mm to (-30.5, 68.6)
- moved R6 81.2 mm to (-43.2, 68.6)
- moved C7 77.9 mm to (-35.6, 74.9), turned to 0 degrees
- moved D1 76.5 mm to (-26.7, 81.3), turned to 0 degrees
- moved R7 74.6 mm to (-49.5, 68.6)
- moved C8 73.1 mm to (-41.9, 74.9)
- moved D2 72.7 mm to (-34.3, 81.3), turned to 0 degrees
- moved C12 70.8 mm to (-36.8, 68.6)
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Connections:
- removed net RXD_ESP: SJR1.15
- removed net TXD_ESP: SJR1.16
- new net LED+_5V: J2.P$7, J4.P$2, U4.11
- new net LED-_5V: J2.P$8, U4.10
- new net N$2: J2.P$3, VR1.2
- new net N$6: J6.P$3, R10.2
- new net N$9: J11.P$3, R13.2
- new net SCL_5V: J2.P$4, J3.P$3, J5.P$3, U4.13
- new net SDA_5V: J2.P$5, J3.P$4, J5.P$4, U4.12
- net 12V: now also C3.1, J6.P$2, U1.3; no longer C4.1, U2.3
- net 3.3V: now also C8.2, J10.P$2, J9.P$2, R1.1, R2.1, U2.2, U2.4, U4.1, U4.8; no longer C9.2, R5.1, R8.1, U3.2, U3.4
- net 5V: now also C10.2, C4.1, C5.+, C7.1, J11.P$2, J2.P$2, J3.P$2, J5.P$2, J8.P$2, U1.2, U1.4, U2.3, U3.16, U4.14, VR1.3; no longer C3.2, C5.1, C7.+, C8.1, U1.16, U2.2, U2.4, U3.3
- net ADC: now also R11.1, R12.2
- net D+_USB: now also U3.5; no longer U1.5
- net D-_USB: now also U3.6; no longer U1.6
- net DTR: now also U3.13; no longer U1.13
- net EN: now also R3.2; no longer R5.2
- net GND: now also C3.2, C5.-, C7.2, C8.1, J10.P$1, J11.P$1, J2.P$1, J3.P$1, J4.P$1, J5.P$1, J6.P$1, J8.P$1, J9.P$1, LED1.C, R12.1, R5.1, U4.7, VR1.1; no longer C3.1, C5.2, C7.-, C8.2, R7.1
- net GPIO0: now also R1.2, U4.4; no longer R3.2
- net GPIO12: now also R10.1
- net GPIO13: now also J6.P$4
- net GPIO14: now also R13.1
- net GPIO15: now also J10.P$3, R5.2; no longer R7.2
- net GPIO16: now also J11.P$4, R8.1; no longer LED1.C, R10.1
- net GPIO2: now also R2.2, U4.5; no longer R4.2
- net GPIO4: now also J9.P$4, U4.3
- net GPIO5: now also J9.P$3, U4.2
- net N$1: now also C9.2, U3.4; no longer C2.2, U1.4
- net N$3: now also R9.2, U3.2; no longer R1.2, U1.2
- net N$4: now also R6.2; no longer R8.2
- net N$5: now also J8.P$3, R11.2; no longer R2.2, U1.3
- net POWER: now also R7.2; no longer R9.2
- net POWER1: now also R8.2; no longer R10.2
- net RST: now also C2.2, R4.2, R7.1; no longer C10.2, R6.2, R9.1
- net RTS: now also U3.14; no longer U1.14
- net RXD: now also R9.1, SJR1.15; no longer R1.1
- net TXD: now also SJR1.16, U3.3; no longer R2.1
Other:
- board size 70 x 75 mm -> 70 x 70 mm

Commit message: PCB artwork
Parts:
- removed J11: DUST_SENSOR, con-molex-spox:5267-4
- added J7: RADON_SENSOR, con-molex-spox:5267-4
- J10: value BUTTON1 -> DUST_SENSOR; device con-molex-spox:5267-3 -> con-molex-spox:5267-4
- J2: value LCD_CONN -> I2C; device con-molex-spox:5267-8 -> con-molex-spox:5267-4
- J3: value I2C -> LCD; device con-molex-spox:5267-4 -> con-molex-spox:5267-8
- J4: value LCD_BACKLIGHT -> I2C; device con-molex-spox:5267-2 -> con-molex-spox:5267-4
- J5: value I2C -> LCD_BACKLIGHT; device con-molex-spox:5267-4 -> con-molex-spox:5267-2
- J6: value RADON_SENSOR -> TEMP/HUM SENSOR
- J8: value ADC -> BUTTON1
- J9: value TEMP/HUM SENSOR -> ADC; device con-molex-spox:5267-4 -> con-molex-spox:5267-3
- R12: value 10k(1%) -> 470Ω
- R13: value 470Ω -> 10k(1%)
- moved S1 152.0 mm to (59.4, 3.81)
- moved R12 141.6 mm to (65.5, 43.4), turned to 180 degrees
- moved R10 138.1 mm to (65.5, 35.8), turned to 180 degrees
- moved R7 120.2 mm to (54.4, 8.13)
- moved R5 113.5 mm to (41.4, 42.2), turned to 180 degrees
- moved C5 112.7 mm to (65.3, 30.2)
- moved U1 111.5 mm to (41.7, 17.5), turned to 90 degrees
- moved R6 108.1 mm to (44.7, 5.59), turned to 180 degrees
- moved J1 103.6 mm to (34.8, 2.54)
- moved J2 102.1 mm to (51.3, 67.1)
- moved LED1 100.6 mm to (44.7, 2.03), turned to 270 degrees
- moved D2 98.2 mm to (31.5, 8.38), turned to 180 degrees
- moved R13 97.5 mm to (18.5, 40.9), turned to 180 degrees
- moved J10 97.3 mm to (51.3, 44.2)
- moved R9 96.1 mm to (25.9, 30.2)
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Connections:
- net 12V: now also J7.P$2; no longer J6.P$2
- net 3.3V: now also J6.P$2, J8.P$2; no longer J10.P$2, J9.P$2
- net 5V: now also J10.P$2, J4.P$2, J9.P$2; no longer J11.P$2, J5.P$2, J8.P$2
- net ADC: now also R13.2; no longer R12.2
- net GND: now also J7.P$1, R13.1; no longer J11.P$1, R12.1
- net GPIO13: now also J7.P$4; no longer J6.P$4
- net GPIO14: now also R12.1; no longer R13.1
- net GPIO15: now also J8.P$3; no longer J10.P$3
- net GPIO16: now also J10.P$4; no longer J11.P$4
- net GPIO4: now also J6.P$4; no longer J9.P$4
- net GPIO5: now also J6.P$3; no longer J9.P$3
- net LED+_5V: now also J5.P$2; no longer J2.P$7, J4.P$2
- net LED-_5V: no longer J2.P$8
- net N$2: now also J3.P$3; no longer J2.P$3
- net N$5: now also J9.P$3; no longer J8.P$3
- net N$6: now also J7.P$3; no longer J6.P$3
- net N$9: now also J10.P$3, R12.2; no longer J11.P$3, R13.2
- net SCL_5V: now also J2.P$3, J3.P$4, J4.P$3; no longer J2.P$4, J3.P$3, J5.P$3
- net SDA_5V: now also J2.P$4, J3.P$5, J4.P$4; no longer J2.P$5, J3.P$4, J5.P$4
Routing:
- added copper zone on layer 1, net GND
- added copper zone on layer 16, net GND

Commit message: PCB layout V1
Parts:
- removed R9: 470Ω, rcl:R0805
- added J11: BTN2, con-molex-spox:5267-3
- J10: value DUST_SENSOR -> DUST
- J6: value TEMP/HUM SENSOR -> TEMP/HUM
- J7: value RADON_SENSOR -> RADON
- J8: value BUTTON1 -> BTN1
- U2: value 3.3V_REG -> 3V3_REG
- moved R12 60.5 mm to (11.6, 16.0), turned to 270 degrees
- moved J5 55.9 mm to (2.03, 5.89), turned to 90 degrees
- moved R10 55.3 mm to (13.9, 16.0), turned to 270 degrees
- moved R7 48.0 mm to (6.99, 16.0), turned to 270 degrees
- moved J7 45.9 mm to (5.76, 41.9)
- moved U4 37.1 mm to (35.9, 18.7)
- moved R5 36.5 mm to (16.0, 16.0), turned to 90 degrees
- moved J3 36.1 mm to (1.78, 16.6), turned to 90 degrees
- moved VR1 34.9 mm to (11.3, 57.8), turned to 0 degrees
- moved J8 32.5 mm to (8.21, 35.0)
- moved C11 28.6 mm to (42.4, 18.2), turned to 270 degrees
- moved C10 27.1 mm to (20.1, 20.4), turned to 90 degrees
- moved J9 26.5 mm to (39.6, 55.8)
- moved C5 23.1 mm to (45.5, 18.2), turned to 270 degrees
- moved J2 21.4 mm to (39.8, 49.0)
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Connections:
- removed net 12V_INPUT: D1.+, JP1.PWR
- removed net LED+_5V: J5.P$2, U4.11
- removed net LED-_5V: U4.10
- new net LED+: J3.P$7, J5.P$2
- new net RXD_5V: U3.2, U4.10
- new net TXD_5V: U3.3, U4.11
- net 12V: no longer C1.2
- net 3.3V: no longer J8.P$2
- net 5V: now also J11.P$2, J8.P$2
- net GND: now also J11.P$1, J3.P$8
- net GPIO0: now also R12.1; no longer U4.4
- net GPIO12: now also J7.P$4; no longer R10.1
- net GPIO13: now also J8.P$3; no longer J7.P$4
- net GPIO14: now also R10.1; no longer R12.1
- net GPIO15: now also J11.P$3; no longer J8.P$3
- net GPIO16: no longer J10.P$4
- net GPIO2: now also J10.P$4; no longer U4.5
- net N$3: now also C1.2, D1.+, JP1.PWR; no longer R9.2, U3.2
- net RXD: now also U4.5; no longer R9.1
- net TXD: now also U4.4; no longer U3.3
Other:
- board size 70 x 70 mm -> 52 x 60 mm
- board text added: "12V"
- board text added: "5V"
- board text added: "A0"
- board text added: "D3"
- board text added: "D4"
- board text added: "D5"
- board text added: "D6"
- board text added: "D7"
- board text added: "D8"
- board text added: "GND"
- board text added: "SCL"
- board text added: "SDA"

Commit message: update
Parts:
- moved R11 34.8 mm to (33.2, 30.2), turned to 270 degrees
- moved R13 32.1 mm to (31.2, 30.2), turned to 90 degrees
- moved Q1 12.1 mm to (18.7, 24.2), turned to 180 degrees
- moved R10 2.55 mm to (14.1, 18.6)
- moved R12 2.55 mm to (11.9, 18.6)
- moved R5 2.55 mm to (16.2, 18.6)
- moved R7 2.55 mm to (7.24, 18.6)
- moved R8 2.55 mm to (9.53, 18.6)
- moved C12 1.98 mm to (18.5, 31.5)
- moved VR1 1.02 mm to (10.2, 57.8)
- moved SJR1 0.51 mm to (26.0, 44.1)
- moved J9 0.15 mm to (39.8, 55.8)
Routing:
- net 5V: track 0.00 -> 134.3 mm
- net 3.3V: track 0.00 -> 77.9 mm
- net 12V: track 0.00 -> 55.2 mm, vias 0 -> 1
- net POWER: track 0.00 -> 40.2 mm
- net N$5: track 0.00 -> 31.8 mm, vias 0 -> 1
- net POWER1: track 0.00 -> 27.8 mm, vias 0 -> 2
- net N$3: track 0.00 -> 13.9 mm
- net SDA_5V: track 0.00 -> 6.86 mm
- net SCL_5V: track 0.00 -> 6.86 mm
- net 5V_INPUT: track 0.00 -> 5.41 mm
- net ADC: track 0.00 -> 2.03 mm
- net RST: track 0.00 -> 2.03 mm
Other:
- outline, holes or cut-outs redrawn

Commit message: PCB artwork V1
Parts:
- moved C12 1.37 mm to (19.0, 30.2)
- moved VR1 0.80 mm to (11.0, 58.0)
Routing:
- net SDA_5V: track 6.86 -> 118.2 mm, vias 0 -> 3
- net SCL_5V: track 6.86 -> 98.8 mm, vias 0 -> 5
- net GPIO2: track 0.00 -> 78.6 mm
- net GPIO0: track 0.00 -> 61.9 mm, vias 0 -> 5
- net RST: track 2.03 -> 57.5 mm, vias 0 -> 6
- net GPIO16: track 0.00 -> 53.8 mm
- net GPIO4: track 0.00 -> 46.5 mm, vias 0 -> 2
- net N$9: track 0.00 -> 43.0 mm, vias 0 -> 1
- net GND: track 0.00 -> 42.7 mm, vias 1 -> 39
- net GPIO15: track 0.00 -> 38.8 mm, vias 0 -> 1
- net RXD: track 0.00 -> 37.8 mm, vias 0 -> 2
- net TXD: track 0.00 -> 37.1 mm, vias 0 -> 2
- net GPIO5: track 0.00 -> 36.5 mm, vias 0 -> 2
- net EN: track 0.00 -> 36.4 mm
- net 5V: track 134.3 -> 169.2 mm, vias 0 -> 3
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