File: _PCB/ESP12_DevBoard/ASDF.brd (EAGLE design)
At the start: 52 x 60 mm, 51 parts, among them J1 ZX62-B-5PA(33), J10 DUST, J11 BTN2, J2 I2C, J3 LCD, J4 I2C, J5 LCD_BACKLIGHT, J6 TEMP/HUM, J7 RADON, J8 BTN1, J9 ADC, Q1 UMH3N, U1 5V_REG, U2 3V3_REG, U3 CH340C, U4 TXB0104

Commit message: PCB V1.3 update
Routing:
- net ADC: track 4.61 -> 36.1 mm, vias 1 -> 2
- net EN: track 20.0 -> 36.4 mm, vias 2 -> 0
- net RST: track 60.7 -> 57.2 mm
- net GPIO0: track 73.9 -> 71.9 mm
- net GPIO4: track 56.5 -> 55.1 mm
- net GPIO5: track 39.0 -> 38.1 mm
