File: _PCB/ESP12_DevBoard/ESP-12E Dev Board.sch (EAGLE design)
At the start: 48 parts, among them J1 ZX62-B-5PA(33), J10 BUTTON1, J11 DUST_SENSOR, J2 LCD_CONN, J3 I2C, J4 LCD_BACKLIGHT, J5 I2C, J6 RADON_SENSOR, J8 ADC, J9 TEMP/HUM SENSOR, Q1 UMH3N, U1 5V_REG, U2 3.3V_REG, U3 CH340C, U4 TXB0104

Commit message: PCB artwork
Parts:
- removed J11: DUST_SENSOR, con-molex-spox:5267-4
- added J7: RADON_SENSOR, con-molex-spox:5267-4
- J10: value BUTTON1 -> DUST_SENSOR; device con-molex-spox:5267-3 -> con-molex-spox:5267-4
- J2: value LCD_CONN -> I2C; device con-molex-spox:5267-8 -> con-molex-spox:5267-4
- J3: value I2C -> LCD; device con-molex-spox:5267-4 -> con-molex-spox:5267-8
- J4: value LCD_BACKLIGHT -> I2C; device con-molex-spox:5267-2 -> con-molex-spox:5267-4
- J5: value I2C -> LCD_BACKLIGHT; device con-molex-spox:5267-4 -> con-molex-spox:5267-2
- J6: value RADON_SENSOR -> TEMP/HUM SENSOR
- J8: value ADC -> BUTTON1
- J9: value TEMP/HUM SENSOR -> ADC; device con-molex-spox:5267-4 -> con-molex-spox:5267-3
- R12: value 10k(1%) -> 470Ω
- R13: value 470Ω -> 10k(1%)
Connections:
- net 12V: now also J7.-2; no longer J6.-2
- net 3.3V: now also J6.-2, J8.-2; no longer J10.-2, J9.-2
- net 5V: now also J10.-2, J4.-2, J9.-2; no longer J11.-2, J5.-2, J8.-2
- net ADC: now also R13.2; no longer R12.2
- net GND: now also J7.-1, R13.1; no longer J11.-1, R12.1
- net GPIO13: now also J7.-4; no longer J6.-4
- net GPIO14: now also R12.1; no longer R13.1
- net GPIO15: now also J8.-3; no longer J10.-3
- net GPIO16: now also J10.-4; no longer J11.-4
- net GPIO4: now also J6.-4; no longer J9.-4
- net GPIO5: now also J6.-3; no longer J9.-3
- net LED+_5V: now also J5.-2; no longer J2.-7, J4.-2
- net LED-_5V: no longer J2.-8
- net N$2: now also J3.-3; no longer J2.-3
- net N$5: now also J9.-3; no longer J8.-3
- net N$6: now also J7.-3; no longer J6.-3
- net N$9: now also J10.-3, R12.2; no longer J11.-3, R13.2
- net SCL_5V: now also J2.-3, J3.-4, J4.-3; no longer J2.-4, J3.-3, J5.-3
- net SDA_5V: now also J2.-4, J3.-5, J4.-4; no longer J2.-5, J3.-4, J5.-4
Other:
- note added: "SCL : D1 SDA: D2 LED+(pullup) : D3 LED-(pullup) : D4 button1(pulldown): D8 미세먼지센서: D5, D0 (RX/TX) 라돈센서: D6, D7 (RX/TX)"
- note removed: "SCL : D1 - 5 SDA: D2 - 4 LED+ : D3 - 0 LED- : D4 - 2 button1: D8 - 15 미세먼지센서: D5, D0 (RX/TX) - 14, 16 라돈센서: D6, D7 (RX/TX) - 12, 13"
- moved on the sheet: J6, J8, R12, R13

Commit message: PCB layout V1
Parts:
- removed R9: 470Ω, rcl:R-US_R0805
- added J11: BTN2, con-molex-spox:5267-3
- J10: value DUST_SENSOR -> DUST
- J6: value TEMP/HUM SENSOR -> TEMP/HUM
- J7: value RADON_SENSOR -> RADON
- J8: value BUTTON1 -> BTN1
- U2: value 3.3V_REG -> 3V3_REG
Connections:
- removed net 12V_INPUT: D1.+, JP1.PWR
- removed net LED+_5V: J5.-2, U4.B3
- removed net LED-_5V: U4.B4
- new net LED+: J3.-7, J5.-2
- new net RXD_5V: U3.TX, U4.B4
- new net TXD_5V: U3.RX, U4.B3
- net 12V: no longer C1.2
- net 3.3V: no longer J8.-2
- net 5V: now also J11.-2, J8.-2
- net GND: now also J11.-1, J3.-8
- net GPIO0: now also R12.1; no longer U4.A3
- net GPIO12: now also J7.-4; no longer R10.1
- net GPIO13: now also J8.-3; no longer J7.-4
- net GPIO14: now also R10.1; no longer R12.1
- net GPIO15: now also J11.-3; no longer J8.-3
- net GPIO16: no longer J10.-4
- net GPIO2: now also J10.-4; no longer U4.A4
- net N$3: now also C1.2, D1.+, JP1.PWR; no longer R9.2, U3.TX
- net RXD: now also U4.A4; no longer R9.1
- net TXD: now also U4.A3; no longer U3.RX
Other:
- note added: "SCL/SDA : D1/D2 (5/4) 미세먼지센서: D3/D4 (0/2) 라돈센서: D5/D6 (14/12) Button1: D7 (13) Button2: D8 (15) Analog: ADC"
- note added: "VDD"
- note added: "VSS"
- note removed: "Button1_pulldown"
- note removed: "I2C_SCL"
- note removed: "I2C_SDA"
- note removed: "LCD_LED+_pullup"
- note removed: "LCD_LED-_pullup"
- note removed: "SCL : D1 SDA: D2 LED+(pullup) : D3 LED-(pullup) : D4 button1(pulldown): D8 미세먼지센서: D5, D0 (RX/TX) 라돈센서: D6, D7 (RX/TX)"
- moved on the sheet: C1, D1, J10, J3, J8, R12, VR1

Commit message: PCB edit
Connections:
- net 5V: now also J5.-1
- net GND: no longer J5.-1
Changed lines of the file:
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@@
 <?xml version="1.0" encoding="utf-8"?>
 <!DOCTYPE eagle SYSTEM "eagle.dtd">
-<eagle version="9.3.2">
+<eagle version="9.4.0">
 <drawing>
 <settings>
@@
 <setting verticaltext="up"/>
 </settings>
-<grid distance="0.1" unitdist="inch" unit="inch" style="lines" multiple="1" display="no" altdistance="0.01" altunitdist="inch" altunit="inch"/>
+<grid distance="50" unitdist="mil" unit="mil" style="lines" multiple="1" display="no" altdistance="0.01" altunitdist="inch" altunit="inch"/>
 <layers>
 <layer number="1" name="Top" color="4" fill="1" visible="no" active="no"/>
@@
 <part name="GND11" library="SparkFun-PowerSymbols" library_urn="urn:adsk.eagle:library:530" deviceset="GND" device=""/>
 <part name="SUPPLY11" library="SparkFun-PowerSymbols" library_urn="urn:adsk.eagle:library:530" deviceset="5V" device=""/>
-<part name="GND16" library="SparkFun-PowerSymbols" library_urn="urn:adsk.eagle:library:530" deviceset="GND" device=""/>
 <part name="FRAME2" library="frames" library_urn="urn:adsk.eagle:library:229" deviceset="A4L-LOC" device=""/>
 <part name="FRAME1" library="frames" library_urn="urn:adsk.eagle:library:229" deviceset="A4L-LOC" device=""/>
@@
 <part name="SUPPLY18" library="SparkFun-PowerSymbols" library_urn="urn:adsk.eagle:library:530" deviceset="5V" device=""/>
 <part name="SUPPLY22" library="SparkFun-PowerSymbols" library_urn="urn:adsk.eagle:library:530" deviceset="5V" device=""/>
+<part name="SUPPLY23" library="SparkFun-PowerSymbols" library_urn="urn:adsk.eagle:library:530" deviceset="5V" device=""/>
 </parts>
 <sheets>
@@
 <attribute name="VALUE" x="222.25" y="164.084" size="1.778" layer="96" align="bottom-center"/>
 </instance>
-<instance part="GND16" gate="1" x="187.96" y="130.81" smashed="yes" rot="R180">
-<attribute name="VALUE" x="187.96" y="131.064" size="1.778" layer="96" rot="R180" align="top-center"/>
-</instance>
 <instance part="FRAME2" gate="G$1" x="1.27" y="1.27" smashed="yes">
 <attribute name="DRAWING_NAME" x="218.44" y="16.51" size="2.54" layer="94"/>
@@
 <instance part="SUPPLY22" gate="G$1" x="224.79" y="54.61" smashed="yes">
 <attribute name="VALUE" x="224.79" y="57.404" size="1.778" layer="96" align="bottom-center"/>
+</instance>
+<instance part="SUPPLY23" gate="G$1" x="187.96" y="129.54" smashed="yes">
+<attribute name="VALUE" x="187.96" y="132.334" size="1.778" layer="96" align="bottom-center"/>
 </instance>
 </instances>
@@
 <wire x1="233.68" y1="157.48" x2="228.6" y2="157.48" width="0.1524" layer="91"/>
 <wire x1="228.6" y1="157.48" x2="228.6" y2="161.29" width="0.1524" layer="91"/>
-</segment>
-<segment>
-<pinref part="GND16" gate="1" pin="GND"/>
-<pinref part="J5" gate="G$1" pin="-1"/>
-<wire x1="187.96" y1="128.27" x2="187.96" y2="124.46" width="0.1524" layer="91"/>
-<wire x1="187.96" y1="124.46" x2="193.04" y2="124.46" width="0.1524" layer="91"/>
 </segment>
 <segment>
@@
 <wire x1="224.79" y1="48.26" x2="224.79" y2="54.61" width="0.1524" layer="91"/>
 </segment>
-</net>
+<segment>
+<pinref part="J5" gate="G$1" pin="-1"/>
+<wire x1="187.96" y1="124.46" x2="193.04" y2="124.46" width="0.1524" layer="91"/>
+<pinref part="SUPPLY23" gate="G$1" pin="5V"/>
+<wire x1="187.96" y1="129.54" x2="187.96" y2="124.46" width="0.1524" layer="91"/>
+</segment>
+</net>

Commit message: final edit sample edit
Changed lines of the file:
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@@
 <setting verticaltext="up"/>
 </settings>
-<grid distance="50" unitdist="mil" unit="mil" style="lines" multiple="1" display="no" altdistance="0.01" altunitdist="inch" altunit="inch"/>
+<grid distance="0.1" unitdist="inch" unit="inch" style="lines" multiple="1" display="no" altdistance="0.01" altunitdist="inch" altunit="inch"/>
 <layers>
 <layer number="1" name="Top" color="4" fill="1" visible="no" active="no"/>
@@
 <text x="203.962" y="156.718" size="1.524" layer="97">VDD</text>
 <text x="203.962" y="159.258" size="1.524" layer="97">VSS</text>
+<text x="244.602" y="131.318" size="1.524" layer="97">SCL</text>
+<text x="244.602" y="128.778" size="1.524" layer="97">SDA</text>
+<text x="244.602" y="108.458" size="1.524" layer="97">SCL</text>
+<text x="244.602" y="105.918" size="1.524" layer="97">SDA</text>
 </plain>
 <instances>

Commit message: PCB V1.3 update
Parts:
- removed R7: 470Ω, rcl:R-US_R0805
- added C13: 220uF, rcl:CPOL-USUD-6,3X7,7
- added C14: 100nF, rcl:C-EUC0805
- added R14, R9: 10k, rcl:R-US_R0805
- C6: value 220uF(optional) -> 220uF
- R6: value 470Ω -> 10k
Connections:
- removed net 5V_INPUT: D2.+, J1.VCC
- removed net POWER: R7.2, S1.1
- new net N$10: C14.2, D2.+, J1.VCC
- new net N$7: R9.2, U3.DTR
- new net N$8: R14.2, U3.RTS
- net 3.3V: now also C13.+
- net DTR: now also R9.1; no longer U3.DTR
- net GND: now also C13.-, C14.1
- net GPIO0: now also R8.1
- net GPIO16: no longer R8.1
- net RST: now also S1.1; no longer R7.1
- net RTS: now also R14.1; no longer U3.RTS
Other:
- moved on the sheet: C6, D2

Commit message: optimization _ gerber errors
Parts:
- removed C7: 10uF, rcl:C-EUC0805
Connections:
- net 5V: no longer C7.1
- net GND: no longer C7.2
Changed lines of the file:
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@@
 <part name="SUPPLY8" library="SparkFun-PowerSymbols" library_urn="urn:adsk.eagle:library:530" deviceset="3.3V" device=""/>
 <part name="C3" library="rcl" library_urn="urn:adsk.eagle:library:334" deviceset="C-EU" device="C0805" package3d_urn="urn:adsk.eagle:package:23617/2" value="10uF"/>
-<part name="C7" library="rcl" library_urn="urn:adsk.eagle:library:334" deviceset="C-EU" device="C0805" package3d_urn="urn:adsk.eagle:package:23617/2" value="10uF"/>
 <part name="C4" library="rcl" library_urn="urn:adsk.eagle:library:334" deviceset="C-EU" device="C0805" package3d_urn="urn:adsk.eagle:package:23617/2" value="22uF"/>
 <part name="C8" library="rcl" library_urn="urn:adsk.eagle:library:334" deviceset="C-EU" device="C0805" package3d_urn="urn:adsk.eagle:package:23617/2" value="22uF"/>
@@
 <attribute name="VALUE" x="176.022" y="116.459" size="1.778" layer="96"/>
 </instance>
-<instance part="C7" gate="G$1" x="175.26" y="63.5" smashed="yes">
-<attribute name="NAME" x="176.022" y="63.627" size="1.778" layer="95"/>
-<attribute name="VALUE" x="175.768" y="59.309" size="1.778" layer="96"/>
-</instance>
 <instance part="C4" gate="G$1" x="218.44" y="120.65" smashed="yes">
 <attribute name="NAME" x="219.202" y="121.031" size="1.778" layer="95"/>
@@
 <wire x1="185.42" y1="63.5" x2="185.42" y2="57.15" width="0.1524" layer="91"/>
 <wire x1="185.42" y1="57.15" x2="185.42" y2="53.34" width="0.1524" layer="91"/>
-<wire x1="175.26" y1="57.15" x2="185.42" y2="57.15" width="0.1524" layer="91"/>
 <junction x="185.42" y="57.15"/>
 <pinref part="C8" gate="G$1" pin="1"/>
 <wire x1="185.42" y1="57.15" x2="218.44" y2="57.15" width="0.1524" layer="91"/>
 <wire x1="218.44" y1="57.15" x2="218.44" y2="58.42" width="0.1524" layer="91"/>
-<pinref part="C7" gate="G$1" pin="2"/>
-<wire x1="175.26" y1="58.42" x2="175.26" y2="57.15" width="0.1524" layer="91"/>
 <pinref part="C13" gate="G$1" pin="-"/>
 <wire x1="218.44" y1="57.15" x2="228.6" y2="57.15" width="0.1524" layer="91"/>
@@
 <wire x1="185.42" y1="67.31" x2="189.23" y2="67.31" width="0.1524" layer="91"/>
 <pinref part="SUPPLY7" gate="G$1" pin="5V"/>
-<wire x1="175.26" y1="67.31" x2="185.42" y2="67.31" width="0.1524" layer="91"/>
-<junction x="185.42" y="67.31"/>
-<pinref part="C7" gate="G$1" pin="1"/>
-<wire x1="175.26" y1="66.04" x2="175.26" y2="67.31" width="0.1524" layer="91"/>
-</segment>
-<segment>
+</segment>
+<segment>
