File: _PCB/ESP12_DevBoard/ESP-12E Dev Board_with_level_shifter.brd (EAGLE design)
At the start: 52 x 60 mm, 47 parts, among them J1 ZX62-B-5PA(33), J10 BTN1, J11 BTN2, J2 I2C, J3 LCD, J4 I2C, J5 LCD_BACKLIGHT, J6 TEMP/HUM, J7 RADON, J8 DUST, J9 ADC, Q1 UMH3N, U1 5V_REG, U2 3V3_REG, U3 CH340C

Commit message: ESP12 dev board V1.4 final commit
Parts:
- added C12, C15: 100nF, rcl:C0805
- added U4: TXS0104, SparkFun-IC-Comms:TSSOP14
Connections:
- new net SCL_5V: J2.P$3, J3.P$4, J4.P$3, U4.13
- new net SDA_5V: J2.P$4, J3.P$5, J4.P$4, U4.12
- net 3.3V: now also C15.2, U4.1, U4.8
- net 5V: now also C12.2, U4.14
- net GND: now also C12.1, C15.1, U4.7
- net GPIO4: now also U4.3; no longer J2.P$4, J3.P$5, J4.P$4
- net GPIO5: now also U4.2; no longer J2.P$3, J3.P$4, J4.P$3
Routing:
- net SCL_5V: track 0.00 -> 102.5 mm, vias 0 -> 3
- net SDA_5V: track 0.00 -> 79.9 mm, vias 0 -> 4
- net GPIO5: track 83.0 -> 40.8 mm
- net GPIO4: track 89.9 -> 51.0 mm, vias 4 -> 2
- net GPIO2: track 40.1 -> 74.7 mm, vias 2 -> 0
- net 5V: track 163.8 -> 176.3 mm, vias 1 -> 2
- net 3.3V: track 115.0 -> 127.2 mm, vias 5 -> 6
