File: _PCB/_Prototyping_Boards/Universal PCB/DoubleBoard_TypeC.brd (EAGLE design)
At the start: 49 x 70 mm, 4 parts, among them J1 TYPE-C-31-M-17, J2 TYPE-C-31-M-17

Commit message: PCB misc update
Routing:
- net N$1: track 7.37 -> 0.00 mm
- net GND: track 113.1 -> 118.5 mm, vias 12 -> 14
- net 5V: track 79.2 -> 83.4 mm
Changed lines of the file:
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@@
 <?xml version="1.0" encoding="utf-8"?>
 <!DOCTYPE eagle SYSTEM "eagle.dtd">
-<eagle version="9.4.2">
+<eagle version="9.5.0">
 <drawing>
 <settings>
@@
 <setting verticaltext="up"/>
 </settings>
-<grid distance="1" unitdist="mil" unit="mil" style="lines" multiple="1" display="no" altdistance="5" altunitdist="mil" altunit="mil"/>
+<grid distance="0.2" unitdist="mm" unit="mm" style="lines" multiple="1" display="no" altdistance="5" altunitdist="mil" altunit="mil"/>
 <layers>
 <layer number="1" name="Top" color="4" fill="1" visible="yes" active="yes"/>
@@
 <wire x1="1" y1="0" x2="1" y2="7" width="0.1524" layer="21"/>
 <dimension x1="0" y1="0" x2="0" y2="70" x3="-3" y3="35" textsize="1.778" layer="51"/>
-<dimension x1="0" y1="0" x2="49" y2="0" x3="24.5" y3="-3" textsize="1.778" layer="51"/>
+<dimension x1="0" y1="-0.1" x2="49" y2="0" x3="24.506121875" y3="-3.04999375" textsize="1.778" layer="51"/>
 <wire x1="16.256" y1="2.3622" x2="30.226" y2="2.3622" width="0.1524" layer="21"/>
 <wire x1="30.226" y1="2.3622" x2="30.734" y2="1.905" width="0.1524" layer="21"/>
@@
 <text x="27.94" y="67.564" size="1.016" layer="21" font="vector" ratio="12" rot="R180">5V</text>
 <text x="36.068" y="67.564" size="1.016" layer="21" font="vector" ratio="12" rot="R180">GND</text>
-<rectangle x1="6.7818" y1="64.4398" x2="7.3914" y2="64.5668" layer="29"/>
+<rectangle x1="5.08" y1="7.112" x2="11.684" y2="8.382" layer="29"/>
+<rectangle x1="6.731" y1="63.246" x2="10.033" y2="64.897" layer="29"/>
 </plain>
 <attributes>
@@
 <via x="4.225340625" y="62.91061875" extent="1-16" drill="1.016" diameter="1.8796" shape="octagon"/>
 </signal>
-<signal name="N$448">
-<via x="6.765340625" y="62.91061875" extent="1-16" drill="1.016" diameter="1.8796" shape="octagon"/>
-</signal>
-<signal name="N$449">
-<via x="9.305340625" y="62.91061875" extent="1-16" drill="1.016" diameter="1.8796" shape="octagon"/>
-</signal>
 <signal name="N$450">
 <via x="11.845340625" y="62.91061875" extent="1-16" drill="1.016" diameter="1.8796" shape="octagon"/>
@@
 <wire x1="16.925340625" y1="68.75261875" x2="19.465340625" y2="68.75261875" width="0.508" layer="16"/>
 <wire x1="19.465340625" y1="68.75261875" x2="29.625340625" y2="68.75261875" width="0.508" layer="16"/>
-<wire x1="9.682" y1="65.347" x2="9.682" y2="64.8416" width="0.4064" layer="1"/>
-<wire x1="9.682" y1="64.8416" x2="9.7536" y2="64.77" width="0.4064" layer="1"/>
-<wire x1="13.617296875" y1="67.30481875" x2="16.002" y2="67.30481875" width="0.4064" layer="1"/>
-<wire x1="12.531140625" y1="66.2186625" x2="13.617296875" y2="67.30481875" width="0.4064" layer="1"/>
-<wire x1="16.002" y1="67.30481875" x2="16.925340625" y2="68.228159375" width="0.4064" layer="1"/>
+<wire x1="16.925340625" y1="68.228159375" x2="16.002" y2="67.30481875" width="0.4064" layer="1"/>
 <wire x1="16.925340625" y1="68.228159375" x2="16.925340625" y2="68.75261875" width="0.4064" layer="1"/>
-<wire x1="11.082478125" y1="64.77" x2="11.133278125" y2="64.8208" width="0.4064" layer="1"/>
-<wire x1="11.082478125" y1="64.77" x2="9.7536" y2="64.77" width="0.4064" layer="1"/>
-<wire x1="11.133278125" y1="64.8208" x2="11.96053125" y2="64.8208" width="0.4064" layer="1"/>
-<wire x1="11.96053125" y1="64.8208" x2="12.531140625" y2="65.391409375" width="0.4064" layer="1"/>
-<wire x1="12.531140625" y1="65.391409375" x2="12.531140625" y2="66.2186625" width="0.4064" layer="1"/>
-<wire x1="9.902" y1="6.496" x2="9.7536" y2="64.77" width="0" layer="19" extent="1-1"/>
+<wire x1="9.902" y1="6.496" x2="9.902" y2="7.87" width="0.762" layer="1"/>
+<wire x1="9.902" y1="7.87" x2="9.906" y2="7.874" width="0.762" layer="1"/>
+<wire x1="6.862" y1="6.496" x2="6.858" y2="6.5" width="0.762" layer="1"/>
+<wire x1="6.858" y1="6.5" x2="6.858" y2="7.874" width="0.762" layer="1"/>
+<wire x1="13.11429375" y1="66.9664" x2="13.4527125" y2="67.30481875" width="0.4064" layer="1"/>
+<wire x1="16.002" y1="67.30481875" x2="13.4527125" y2="67.30481875" width="0.4064" layer="1"/>
+<wire x1="9.990225" y1="65.1676" x2="10.573775" y2="65.1676" width="0.4064" layer="1"/>
+<wire x1="10.573775" y1="65.1676" x2="10.9864" y2="65.580225" width="0.4064" layer="1"/>
+<wire x1="9.810825" y1="65.347" x2="9.990225" y2="65.1676" width="0.4064" layer="1"/>
+<wire x1="9.682" y1="65.347" x2="9.810825" y2="65.347" width="0.4064" layer="1"/>
+<wire x1="10.9864" y1="65.580225" x2="10.9864" y2="66.5228" width="0.4064" layer="1"/>
+<wire x1="10.9864" y1="66.5228" x2="11.43" y2="66.9664" width="0.4064" layer="1"/>
+<wire x1="11.43" y1="66.9664" x2="13.11429375" y2="66.9664" width="0.4064" layer="1"/>
+<wire x1="9.682" y1="65.347" x2="9.682" y2="63.276" width="0.4064" layer="1"/>
+<wire x1="9.906" y1="7.874" x2="9.682" y2="63.276" width="0" layer="19" extent="1-1"/>
 </signal>
 <signal name="GND">
@@
 <contactref element="J2" pad="GND"/>
 <contactref element="J2" pad="GND_2"/>
-<wire x1="5.632" y1="6.496" x2="5.632" y2="8.0958" width="0.508" layer="1"/>
-<wire x1="10.9583375" y1="8.2072" x2="11.132" y2="8.0335375" width="0.508" layer="1"/>
-<wire x1="11.132" y1="8.0335375" x2="11.132" y2="6.496" width="0.508" layer="1"/>
-<wire x1="5.632" y1="8.0958" x2="5.7434" y2="8.2072" width="0.508" layer="1"/>
-<wire x1="5.7434" y1="8.2072" x2="10.9583375" y2="8.2072" width="0.508" layer="1"/>
-<wire x1="11.132" y1="6.496" x2="11.132" y2="3.854" width="0.508" layer="1"/>
 <wire x1="31.529159375" y1="1.31561875" x2="32.165340625" y2="1.31561875" width="0.508" layer="1"/>
-<wire x1="11.3256" y1="3.6604" x2="13.0998125" y2="3.6604" width="0.508" layer="1"/>
+<wire x1="13.0998125" y1="3.6604" x2="11.3256" y2="3.6604" width="0.508" layer="1"/>
 <wire x1="30.182959375" y1="2.66181875" x2="31.529159375" y2="1.31561875" width="0.508" layer="1"/>
 <wire x1="13.0998125" y1="3.6604" x2="14.09839375" y2="2.66181875" width="0.508" layer="1"/>
 <wire x1="14.09839375" y1="2.66181875" x2="30.182959375" y2="2.66181875" width="0.508" layer="1"/>
-<wire x1="11.132" y1="3.854" x2="11.3256" y2="3.6604" width="0.508" layer="1"/>
 <via x="32.165340625" y="68.75261875" extent="1-16" drill="1.016" diameter="1.8796" shape="octagon"/>
 <via x="34.705340625" y="68.75261875" extent="1-16" drill="1.016" diameter="1.8796" shape="octagon"/>
@@
 <wire x1="42.325340625" y1="68.75261875" x2="44.865340625" y2="68.75261875" width="0.508" layer="1"/>
 <wire x1="32.165340625" y1="68.75261875" x2="44.865340625" y2="68.75261875" width="0.508" layer="16"/>
-<wire x1="7.082" y1="65.347" x2="7.082" y2="64.292" width="0.4064" layer="1"/>
-<wire x1="7.082" y1="64.292" x2="7.1628" y2="64.2112" width="0.4064" layer="1"/>
-<wire x1="7.1628" y1="64.2112" x2="12.1412" y2="64.2112" width="0.4064" layer="1"/>
-<wire x1="12.1412" y1="64.2112" x2="13.089940625" y2="65.159940625" width="0.4064" layer="1"/>
-<wire x1="13.089940625" y1="65.159940625" x2="13.089940625" y2="65.98719375" width="0.4064" layer="1"/>
-<wire x1="13.089940625" y1="65.98719375" x2="13.848765625" y2="66.74601875" width="0.4064" layer="1"/>
-<wire x1="32.165340625" y1="68.233340625" x2="32.165340625" y2="68.75261875" width="0.4064" layer="1"/>
-<wire x1="13.848765625" y1="66.74601875" x2="30.67801875" y2="66.74601875" width="0.4064" layer="1"/>
-<wire x1="30.67801875" y1="66.74601875" x2="32.165340625" y2="68.233340625" width="0.4064" layer="1"/>
-<wire x1="11.132" y1="6.496" x2="7.1628" y2="64.2112" width="0" layer="19" extent="1-1"/>
+<wire x1="5.632" y1="6.496" x2="5.632" y2="4.02" width="0.508" layer="1"/>
+<wire x1="11.132" y1="6.496" x2="11.132" y2="3.854" width="0.508" layer="1"/>
+<wire x1="11.132" y1="3.854" x2="11.3256" y2="3.6604" width="0.508" layer="1"/>
+<via x="6.858" y="3.556" extent="1-16" drill="0.35"/>
+<wire x1="5.632" y1="4.02" x2="6.096" y2="3.556" width="0.508" layer="1"/>
+<wire x1="6.096" y1="3.556" x2="6.858" y2="3.556" width="0.508" layer="1"/>
+<via x="9.652" y="3.556" extent="1-16" drill="0.35"/>
+<wire x1="6.858" y1="3.556" x2="9.652" y2="3.556" width="0.508" layer="16"/>
+<wire x1="11.3256" y1="3.6604" x2="9.7564" y2="3.6604" width="0.508" layer="1"/>
+<wire x1="9.7564" y1="3.6604" x2="9.652" y2="3.556" width="0.508" layer="1"/>
+<wire x1="11.132" y1="6.496" x2="11.132" y2="7.83" width="0.762" layer="1"/>
+<wire x1="5.632" y1="6.496" x2="5.632" y2="7.918" width="0.762" layer="1"/>
+<wire x1="32.165340625" y1="68.75261875" x2="30.158740625" y2="66.74601875" width="0.4064" layer="1"/>
+<wire x1="13.84876875" y1="66.74601875" x2="13.08994375" y2="65.98719375" width="0.4064" layer="1"/>
+<wire x1="30.158740625" y1="66.74601875" x2="13.84876875" y2="66.74601875" width="0.4064" layer="1"/>
+<wire x1="13.08994375" y1="65.98719375" x2="13.08994375" y2="64.39794375" width="0.4064" layer="1"/>
+<wire x1="11.30876875" y1="64.20601875" x2="10.54994375" y2="63.44719375" width="0.4064" layer="1"/>
+<wire x1="10.54994375" y1="63.44719375" x2="10.54994375" y2="62.61994375" width="0.4064" layer="1"/>
+<wire x1="10.54994375" y1="62.61994375" x2="10.16" y2="62.23" width="0.4064" layer="1"/>
+<wire x1="12.89801875" y1="64.20601875" x2="11.30876875" y2="64.20601875" width="0.4064" layer="1"/>
+<wire x1="10.16" y1="62.23" x2="7.874" y2="62.23" width="0.4064" layer="1"/>
+<wire x1="7.082" y1="63.022" x2="7.082" y2="65.347" width="0.4064" layer="1"/>
+<wire x1="13.08994375" y1="64.39794375" x2="12.89801875" y2="64.20601875" width="0.4064" layer="1"/>
+<wire x1="7.874" y1="62.23" x2="7.082" y2="63.022" width="0.4064" layer="1"/>
+<wire x1="5.632" y1="7.918" x2="7.082" y2="65.347" width="0" layer="19" extent="1-1"/>
 </signal>
 <signal name="N$1">
@@
 <contactref element="J3" pad="SHIELD1"/>
 <contactref element="J3" pad="SHIELD2"/>
-<wire x1="4.697" y1="68.072" x2="8.382" y2="68.072" width="0.508" layer="1"/>
-<wire x1="8.382" y1="68.072" x2="12.067" y2="68.072" width="0.508" layer="1"/>
+<wire x1="8.382" y1="68.072" x2="12.067" y2="68.072" width="0" layer="19" extent="1-1"/>
+<wire x1="4.697" y1="68.072" x2="8.382" y2="68.072" width="0" layer="19" extent="1-1"/>
 </signal>
 <signal name="N$3">
