File: _PCB/SAMD21_DevBoard/board.sch (EAGLE design)
At the start: 1 part, among them U1 ATSAMD21G-A

Commit message: added samples
Parts:
- removed U1: ATSAMD21G-A, SparkFun-IC-Microcontroller:ATSAMD21G-A
- added IC1: ATSAMD21G18A-AU, SamacSys_Parts:ATSAMD21G18A-AU
Changed lines of the file:
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@@
 <parts>
 <part name="FRAME1" library="frames" library_urn="urn:adsk.eagle:library:229" deviceset="A4L-LOC" device=""/>
-<part name="U1" library="SparkFun-IC-Microcontroller" library_urn="urn:adsk.eagle:library:525" deviceset="ATSAMD21G" device="-A" package3d_urn="urn:adsk.eagle:package:38963/1"/>
+<part name="IC1" library="SamacSys_Parts" deviceset="ATSAMD21G18A-AU" device=""/>
 </parts>
 <sheets>
@@
 <attribute name="SHEET" x="230.505" y="5.08" size="2.54" layer="94"/>
 </instance>
-<instance part="U1" gate="G$1" x="116.84" y="91.44" smashed="yes">
-<attribute name="NAME" x="86.36" y="137.414" size="1.778" layer="95"/>
-<attribute name="VALUE" x="86.36" y="58.166" size="1.778" layer="96" align="top-left"/>
+<instance part="IC1" gate="G$1" x="104.14" y="101.6" smashed="yes">
+<attribute name="NAME" x="121.92" y="129.54" size="1.778" layer="95" align="center-left"/>
+<attribute name="VALUE" x="121.92" y="127" size="1.778" layer="96" align="center-left"/>
 </instance>
 </instances>
@@
 will not be understood (or retained) with this version.
 </note>
-<note version="8.3" severity="warning">
-Since Version 8.3, EAGLE supports the association of 3D packages
-with devices in libraries, schematics, and board files. Those 3D
-packages will not be understood (or retained) with this version.
-</note>
 </compatibility>

Commit message: SAMD21 dev board update
Parts:
- removed IC1: ATSAMD21G18A-AU, SamacSys_Parts:ATSAMD21G18A-AU
- added C1: 4.7n / 1kv, rcl:C-EUC0402K
- added D1: PRTR5V0U2X,215, SamacSys_Parts:PRTR5V0U2X,215
- added J1: U-F-M5DD-Y-L, SamacSys_Parts:U-F-M5DD-Y-L
- added JP1, JP2: JUMPER-SMT_2_NO_SILK, SparkFun-Jumpers:JUMPER-SMT_2_NO_SILK
- added R1: 1M, rcl:R-US_R0402
- added U1: ATSAMD21G-A, SparkFun-IC-Microcontroller:ATSAMD21G-A
Connections:
- new net GND: C1.2, D1.GND, J1.GND, R1.1
- new net N$1: C1.1, J1.SHIELD, R1.2
- new net N$2: D1.I/O_2, J1.D-
- new net N$3: D1.I/O_1, J1.D+
- new net V_USB: D1.VCC, J1.VBUS

Commit message: library update
Connections:
- net N$2 renamed USB_D-
- net N$3 renamed USB_D+
Changed lines of the file:
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@@
 <setting verticaltext="up"/>
 </settings>
-<grid distance="0.05" unitdist="inch" unit="inch" style="lines" multiple="1" display="no" altdistance="0.01" altunitdist="inch" altunit="inch"/>
+<grid distance="0.05" unitdist="inch" unit="mil" style="lines" multiple="1" display="no" altdistance="0.01" altunitdist="inch" altunit="inch"/>
 <layers>
 <layer number="1" name="Top" color="4" fill="1" visible="no" active="no"/>
@@
 <layer number="230" name="230bmp" color="7" fill="1" visible="yes" active="yes"/>
 <layer number="231" name="231bmp" color="7" fill="1" visible="yes" active="yes"/>
+<layer number="232" name="Eagle3D_PG2" color="7" fill="1" visible="no" active="no"/>
+<layer number="233" name="Eagle3D_PG3" color="7" fill="1" visible="no" active="no"/>
 <layer number="248" name="Housing" color="7" fill="1" visible="yes" active="yes"/>
 <layer number="249" name="Edge" color="7" fill="1" visible="yes" active="yes"/>
@@
 </variantdefs>
 <classes>
-<class number="0" name="default" width="0" drill="0">
+<class number="0" name="default" width="0.2032" drill="0">
+</class>
+<class number="1" name="power" width="0.508" drill="0">
 </class>
 </classes>
 <parts>
 <part name="FRAME1" library="frames" library_urn="urn:adsk.eagle:library:229" deviceset="A4L-LOC" device=""/>
-<part name="SUPPLY1" library="SparkFun-PowerSymbols" library_urn="urn:adsk.eagle:library:530" deviceset="V_USB" device=""/>
-<part name="SUPPLY2" library="SparkFun-PowerSymbols" library_urn="urn:adsk.eagle:library:530" deviceset="3.3V" device=""/>
-<part name="SUPPLY3" library="SparkFun-PowerSymbols" library_urn="urn:adsk.eagle:library:530" deviceset="5V" device=""/>
-<part name="GND1" library="SparkFun-PowerSymbols" library_urn="urn:adsk.eagle:library:530" deviceset="GND" device=""/>
-<part name="SUPPLY4" library="SparkFun-PowerSymbols" library_urn="urn:adsk.eagle:library:530" deviceset="VIN" device=""/>
-<part name="SUPPLY5" library="SparkFun-PowerSymbols" library_urn="urn:adsk.eagle:library:530" deviceset="V_BATT" device=""/>
-<part name="JP1" library="SparkFun-Jumpers" library_urn="urn:adsk.eagle:library:528" deviceset="JUMPER-SMT_2_NO" device="_SILK" package3d_urn="urn:adsk.eagle:package:39279/1"/>
+<part name="SUPPLY1" library="SparkFun-PowerSymbols" deviceset="V_USB" device=""/>
+<part name="SUPPLY2" library="SparkFun-PowerSymbols" deviceset="3.3V" device=""/>
+<part name="SUPPLY3" library="SparkFun-PowerSymbols" deviceset="5V" device=""/>
+<part name="GND1" library="SparkFun-PowerSymbols" deviceset="GND" device=""/>
+<part name="SUPPLY4" library="SparkFun-PowerSymbols" deviceset="VIN" device=""/>
+<part name="SUPPLY5" library="SparkFun-PowerSymbols" deviceset="V_BATT" device=""/>
+<part name="JP1" library="SparkFun-Jumpers" deviceset="JUMPER-SMT_2_NO" device="_SILK" package3d_urn="urn:adsk.eagle:package:39279/1"/>
 <part name="D1" library="SamacSys_Parts" deviceset="PRTR5V0U2X,215" device=""/>
 <part name="J1" library="SamacSys_Parts" deviceset="U-F-M5DD-Y-L" device=""/>
 <part name="FRAME2" library="frames" library_urn="urn:adsk.eagle:library:229" deviceset="A4L-LOC" device=""/>
-<part name="SUPPLY6" library="SparkFun-PowerSymbols" library_urn="urn:adsk.eagle:library:530" deviceset="V_USB" device=""/>
-<part name="SUPPLY7" library="SparkFun-PowerSymbols" library_urn="urn:adsk.eagle:library:530" deviceset="3.3V" device=""/>
-<part name="SUPPLY8" library="SparkFun-PowerSymbols" library_urn="urn:adsk.eagle:library:530" deviceset="5V" device=""/>
-<part name="GND2" library="SparkFun-PowerSymbols" library_urn="urn:adsk.eagle:library:530" deviceset="GND" device=""/>
-<part name="SUPPLY9" library="SparkFun-PowerSymbols" library_urn="urn:adsk.eagle:library:530" deviceset="VIN" device=""/>
-<part name="SUPPLY10" library="SparkFun-PowerSymbols" library_urn="urn:adsk.eagle:library:530" deviceset="V_BATT" device=""/>
-<part name="JP2" library="SparkFun-Jumpers" library_urn="urn:adsk.eagle:library:528" deviceset="JUMPER-SMT_2_NO" device="_SILK" package3d_urn="urn:adsk.eagle:package:39279/1"/>
-<part name="U1" library="SparkFun-IC-Microcontroller" library_urn="urn:adsk.eagle:library:525" deviceset="ATSAMD21G" device="-A" package3d_urn="urn:adsk.eagle:package:38963/1"/>
-<part name="SUPPLY11" library="SparkFun-PowerSymbols" library_urn="urn:adsk.eagle:library:530" deviceset="V_USB" device=""/>
-<part name="GND3" library="SparkFun-PowerSymbols" library_urn="urn:adsk.eagle:library:530" deviceset="GND" device=""/>
-<part name="GND4" library="SparkFun-PowerSymbols" library_urn="urn:adsk.eagle:library:530" deviceset="GND" device=""/>
+<part name="SUPPLY6" library="SparkFun-PowerSymbols" deviceset="V_USB" device=""/>
+<part name="SUPPLY7" library="SparkFun-PowerSymbols" deviceset="3.3V" device=""/>
+<part name="SUPPLY8" library="SparkFun-PowerSymbols" deviceset="5V" device=""/>
+<part name="GND2" library="SparkFun-PowerSymbols" deviceset="GND" device=""/>
+<part name="SUPPLY9" library="SparkFun-PowerSymbols" deviceset="VIN" device=""/>
+<part name="SUPPLY10" library="SparkFun-PowerSymbols" deviceset="V_BATT" device=""/>
+<part name="JP2" library="SparkFun-Jumpers" deviceset="JUMPER-SMT_2_NO" device="_SILK" package3d_urn="urn:adsk.eagle:package:39279/1"/>
+<part name="U1" library="SparkFun-IC-Microcontroller" deviceset="ATSAMD21G" device="-A"/>
+<part name="SUPPLY11" library="SparkFun-PowerSymbols" deviceset="V_USB" device=""/>
+<part name="GND3" library="SparkFun-PowerSymbols" deviceset="GND" device=""/>
+<part name="GND4" library="SparkFun-PowerSymbols" deviceset="GND" device=""/>
 <part name="C1" library="rcl" library_urn="urn:adsk.eagle:library:334" deviceset="C-EU" device="C0402K" package3d_urn="urn:adsk.eagle:package:23679/2" value="4.7n / 1kv"/>
 <part name="R1" library="rcl" library_urn="urn:adsk.eagle:library:334" deviceset="R-US_" device="R0402" package3d_urn="urn:adsk.eagle:package:23547/3" value="1M"/>
@@
 </busses>
 <nets>
-<net name="GND" class="0">
+<net name="GND" class="1">
 <segment>
 <pinref part="J1" gate="G$1" pin="GND"/>
@@
 </segment>
 </net>
-<net name="V_USB" class="0">
+<net name="V_USB" class="1">
 <segment>
 <pinref part="J1" gate="G$1" pin="VBUS"/>
@@
 </segment>
 </net>
-<net name="N$2" class="0">
+<net name="USB_D-" class="0">
 <segment>
 <pinref part="J1" gate="G$1" pin="D-"/>
@@
 <wire x1="68.58" y1="114.3" x2="68.58" y2="125.73" width="0.1524" layer="91"/>
 <junction x="68.58" y="125.73"/>
-</segment>
-</net>
-<net name="N$3" class="0">
+<label x="87.63" y="125.73" size="1.27" layer="95" xref="yes"/>
+</segment>
+</net>
+<net name="USB_D+" class="0">
 <segment>
 <pinref part="J1" gate="G$1" pin="D+"/>
@@
 <wire x1="71.12" y1="114.3" x2="71.12" y2="123.19" width="0.1524" layer="91"/>
 <junction x="71.12" y="123.19"/>
-</segment>
-</net>
+<label x="87.63" y="123.19" size="1.27" layer="95" xref="yes"/>
+</segment>
+</net>
