File: _PCB/_Prototyping_Boards/Universal PCB with USB connectors/DoubleBoard_TypeC.brd (EAGLE design)
At the start: 49 x 70 mm, 4 parts, among them J1 TYPE-C-31-M-17, J2 TYPE-C-31-M-17

Commit message: Type-C proto PCB
Parts:
- removed J3, J4: (no value), SparkFun-Connectors:USB-B-MICRO-SMD
- J1: value TYPE-C-31-M-17 -> ZX62D-B-5P8; device Type-C_Hroparts:TYPE-C-31-M-17 -> angrypig7_Library:HRS_ZX62D-B-5P8
- moved J1 57.4 mm to (30.5, 3.05)
- moved J2 11.2 mm to (19.6, 6.60)
Connections:
- removed net 5V: J2.VBUS, J2.VBUS_2, J3.VBUS
- removed net N$1: J3.SHIELD1, J3.SHIELD2, J3.SHIELD3
- removed net N$10: J1.GND, J1.GND_2, J4.GND
- removed net N$2: J1.VBUS, J1.VBUS_2, J4.VBUS
- removed net N$3: J4.SHIELD1, J4.SHIELD2, J4.SHIELD3
- new net D+: J1.3
- new net D-: J1.2
- new net SHIELD: J1.S1, J1.S2, J1.S3, J1.S4, J1.S5, J1.S6, J2.P$1, J2.P$2, J2.P$3, J2.P$4
- new net VCC: J1.1, J2.VBUS, J2.VBUS_2
- net GND: now also J1.5; no longer J3.GND
Routing:
- net 5V: track 81.9 -> 0.00 mm, vias 12 -> 0
- net VCC: track 0.00 -> 64.9 mm, vias 0 -> 9
- net GND: track 115.5 -> 65.6 mm, vias 14 -> 9
- net SHIELD: track 0.00 -> 41.6 mm
- net N$1: track 7.37 -> 0.00 mm
- net D+: track 0.00 -> 4.41 mm, vias 0 -> 2
- net D-: track 0.00 -> 4.34 mm, vias 0 -> 2
Other:
- board text added: "D+"
- board text added: "D-"
- board text added: "VCC"
- board text removed: "5V"
