File: _PCB/_Prototyping_Boards/Universal PCB with USB connectors/ProtoBoard_Type-C_Micro5pin.brd (EAGLE design)
At the start: 49 x 70 mm, 2 parts, among them J1 ZX62D-B-5P8, J2 TYPE-C-31-M-17

Commit message: cleanup
Routing:
- net GND: track 65.6 -> 64.7 mm
- net VCC: vias 9 -> 8
