File: _EAGLE/Projects/_Development_Boards/JTAG adapter board/board.sch (EAGLE design)
At the start: 9 parts, among them J1 PROG-HEADER_2X3_SHROUDED, J10 PROG-HEADER_2X5_1.27MM-PTH+SMD, J2 PROG-HEADER_2X5_2.00MM-SHROUD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, J3 PROG-HEADER_2X5_SHROUDED, J5 PROG-HEADER_2X10_RIGHT-ANGLE, J6 PROG-HEADER_2X10_SHROUDED, J8 CONN-1X4, J9 CONN-1X6

Commit message: JTAG board V1
Parts:
- added JP2: (no value), pinhead_v2:PINHD-1X6/OCT
Connections:
- removed net N$2: J10.9
- net GND: now also JP2.3
- net RST: now also JP2.5
- net TCK: now also JP2.2
- net TDO: now also JP2.6
- net TMS: now also JP2.4
- net VCC: now also JP2.1
Changed lines of the file:
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@@
 <schematic xreflabel="%F%N/%S.%C%R" xrefpart="/%S.%C%R">
 <attributes>
-<attribute name="CNAME" value="J-Link adapter"/>
+<attribute name="CNAME" value="JTAG adapter"/>
 <attribute name="CREVISION" value="V1"/>
 </attributes>
@@
 <part name="J2" library="angrypig7-Connectors-Programming" deviceset="PROG-HEADER_2X5" device="_2.00MM-SHROUDED"/>
 <part name="J5" library="angrypig7-Connectors-Programming" deviceset="PROG-HEADER_2X10" device="_RIGHT-ANGLE"/>
+<part name="JP2" library="pinhead_v2" deviceset="PINHD-1X6" device="/OCT"/>
 </parts>
 <sheets>
@@
 <attribute name="VALUE" x="132.08" y="108.204" size="1.778" layer="96" font="vector"/>
 </instance>
+<instance part="JP2" gate="A" x="224.79" y="114.3" smashed="yes">
+<attribute name="NAME" x="218.44" y="125.095" size="1.778" layer="95"/>
+<attribute name="VALUE" x="218.44" y="104.14" size="1.778" layer="96"/>
+</instance>
 </instances>
 <busses>
@@
 </segment>
 <segment>
-<wire x1="201.93" y1="121.92" x2="207.01" y2="121.92" width="0.1524" layer="91"/>
 <label x="207.01" y="121.92" size="1.27" layer="95" xref="yes"/>
 <pinref part="J9" gate="G$1" pin="1"/>
+<pinref part="JP2" gate="A" pin="1"/>
+<wire x1="222.25" y1="121.92" x2="201.93" y2="121.92" width="0.1524" layer="91"/>
 </segment>
 <segment>
@@
 </segment>
 <segment>
-<wire x1="201.93" y1="114.3" x2="207.01" y2="114.3" width="0.1524" layer="91"/>
 <label x="207.01" y="114.3" size="1.27" layer="95" xref="yes"/>
 <pinref part="J9" gate="G$1" pin="4"/>
+<pinref part="JP2" gate="A" pin="4"/>
+<wire x1="201.93" y1="114.3" x2="222.25" y2="114.3" width="0.1524" layer="91"/>
 </segment>
 </net>
@@
 </segment>
 <segment>
-<wire x1="201.93" y1="109.22" x2="207.01" y2="109.22" width="0.1524" layer="91"/>
 <label x="207.01" y="109.22" size="1.27" layer="95" xref="yes"/>
 <pinref part="J9" gate="G$1" pin="6"/>
+<pinref part="JP2" gate="A" pin="6"/>
+<wire x1="201.93" y1="109.22" x2="222.25" y2="109.22" width="0.1524" layer="91"/>
 </segment>
 </net>
@@
 </segment>
 <segment>
-<wire x1="201.93" y1="111.76" x2="207.01" y2="111.76" width="0.1524" layer="91"/>
 <label x="207.01" y="111.76" size="1.27" layer="95" xref="yes"/>
 <pinref part="J9" gate="G$1" pin="5"/>
+<pinref part="JP2" gate="A" pin="5"/>
+<wire x1="201.93" y1="111.76" x2="222.25" y2="111.76" width="0.1524" layer="91"/>
 </segment>
 </net>
@@
 </segment>
 <segment>
-<wire x1="201.93" y1="116.84" x2="207.01" y2="116.84" width="0.1524" layer="91"/>
 <label x="207.01" y="116.84" size="1.27" layer="95" xref="yes"/>
 <pinref part="J9" gate="G$1" pin="3"/>
+<pinref part="JP2" gate="A" pin="3"/>
+<wire x1="222.25" y1="116.84" x2="201.93" y2="116.84" width="0.1524" layer="91"/>
 </segment>
 </net>
@@
 </segment>
 <segment>
-<wire x1="201.93" y1="119.38" x2="207.01" y2="119.38" width="0.1524" layer="91"/>
 <label x="207.01" y="119.38" size="1.27" layer="95" xref="yes"/>
 <pinref part="J9" gate="G$1" pin="2"/>
+<pinref part="JP2" gate="A" pin="2"/>
+<wire x1="201.93" y1="119.38" x2="222.25" y2="119.38" width="0.1524" layer="91"/>
 </segment>
 </net>
@@
 </segment>
 </net>
-<net name="N$2" class="0">
-<segment>
-<pinref part="J10" gate="G$1" pin="9"/>
-<wire x1="54.61" y1="92.71" x2="53.34" y2="92.71" width="0.1524" layer="91"/>
-</segment>
-</net>
